File: matrix.kicad_sch (KiCad schematic)
At the start: 216 parts, among them SW1 ESC, SW10 F8, SW100 MENU, SW101 R_CTRL, SW102 L_ARROW, SW103 DN_ARROW, SW104 R_ARROW, SW105 PAD_0, SW106 SW_Push, SW107 PAD_., SW108 PAD_ENTER, SW11 F9, SW12 F10, SW13 F11, SW14 F12, SW15 PRT_SC, SW16 SCR_LK, SW17 PAUSE, SW18 TILDE, SW19 1, SW2 SW_Push, SW20 2, SW21 3, SW22 4, SW23 5, SW24 6, SW25 7, SW26 8, SW27 9, SW28 0, SW29 -, SW3 F1, SW30 =, SW31 BACKSPACE, SW32 INSERT, SW33 HOME, SW34 PG_UP, SW35 NUM_LK, SW36 PAD_/, SW37 *, SW38 PAD_-, SW39 TAB, SW4 F2, SW40 Q, SW41 W, SW42 E, SW43 R, SW44 T, SW45 Y, SW46 U, SW47 I, SW48 O, SW49 P, SW5 F3, SW50 [, SW51 ], SW52 \, SW53 DEL, SW54 END, SW55 PG_DN, SW56 PAD_7, SW57 PAD_8, SW58 PAD_9, SW59 +, SW6 F4, SW60 CAPS, SW61 A, SW62 S, SW63 D, SW64 F, SW65 G, SW66 H, SW67 J, SW68 K, SW69 L, SW7 F5, SW70 ;, SW71 ', SW72 ENTER, SW73 PAD_4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

Commit message: Finished Electric Schematic Of Keyboard
All components are now wired. Positions for spacers, button stabilizers, and threated holes not accounted.
Parts:
- removed D3: D_Small, symbol Device:D_Small
- removed SW2: SW_Push, symbol Switch:SW_Push
- renumbered D11 to D10, D101 to D100, D102 to D101, D103 to D102, D104 to D103, D105 to D104, D106 to D105, D107 to D106, D108 to D107, D109 to D108, D12 to D11, D13 to D12, D14 to D13, D15 to D14, D16 to D15, D17 to D16, D18 to D17, D19 to D18, D20 to D19, D21 to D20, D22 to D21, D23 to D22, D24 to D23, D25 to D24, D26 to D25, D27 to D26, D28 to D27, D29 to D28, D30 to D29, D4 to D3, D31 to D30, D32 to D31, D34 to D32, D35 to D33, D36 to D34, D37 to D35, D38 to D36, D39 to D37, D33 to D38, D40 to D39, D5 to D4, D41 to D40, D42 to D41, D43 to D42, D44 to D43, D45 to D44, D46 to D45, D47 to D46, D48 to D47, D49 to D48, D50 to D49, D6 to D5, D51 to D50, D52 to D51, D53 to D52, D54 to D53, D55 to D54, D56 to D55, D57 to D56, D58 to D57, D59 to D58, D60 to D59, D7 to D6, D61 to D60, D62 to D61, D63 to D62, D64 to D63, D65 to D64, D66 to D65, D67 to D66, D68 to D67, D69 to D68, D70 to D69, D8 to D7, D71 to D70, D72 to D71, D73 to D72, D74 to D73, D75 to D74, D76 to D75, D77 to D76, D78 to D77, D79 to D78, D80 to D79, D9 to D8, D81 to D80, D82 to D81, D83 to D82, D84 to D83, D85 to D84, D86 to D85, D87 to D86, D88 to D87, D89 to D88, D90 to D89, D10 to D9, D91 to D90, D92 to D91, D93 to D92, D94 to D93, D95 to D94, D96 to D95, D97 to D96, D98 to D97, D99 to D98, D100 to D99, SW9 to SW10, SW99 to SW100, SW100 to SW101, SW101 to SW102, SW102 to SW103, SW103 to SW104, SW104 to SW105, SW105 to SW106, SW106 to SW107, SW107 to SW108, SW108 to SW109, SW10 to SW11, SW11 to SW12, SW12 to SW13, SW13 to SW14, SW14 to SW15, SW15 to SW16, SW16 to SW17, SW17 to SW18, SW18 to SW19, SW19 to SW20, SW20 to SW21, SW21 to SW22, SW22 to SW23, SW23 to SW24, SW24 to SW25, SW25 to SW26, SW26 to SW27, SW27 to SW28, SW28 to SW29, SW1 to SW3, SW29 to SW30, SW30 to SW31, SW31 to SW32, SW32 to SW39, SW3 to SW4, SW39 to SW40, SW40 to SW41, SW41 to SW42, SW42 to SW43, SW43 to SW44, SW44 to SW45, SW45 to SW46, SW46 to SW47, SW47 to SW48, SW48 to SW49, SW4 to SW5, SW49 to SW50, SW50 to SW51, SW51 to SW52, SW52 to SW53, SW53 to SW54, SW54 to SW55, SW55 to SW56, SW56 to SW57, SW57 to SW58, SW58 to SW59, SW5 to SW6, SW59 to SW60, SW60 to SW61, SW61 to SW62, SW62 to SW63, SW63 to SW64, SW64 to SW65, SW65 to SW66, SW66 to SW67, SW67 to SW68, SW68 to SW69, SW6 to SW7, SW69 to SW70, SW70 to SW71, SW71 to SW72, SW72 to SW73, SW73 to SW74, SW74 to SW75, SW75 to SW76, SW76 to SW77, SW77 to SW78, SW78 to SW79, SW7 to SW8, SW79 to SW80, SW80 to SW81, SW81 to SW82, SW82 to SW83, SW83 to SW84, SW84 to SW85, SW85 to SW86, SW86 to SW87, SW87 to SW88, SW88 to SW89, SW8 to SW9, SW89 to SW90, SW90 to SW91, SW91 to SW92, SW92 to SW93, SW93 to SW94, SW94 to SW95, SW95 to SW96, SW96 to SW97, SW97 to SW98, SW98 to SW99
Connections:
- net COL20 is gone; now on net COL19: SW109.2, SW38.2, SW60.2, SW77.2, SW94.2
- net COL13: now also SW103.2
- net COL14: now also SW17.2, SW33.2, SW55.2; no longer SW103.2
- net COL15: no longer SW104.2, SW17.2, SW33.2, SW55.2, SW90.2
- net COL16: now also SW106.2, SW35.2, SW57.2, SW74.2, SW91.2; no longer SW105.2, SW18.2, SW34.2, SW56.2
- net COL17: now also SW107.2, SW36.2, SW58.2, SW75.2, SW92.2; no longer SW106.2, SW35.2, SW57.2, SW74.2, SW91.2
- net COL18: now also SW108.2, SW37.2, SW59.2, SW76.2, SW93.2; no longer SW107.2, SW36.2, SW58.2, SW75.2, SW92.2
- net COL19: no longer SW108.2, SW37.2, SW59.2, SW76.2, SW93.2
- net ROW0: no longer D15.1 (K)
- net ROW1: no longer D38.1 (K)
- net ROW2: no longer D53.1 (K)
- net ROW3: now also D15.1 (K), D89.1 (K)
- net ROW4: now also D103.1 (K), D38.1 (K); no longer D89.1 (K)
- net ROW5: now also D53.1 (K); no longer D103.1 (K)
- new net: SW104.2, SW105.2, SW18.2, SW34.2, SW56.2, SW90.2
Other:
- note added: "COL 13"
- note added: "COL 14"
- note added: "ROW 3"
- note added: "ROW 4"
- note added: "ROW 5"
- moved on the sheet: D103, D15, D38, D53, D89, SW104, SW16, SW39, SW54, SW90

Commit message: Started work on PCB layout
Slightly Adjusted electric schematic as well.
Parts:
- removed D106, D76, D93: D_Small, symbol Device:D_Small
- removed SW107, SW94: SW_Push, symbol Switch:SW_Push
- removed SW77: PAD_BACK, symbol Switch:SW_Push
- D10, D11, D12, D13, D14, D15, D16, D17, D18, D19, D2, D20, D21, D22, D23, D24, D25, D26, D27, D28, D29, D3, D30, D31, D39, D4, D40, D41, D42, D43, D44, D45, D46, D47, D48, D49, D5, D50, D51, D52, D53, D54, D55, D56, D57, D58, D59, D6, D60, D61, D62, D63, D64, D65, D66, D67, D68, D69, D7, D70, D71, D72, D73, D74, D75, D8, D9: footprint (none) -> Diode_SMD:D_SOD-123
- D100: renamed from D102; footprint (none) -> Diode_SMD:D_SOD-123
- D101: renamed from D103; footprint (none) -> Diode_SMD:D_SOD-123
- D102: renamed from D104; footprint (none) -> Diode_SMD:D_SOD-123
- D103: renamed from D105; footprint (none) -> Diode_SMD:D_SOD-123
- D104: renamed from D107; footprint (none) -> Diode_SMD:D_SOD-123
- D105: renamed from D108; footprint (none) -> Diode_SMD:D_SOD-123
- D32: renamed from D38; footprint (none) -> Diode_SMD:D_SOD-123
- D33: renamed from D32; footprint (none) -> Diode_SMD:D_SOD-123
- D34: renamed from D33; footprint (none) -> Diode_SMD:D_SOD-123
- D35: renamed from D34; footprint (none) -> Diode_SMD:D_SOD-123
- D36: renamed from D35; footprint (none) -> Diode_SMD:D_SOD-123
- D37: renamed from D36; footprint (none) -> Diode_SMD:D_SOD-123
- D38: renamed from D37; footprint (none) -> Diode_SMD:D_SOD-123
- D76: renamed from D77; footprint (none) -> Diode_SMD:D_SOD-123
- D77: renamed from D78; footprint (none) -> Diode_SMD:D_SOD-123
- D78: renamed from D79; footprint (none) -> Diode_SMD:D_SOD-123
- D79: renamed from D80; footprint (none) -> Diode_SMD:D_SOD-123
- D80: renamed from D81; footprint (none) -> Diode_SMD:D_SOD-123
- D81: renamed from D82; footprint (none) -> Diode_SMD:D_SOD-123
- D82: renamed from D83; footprint (none) -> Diode_SMD:D_SOD-123
- D83: renamed from D84; footprint (none) -> Diode_SMD:D_SOD-123
- D84: renamed from D85; footprint (none) -> Diode_SMD:D_SOD-123
- D85: renamed from D86; footprint (none) -> Diode_SMD:D_SOD-123
- D86: renamed from D87; footprint (none) -> Diode_SMD:D_SOD-123
- D87: renamed from D88; footprint (none) -> Diode_SMD:D_SOD-123
- D88: renamed from D89; footprint (none) -> Diode_SMD:D_SOD-123
- D89: renamed from D90; footprint (none) -> Diode_SMD:D_SOD-123
- D90: renamed from D91; footprint (none) -> Diode_SMD:D_SOD-123
- D91: renamed from D92; footprint (none) -> Diode_SMD:D_SOD-123
- D92: renamed from D94; footprint (none) -> Diode_SMD:D_SOD-123
- D93: renamed from D95; footprint (none) -> Diode_SMD:D_SOD-123
- D94: renamed from D96; footprint (none) -> Diode_SMD:D_SOD-123
- D95: renamed from D97; footprint (none) -> Diode_SMD:D_SOD-123
- D96: renamed from D98; footprint (none) -> Diode_SMD:D_SOD-123
- D97: renamed from D99; footprint (none) -> Diode_SMD:D_SOD-123
- D98: renamed from D100; footprint (none) -> Diode_SMD:D_SOD-123
- D99: renamed from D101; footprint (none) -> Diode_SMD:D_SOD-123
- SW10, SW11, SW12, SW13, SW14, SW15, SW16, SW17, SW18, SW19, SW20, SW21, SW22, SW23, SW24, SW25, SW26, SW27, SW28, SW29, SW3, SW30, SW31, SW4, SW41, SW42, SW43, SW44, SW45, SW46, SW47, SW48, SW49, SW5, SW50, SW51, SW52, SW53, SW54, SW55, SW56, SW57, SW58, SW59, SW6, SW60, SW62, SW63, SW64, SW65, SW66, SW67, SW68, SW69, SW7, SW70, SW71, SW72, SW74, SW75, SW76, SW8, SW9: footprint (none) -> Alps_Only:ALPS-1U
- SW100: renamed from SW102; footprint (none) -> Alps_Only:ALPS-1.5U
- SW101: renamed from SW103; footprint (none) -> Alps_Only:ALPS-1U
- SW102: renamed from SW104; footprint (none) -> Alps_Only:ALPS-1U
- SW103: renamed from SW105; footprint (none) -> Alps_Only:ALPS-1U
- SW104: renamed from SW106; footprint (none) -> Alps_Only:ALPS-2.25U-LED
- SW105: renamed from SW108; footprint (none) -> Alps_Only:ALPS-1U
- SW106: renamed from SW109; footprint (none) -> Alps_Only:ALPS-2.25U
- SW32: footprint (none) -> Alps_Only:ALPS-2U
- SW33: renamed from SW39; footprint (none) -> Alps_Only:ALPS-1U
- SW34: renamed from SW33; footprint (none) -> Alps_Only:ALPS-1U
- SW35: renamed from SW34; footprint (none) -> Alps_Only:ALPS-1U
- SW36: renamed from SW35; footprint (none) -> Alps_Only:ALPS-1U
- SW37: renamed from SW36; footprint (none) -> Alps_Only:ALPS-1U
- SW38: renamed from SW37; footprint (none) -> Alps_Only:ALPS-1U
- SW39: renamed from SW38; footprint (none) -> Alps_Only:ALPS-1U
- SW40: footprint (none) -> Alps_Only:ALPS-1.5U
- SW61: footprint (none) -> Alps_Only:ALPS-1.75U
- SW73: footprint (none) -> Alps_Only:ALPS-2.25U
- SW77: renamed from SW78; footprint (none) -> Alps_Only:ALPS-2.25U
- SW78: renamed from SW79; footprint (none) -> Alps_Only:ALPS-1U
- SW79: renamed from SW80; footprint (none) -> Alps_Only:ALPS-1U
- SW80: renamed from SW81; footprint (none) -> Alps_Only:ALPS-1U
- SW81: renamed from SW82; footprint (none) -> Alps_Only:ALPS-1U
- SW82: renamed from SW83; footprint (none) -> Alps_Only:ALPS-1U
- SW83: renamed from SW84; footprint (none) -> Alps_Only:ALPS-1U
- SW84: renamed from SW85; footprint (none) -> Alps_Only:ALPS-1U
- SW85: renamed from SW86; footprint (none) -> Alps_Only:ALPS-1U
- SW86: renamed from SW87; footprint (none) -> Alps_Only:ALPS-1U
- SW87: renamed from SW88; footprint (none) -> Alps_Only:ALPS-1U
- SW88: renamed from SW89; footprint (none) -> Alps_Only:ALPS-2.25U
- SW89: renamed from SW90; footprint (none) -> Alps_Only:ALPS-1U
- SW90: renamed from SW91; footprint (none) -> Alps_Only:ALPS-1U
- SW91: renamed from SW92; footprint (none) -> Alps_Only:ALPS-1U
- SW92: renamed from SW93; footprint (none) -> Alps_Only:ALPS-1U
- SW93: renamed from SW95; footprint (none) -> Alps_Only:ALPS-1.5U
- SW94: renamed from SW96; footprint (none) -> Alps_Only:ALPS-1U
- SW95: renamed from SW97; footprint (none) -> Alps_Only:ALPS-1.25U
- SW96: renamed from SW98; footprint (none) -> Alps_Only:ALPS-6.5U
- SW97: renamed from SW99; footprint (none) -> Alps_Only:ALPS-1.25U
- SW98: renamed from SW100; footprint (none) -> Alps_Only:ALPS-1U
- SW99: renamed from SW101; footprint (none) -> Alps_Only:ALPS-1U
Connections:
- net COL13: no longer SW101.2
- net COL14: now also SW101.2; no longer SW17.2, SW34.2, SW55.2
- net COL15: now also SW102.2, SW17.2, SW34.2, SW55.2, SW89.2
- net COL16: now also SW103.2, SW18.2, SW35.2, SW56.2; no longer SW104.2, SW36.2, SW57.2, SW74.2, SW90.2
- net COL17: now also SW104.2, SW36.2, SW57.2, SW74.2, SW90.2; no longer SW37.2, SW58.2, SW75.2, SW91.2
- net COL18: now also SW37.2, SW58.2, SW75.2, SW91.2; no longer SW59.2, SW76.2, SW92.2
- net COL19: now also SW59.2, SW76.2, SW92.2
- net ROW0: now also D15.1 (K), D37.1 (K), D38.1 (K)
- net ROW1: now also D32.1 (K), D59.1 (K); no longer D37.1 (K), D38.1 (K)
- net ROW2: now also D53.1 (K); no longer D59.1 (K)
- net ROW3: no longer D15.1 (K), D88.1 (K)
- net ROW4: now also D88.1 (K); no longer D101.1 (K), D32.1 (K)
- net ROW5: now also D101.1 (K); no longer D53.1 (K)
Other:
- note removed: "COL 13"
- note removed: "COL 14"
- note removed: "ROW 3"
- note removed: "ROW 4"
- note removed: "ROW 5"
- moved on the sheet: D101, D104, D15, D32, D37, D38, D53, D59, D88, SW102, SW105, SW16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

Commit message: Changing hotswap switches
Reverse Mount leds not added yet.
Parts:
- SW10, SW101, SW102, SW103, SW105, SW11, SW12, SW13, SW14, SW15, SW16, SW17, SW18, SW19, SW20, SW21, SW22, SW23, SW24, SW25, SW26, SW27, SW28, SW29, SW3, SW30, SW31, SW33, SW34, SW35, SW36, SW37, SW38, SW39, SW4, SW41, SW42, SW43, SW44, SW45, SW46, SW47, SW48, SW49, SW5, SW50, SW51, SW52, SW53, SW54, SW55, SW56, SW57, SW58, SW59, SW6, SW60, SW62, SW63, SW64, SW65, SW66, SW67, SW68, SW69, SW7, SW70, SW71, SW72, SW74, SW75, SW76, SW78, SW79, SW8, SW80, SW81, SW82, SW83, SW84, SW85, SW86, SW87, SW89, SW9, SW90, SW91, SW92, SW94, SW98, SW99: footprint Alps_Only:ALPS-1U -> MX_Only:MXOnly-1U-Hotswap
- SW100, SW40, SW93: footprint Alps_Only:ALPS-1.5U -> MX_Only:MXOnly-1.5U-Hotswap
- SW104: footprint Alps_Only:ALPS-2.25U-LED -> MX_Only:MXOnly-2.25U-Hotswap
- SW106, SW73, SW77, SW88: footprint Alps_Only:ALPS-2.25U -> MX_Only:MXOnly-2.25U-Hotswap
- SW32: footprint Alps_Only:ALPS-2U -> MX_Only:MXOnly-2U-Hotswap
- SW61: footprint Alps_Only:ALPS-1.75U -> MX_Only:MXOnly-1.75U-Hotswap
- SW95, SW97: footprint Alps_Only:ALPS-1.25U -> MX_Only:MXOnly-1.25U-Hotswap
- SW96: footprint Alps_Only:ALPS-6.5U -> MX_Only:MXOnly-6.25U-Hotswap

Commit message: Changed to reverse mount rgb leds
Both symbol and footprint were changed accordingly.
Parts:
- SW100, SW93: footprint MX_Only:MXOnly-1.5U-Hotswap -> MX_Only:MXOnly-1.25U-Hotswap
- SW104, SW106: footprint MX_Only:MXOnly-2.25U-Hotswap -> MX_Only:MXOnly-2U-Hotswap
- SW53: footprint MX_Only:MXOnly-1U-Hotswap -> MX_Only:MXOnly-1.5U-Hotswap
- SW60: footprint MX_Only:MXOnly-1U-Hotswap -> MX_Only:MXOnly-2U-Hotswap
- SW88: footprint MX_Only:MXOnly-2.25U-Hotswap -> MX_Only:MXOnly-2.75U-Hotswap
- SW94, SW98, SW99: footprint MX_Only:MXOnly-1U-Hotswap -> MX_Only:MXOnly-1.25U-Hotswap
Changed lines of the file:
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@@
       (effects (font (size 1.27 1.27)))
     )
-    (property "Footprint" "MX_Only:MXOnly-2.25U-Hotswap" (at 248.666 110.998 0)
+    (property "Footprint" "MX_Only:MXOnly-2.75U-Hotswap" (at 248.666 110.998 0)
       (effects (font (size 1.27 1.27)) hide)
     )
@@
       (effects (font (size 1.27 1.27)))
     )
-    (property "Footprint" "MX_Only:MXOnly-1.5U-Hotswap" (at 36.576 129.032 0)
+    (property "Footprint" "MX_Only:MXOnly-1.25U-Hotswap" (at 36.576 129.032 0)
       (effects (font (size 1.27 1.27)) hide)
     )
@@
       (effects (font (size 1.27 1.27)))
     )
-    (property "Footprint" "MX_Only:MXOnly-2.25U-Hotswap" (at 394.208 129.032 0)
+    (property "Footprint" "MX_Only:MXOnly-2U-Hotswap" (at 394.208 129.032 0)
       (effects (font (size 1.27 1.27)) hide)
     )
@@
       (effects (font (size 1.27 1.27)))
     )
-    (property "Footprint" "MX_Only:MXOnly-1U-Hotswap" (at 247.904 74.93 0)
+    (property "Footprint" "MX_Only:MXOnly-1.5U-Hotswap" (at 247.904 74.93 0)
       (effects (font (size 1.27 1.27)) hide)
     )
@@
       (effects (font (size 1.27 1.27)))
     )
-    (property "Footprint" "MX_Only:MXOnly-2.25U-Hotswap" (at 345.44 129.032 0)
+    (property "Footprint" "MX_Only:MXOnly-2U-Hotswap" (at 345.44 129.032 0)
       (effects (font (size 1.27 1.27)) hide)
     )
@@
       (effects (font (size 1.27 1.27)))
     )
-    (property "Footprint" "MX_Only:MXOnly-1U-Hotswap" (at 394.208 74.93 0)
+    (property "Footprint" "MX_Only:MXOnly-2U-Hotswap" (at 394.208 74.93 0)
       (effects (font (size 1.27 1.27)) hide)
     )
@@
       (effects (font (size 1.27 1.27)))
     )
-    (property "Footprint" "MX_Only:MXOnly-1U-Hotswap" (at 182.88 129.032 0)
+    (property "Footprint" "MX_Only:MXOnly-1.25U-Hotswap" (at 182.88 129.032 0)
       (effects (font (size 1.27 1.27)) hide)
     )
@@
       (effects (font (size 1.27 1.27)))
     )
-    (property "Footprint" "MX_Only:MXOnly-1U-Hotswap" (at 52.832 129.032 0)
+    (property "Footprint" "MX_Only:MXOnly-1.25U-Hotswap" (at 52.832 129.032 0)
       (effects (font (size 1.27 1.27)) hide)
     )
@@
       (effects (font (size 1.27 1.27)))
     )
-    (property "Footprint" "MX_Only:MXOnly-1U-Hotswap" (at 199.136 129.032 0)
+    (property "Footprint" "MX_Only:MXOnly-1.25U-Hotswap" (at 199.136 129.032 0)
       (effects (font (size 1.27 1.27)) hide)
     )
@@
       (effects (font (size 1.27 1.27)))
     )
-    (property "Footprint" "MX_Only:MXOnly-1.5U-Hotswap" (at 215.392 129.032 0)
+    (property "Footprint" "MX_Only:MXOnly-1.25U-Hotswap" (at 215.392 129.032 0)
       (effects (font (size 1.27 1.27)) hide)
     )
