File: matrix.kicad_sch (KiCad schematic)
At the start: 208 parts, among them SW10 F7, SW100 R_CTRL, SW101 L_ARROW, SW102 DN_ARROW, SW103 R_ARROW, SW104 PAD_0, SW105 PAD_., SW106 PAD_ENTER, SW11 F8, SW12 F9, SW13 F10, SW14 F11, SW15 F12, SW16 PRT_SC, SW17 SCR_LK, SW18 PAUSE, SW19 TILDE, SW20 1, SW21 2, SW22 3, SW23 4, SW24 5, SW25 6, SW26 7, SW27 8, SW28 9, SW29 0, SW3 ESC, SW30 -, SW31 =, SW32 BACKSPACE, SW33 INSERT, SW34 HOME, SW35 PG_UP, SW36 NUM_LK, SW37 PAD_/, SW38 *, SW39 PAD_-, SW4 F1, SW40 TAB, SW41 Q, SW42 W, SW43 E, SW44 R, SW45 T, SW46 Y, SW47 U, SW48 I, SW49 O, SW5 F2, SW50 P, SW51 [, SW52 ], SW53 \, SW54 DEL, SW55 END, SW56 PG_DN, SW57 PAD_7, SW58 PAD_8, SW59 PAD_9, SW6 F3, SW60 +, SW61 CAPS, SW62 A, SW63 S, SW64 D, SW65 F, SW66 G, SW67 H, SW68 J, SW69 K, SW7 F4, SW70 L, SW71 ;, SW72 ', SW73 ENTER, SW74 PAD_4, SW75 PAD_5, SW76 PAD_6, SW77 L_SHIFT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

Commit message: Revising for underglow and PD IC
Connections:
- net COL19 is gone; now on net COL18: SW106.2, SW39.2, SW59.2, SW60.2, SW76.2, SW92.2
- net COL14: now also SW102.2, SW89.2
- net COL15: no longer SW102.2, SW89.2
- net COL16: now also SW104.2, SW36.2, SW57.2, SW74.2, SW90.2; no longer SW103.2, SW35.2, SW56.2
- net COL17: now also SW105.2, SW37.2, SW38.2, SW58.2, SW75.2, SW91.2; no longer SW104.2, SW36.2, SW57.2, SW74.2, SW90.2
- net COL18: no longer SW105.2, SW37.2, SW38.2, SW58.2, SW75.2, SW91.2
- net ROW1: no longer D34.1 (K)
- net ROW2: now also D34.1 (K); no longer D54.1 (K), D55.1 (K)
- net ROW3: now also D54.1 (K), D88.1 (K)
- net ROW4: now also D101.1 (K), D55.1 (K); no longer D88.1 (K)
- net ROW5: no longer D101.1 (K)
- new net: SW103.2, SW35.2, SW56.2
Other:
- moved on the sheet: D10, D100, D101, D102, D103, D104, D105, D11, D12, D13, D14, D15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
