File: matrix.kicad_sch (KiCad schematic)
At the start: 208 parts, among them SW10 F7, SW100 R_CTRL, SW101 L_ARROW, SW102 DN_ARROW, SW103 R_ARROW, SW104 PAD_0, SW105 PAD_., SW106 PAD_ENTER, SW11 F8, SW12 F9, SW13 F10, SW14 F11, SW15 F12, SW16 PRT_SC, SW17 SCR_LK, SW18 PAUSE, SW19 TILDE, SW20 1, SW21 2, SW22 3, SW23 4, SW24 5, SW25 6, SW26 7, SW27 8, SW28 9, SW29 0, SW3 ESC, SW30 -, SW31 =, SW32 BACKSPACE, SW33 INSERT, SW34 HOME, SW35 PG_UP, SW36 NUM_LK, SW37 PAD_/, SW38 *, SW39 PAD_-, SW4 F1, SW40 TAB, SW41 Q, SW42 W, SW43 E, SW44 R, SW45 T, SW46 Y, SW47 U, SW48 I, SW49 O, SW5 F2, SW50 P, SW51 [, SW52 ], SW53 \, SW54 DEL, SW55 END, SW56 PG_DN, SW57 PAD_7, SW58 PAD_8, SW59 PAD_9, SW6 F3, SW60 +, SW61 CAPS, SW62 A, SW63 S, SW64 D, SW65 F, SW66 G, SW67 H, SW68 J, SW69 K, SW7 F4, SW70 L, SW71 ;, SW72 ', SW73 ENTER, SW74 PAD_4, SW75 PAD_5, SW76 PAD_6, SW77 L_SHIFT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

Commit message: Rearranged LED Drivers
Connections:
- net COL15: now also SW103.2, SW35.2, SW56.2
Changed lines of the file:
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@@
   (junction (at 367.284 116.967) (diameter 0) (color 0 0 0 0)
   )
+  (junction (at 302.26 53.6101) (diameter 0) (color 0 0 0 0)
+  )
   (junction (at 96.266 67.945) (diameter 0) (color 0 0 0 0)
   )
@@
   (junction (at 286.004 62.865) (diameter 0) (color 0 0 0 0)
   )
+  (junction (at 318.427 62.865) (diameter 0) (color 0 0 0 0)
+  )
   (junction (at 351.028 98.933) (diameter 0) (color 0 0 0 0)
   )
@@
     (stroke (width 0) (type default))
   )
-  (wire (pts (xy 317.754 62.865) (xy 318.516 62.865))
+  (wire (pts (xy 317.754 62.865) (xy 318.427 62.865))
     (stroke (width 0) (type default))
   )
@@
     (stroke (width 0) (type default))
   )
-  (wire (pts (xy 302.26 44.831) (xy 302.26 62.865))
+  (wire (pts (xy 302.26 44.831) (xy 302.26 53.6101))
     (stroke (width 0) (type default))
   )
@@
     (stroke (width 0) (type default))
   )
+  (wire (pts (xy 318.427 62.865) (xy 318.516 62.865))
+    (stroke (width 0) (type default))
+  )
   (wire (pts (xy 80.01 122.047) (xy 96.266 122.047))
     (stroke (width 0) (type default))
@@
     (stroke (width 0) (type default))
   )
+  (wire (pts (xy 302.26 53.6101) (xy 302.26 62.865))
+    (stroke (width 0) (type default))
+  )
   (wire (pts (xy 145.034 49.911) (xy 161.29 49.911))
     (stroke (width 0) (type default))
@@
     (stroke (width 0) (type default))
   )
+  (wire (pts (xy 318.427 62.865) (xy 318.427 53.6101))
+    (stroke (width 0) (type default))
+  )
   (wire (pts (xy 122.682 98.933) (xy 123.444 98.933))
     (stroke (width 0) (type default))
@@
     (stroke (width 0) (type default))
   )
+  (wire (pts (xy 318.427 53.6101) (xy 302.26 53.6101))
+    (stroke (width 0) (type default))
+  )
