File: rgbMatrix.kicad_sch (KiCad schematic)
At the start: 166 parts

Commit message: Changed to reverse mount rgb leds
Both symbol and footprint were changed accordingly.
Parts:
- removed LED1: ESC, mouser_AAA3528SEEZGKQBKS:AAA3528SEEZGKQBKS, symbol AAA3528SEEZGKQBKS:AAA3528SEEZGKQBKS
- removed LED10: F9, mouser_AAA3528SEEZGKQBKS:AAA3528SEEZGKQBKS, symbol AAA3528SEEZGKQBKS:AAA3528SEEZGKQBKS
- removed LED100: R_CTRL, mouser_AAA3528SEEZGKQBKS:AAA3528SEEZGKQBKS, symbol AAA3528SEEZGKQBKS:AAA3528SEEZGKQBKS
- removed LED101: L_ARROW, mouser_AAA3528SEEZGKQBKS:AAA3528SEEZGKQBKS, symbol AAA3528SEEZGKQBKS:AAA3528SEEZGKQBKS
- removed LED102: DN_ARROW, mouser_AAA3528SEEZGKQBKS:AAA3528SEEZGKQBKS, symbol AAA3528SEEZGKQBKS:AAA3528SEEZGKQBKS
- removed LED103: R_ARROW, mouser_AAA3528SEEZGKQBKS:AAA3528SEEZGKQBKS, symbol AAA3528SEEZGKQBKS:AAA3528SEEZGKQBKS
- removed LED104: PAD_0, mouser_AAA3528SEEZGKQBKS:AAA3528SEEZGKQBKS, symbol AAA3528SEEZGKQBKS:AAA3528SEEZGKQBKS
- removed LED105: PAD_., mouser_AAA3528SEEZGKQBKS:AAA3528SEEZGKQBKS, symbol AAA3528SEEZGKQBKS:AAA3528SEEZGKQBKS
- removed LED106: PAD_ENTER, mouser_AAA3528SEEZGKQBKS:AAA3528SEEZGKQBKS, symbol AAA3528SEEZGKQBKS:AAA3528SEEZGKQBKS
- removed LED11: F10, mouser_AAA3528SEEZGKQBKS:AAA3528SEEZGKQBKS, symbol AAA3528SEEZGKQBKS:AAA3528SEEZGKQBKS
- removed LED12: F11, mouser_AAA3528SEEZGKQBKS:AAA3528SEEZGKQBKS, symbol AAA3528SEEZGKQBKS:AAA3528SEEZGKQBKS
- removed LED13: F12, mouser_AAA3528SEEZGKQBKS:AAA3528SEEZGKQBKS, symbol AAA3528SEEZGKQBKS:AAA3528SEEZGKQBKS
- removed LED14: PRT_SC, mouser_AAA3528SEEZGKQBKS:AAA3528SEEZGKQBKS, symbol AAA3528SEEZGKQBKS:AAA3528SEEZGKQBKS
- removed LED15: SCR_LK, mouser_AAA3528SEEZGKQBKS:AAA3528SEEZGKQBKS, symbol AAA3528SEEZGKQBKS:AAA3528SEEZGKQBKS
- removed LED16: PAUSE, mouser_AAA3528SEEZGKQBKS:AAA3528SEEZGKQBKS, symbol AAA3528SEEZGKQBKS:AAA3528SEEZGKQBKS
- removed LED17: TILDE, mouser_AAA3528SEEZGKQBKS:AAA3528SEEZGKQBKS, symbol AAA3528SEEZGKQBKS:AAA3528SEEZGKQBKS
- removed LED18: 1, mouser_AAA3528SEEZGKQBKS:AAA3528SEEZGKQBKS, symbol AAA3528SEEZGKQBKS:AAA3528SEEZGKQBKS
- removed LED19: 2, mouser_AAA3528SEEZGKQBKS:AAA3528SEEZGKQBKS, symbol AAA3528SEEZGKQBKS:AAA3528SEEZGKQBKS
- removed LED2: F1, mouser_AAA3528SEEZGKQBKS:AAA3528SEEZGKQBKS, symbol AAA3528SEEZGKQBKS:AAA3528SEEZGKQBKS
- removed LED20: 3, mouser_AAA3528SEEZGKQBKS:AAA3528SEEZGKQBKS, symbol AAA3528SEEZGKQBKS:AAA3528SEEZGKQBKS
- removed LED21: 4, mouser_AAA3528SEEZGKQBKS:AAA3528SEEZGKQBKS, symbol AAA3528SEEZGKQBKS:AAA3528SEEZGKQBKS
- removed LED22: 5, mouser_AAA3528SEEZGKQBKS:AAA3528SEEZGKQBKS, symbol AAA3528SEEZGKQBKS:AAA3528SEEZGKQBKS
- removed LED23: 6, mouser_AAA3528SEEZGKQBKS:AAA3528SEEZGKQBKS, symbol AAA3528SEEZGKQBKS:AAA3528SEEZGKQBKS
- removed LED24: 7, mouser_AAA3528SEEZGKQBKS:AAA3528SEEZGKQBKS, symbol AAA3528SEEZGKQBKS:AAA3528SEEZGKQBKS
- removed LED25: 8, mouser_AAA3528SEEZGKQBKS:AAA3528SEEZGKQBKS, symbol AAA3528SEEZGKQBKS:AAA3528SEEZGKQBKS
- removed LED26: 9, mouser_AAA3528SEEZGKQBKS:AAA3528SEEZGKQBKS, symbol AAA3528SEEZGKQBKS:AAA3528SEEZGKQBKS
- removed LED27: 0, mouser_AAA3528SEEZGKQBKS:AAA3528SEEZGKQBKS, symbol AAA3528SEEZGKQBKS:AAA3528SEEZGKQBKS
- removed LED28: -, mouser_AAA3528SEEZGKQBKS:AAA3528SEEZGKQBKS, symbol AAA3528SEEZGKQBKS:AAA3528SEEZGKQBKS
- removed LED29: =, mouser_AAA3528SEEZGKQBKS:AAA3528SEEZGKQBKS, symbol AAA3528SEEZGKQBKS:AAA3528SEEZGKQBKS
- removed LED3: F2, mouser_AAA3528SEEZGKQBKS:AAA3528SEEZGKQBKS, symbol AAA3528SEEZGKQBKS:AAA3528SEEZGKQBKS
- removed LED30: BACKSPACE, mouser_AAA3528SEEZGKQBKS:AAA3528SEEZGKQBKS, symbol AAA3528SEEZGKQBKS:AAA3528SEEZGKQBKS
- removed LED31: INSERT, mouser_AAA3528SEEZGKQBKS:AAA3528SEEZGKQBKS, symbol AAA3528SEEZGKQBKS:AAA3528SEEZGKQBKS
- removed LED32: HOME, mouser_AAA3528SEEZGKQBKS:AAA3528SEEZGKQBKS, symbol AAA3528SEEZGKQBKS:AAA3528SEEZGKQBKS
- removed LED33: PG_UP, mouser_AAA3528SEEZGKQBKS:AAA3528SEEZGKQBKS, symbol AAA3528SEEZGKQBKS:AAA3528SEEZGKQBKS
- removed LED34: NUM_LK, mouser_AAA3528SEEZGKQBKS:AAA3528SEEZGKQBKS, symbol AAA3528SEEZGKQBKS:AAA3528SEEZGKQBKS
- removed LED35: PAD_/, mouser_AAA3528SEEZGKQBKS:AAA3528SEEZGKQBKS, symbol AAA3528SEEZGKQBKS:AAA3528SEEZGKQBKS
- removed LED36: *, mouser_AAA3528SEEZGKQBKS:AAA3528SEEZGKQBKS, symbol AAA3528SEEZGKQBKS:AAA3528SEEZGKQBKS
- removed LED37: PAD_-, mouser_AAA3528SEEZGKQBKS:AAA3528SEEZGKQBKS, symbol AAA3528SEEZGKQBKS:AAA3528SEEZGKQBKS
- removed LED38: TAB, mouser_AAA3528SEEZGKQBKS:AAA3528SEEZGKQBKS, symbol AAA3528SEEZGKQBKS:AAA3528SEEZGKQBKS
- removed LED39: Q, mouser_AAA3528SEEZGKQBKS:AAA3528SEEZGKQBKS, symbol AAA3528SEEZGKQBKS:AAA3528SEEZGKQBKS
- removed LED4: F3, mouser_AAA3528SEEZGKQBKS:AAA3528SEEZGKQBKS, symbol AAA3528SEEZGKQBKS:AAA3528SEEZGKQBKS
- removed LED40: W, mouser_AAA3528SEEZGKQBKS:AAA3528SEEZGKQBKS, symbol AAA3528SEEZGKQBKS:AAA3528SEEZGKQBKS
- removed LED41: E, mouser_AAA3528SEEZGKQBKS:AAA3528SEEZGKQBKS, symbol AAA3528SEEZGKQBKS:AAA3528SEEZGKQBKS
- removed LED42: R, mouser_AAA3528SEEZGKQBKS:AAA3528SEEZGKQBKS, symbol AAA3528SEEZGKQBKS:AAA3528SEEZGKQBKS
- removed LED43: T, mouser_AAA3528SEEZGKQBKS:AAA3528SEEZGKQBKS, symbol AAA3528SEEZGKQBKS:AAA3528SEEZGKQBKS
- removed LED44: Y, mouser_AAA3528SEEZGKQBKS:AAA3528SEEZGKQBKS, symbol AAA3528SEEZGKQBKS:AAA3528SEEZGKQBKS
- removed LED45: U, mouser_AAA3528SEEZGKQBKS:AAA3528SEEZGKQBKS, symbol AAA3528SEEZGKQBKS:AAA3528SEEZGKQBKS
- removed LED46: I, mouser_AAA3528SEEZGKQBKS:AAA3528SEEZGKQBKS, symbol AAA3528SEEZGKQBKS:AAA3528SEEZGKQBKS
- removed LED47: O, mouser_AAA3528SEEZGKQBKS:AAA3528SEEZGKQBKS, symbol AAA3528SEEZGKQBKS:AAA3528SEEZGKQBKS
- removed LED48: P, mouser_AAA3528SEEZGKQBKS:AAA3528SEEZGKQBKS, symbol AAA3528SEEZGKQBKS:AAA3528SEEZGKQBKS
- removed LED49: [, mouser_AAA3528SEEZGKQBKS:AAA3528SEEZGKQBKS, symbol AAA3528SEEZGKQBKS:AAA3528SEEZGKQBKS
- removed LED5: F4, mouser_AAA3528SEEZGKQBKS:AAA3528SEEZGKQBKS, symbol AAA3528SEEZGKQBKS:AAA3528SEEZGKQBKS
- removed LED50: ], mouser_AAA3528SEEZGKQBKS:AAA3528SEEZGKQBKS, symbol AAA3528SEEZGKQBKS:AAA3528SEEZGKQBKS
- removed LED51: \, mouser_AAA3528SEEZGKQBKS:AAA3528SEEZGKQBKS, symbol AAA3528SEEZGKQBKS:AAA3528SEEZGKQBKS
- removed LED52: DEL, mouser_AAA3528SEEZGKQBKS:AAA3528SEEZGKQBKS, symbol AAA3528SEEZGKQBKS:AAA3528SEEZGKQBKS
- removed LED53: END, mouser_AAA3528SEEZGKQBKS:AAA3528SEEZGKQBKS, symbol AAA3528SEEZGKQBKS:AAA3528SEEZGKQBKS
- removed LED54: PG_DN, mouser_AAA3528SEEZGKQBKS:AAA3528SEEZGKQBKS, symbol AAA3528SEEZGKQBKS:AAA3528SEEZGKQBKS
- removed LED55: PAD_7, mouser_AAA3528SEEZGKQBKS:AAA3528SEEZGKQBKS, symbol AAA3528SEEZGKQBKS:AAA3528SEEZGKQBKS
- removed LED56: PAD_8, mouser_AAA3528SEEZGKQBKS:AAA3528SEEZGKQBKS, symbol AAA3528SEEZGKQBKS:AAA3528SEEZGKQBKS
- removed LED57: PAD_9, mouser_AAA3528SEEZGKQBKS:AAA3528SEEZGKQBKS, symbol AAA3528SEEZGKQBKS:AAA3528SEEZGKQBKS
- removed LED58: +, mouser_AAA3528SEEZGKQBKS:AAA3528SEEZGKQBKS, symbol AAA3528SEEZGKQBKS:AAA3528SEEZGKQBKS
- removed LED59: CAPS, mouser_AAA3528SEEZGKQBKS:AAA3528SEEZGKQBKS, symbol AAA3528SEEZGKQBKS:AAA3528SEEZGKQBKS
- removed LED6: F5, mouser_AAA3528SEEZGKQBKS:AAA3528SEEZGKQBKS, symbol AAA3528SEEZGKQBKS:AAA3528SEEZGKQBKS
- removed LED60: A, mouser_AAA3528SEEZGKQBKS:AAA3528SEEZGKQBKS, symbol AAA3528SEEZGKQBKS:AAA3528SEEZGKQBKS
- removed LED61: S, mouser_AAA3528SEEZGKQBKS:AAA3528SEEZGKQBKS, symbol AAA3528SEEZGKQBKS:AAA3528SEEZGKQBKS
- removed LED62: D, mouser_AAA3528SEEZGKQBKS:AAA3528SEEZGKQBKS, symbol AAA3528SEEZGKQBKS:AAA3528SEEZGKQBKS
- removed LED63: F, mouser_AAA3528SEEZGKQBKS:AAA3528SEEZGKQBKS, symbol AAA3528SEEZGKQBKS:AAA3528SEEZGKQBKS
- removed LED64: G, mouser_AAA3528SEEZGKQBKS:AAA3528SEEZGKQBKS, symbol AAA3528SEEZGKQBKS:AAA3528SEEZGKQBKS
- removed LED65: H, mouser_AAA3528SEEZGKQBKS:AAA3528SEEZGKQBKS, symbol AAA3528SEEZGKQBKS:AAA3528SEEZGKQBKS
- removed LED66: J, mouser_AAA3528SEEZGKQBKS:AAA3528SEEZGKQBKS, symbol AAA3528SEEZGKQBKS:AAA3528SEEZGKQBKS
- removed LED67: K, mouser_AAA3528SEEZGKQBKS:AAA3528SEEZGKQBKS, symbol AAA3528SEEZGKQBKS:AAA3528SEEZGKQBKS
- removed LED68: L, mouser_AAA3528SEEZGKQBKS:AAA3528SEEZGKQBKS, symbol AAA3528SEEZGKQBKS:AAA3528SEEZGKQBKS
- removed LED69: ;, mouser_AAA3528SEEZGKQBKS:AAA3528SEEZGKQBKS, symbol AAA3528SEEZGKQBKS:AAA3528SEEZGKQBKS
- removed LED7: F6, mouser_AAA3528SEEZGKQBKS:AAA3528SEEZGKQBKS, symbol AAA3528SEEZGKQBKS:AAA3528SEEZGKQBKS
- removed LED70: ', mouser_AAA3528SEEZGKQBKS:AAA3528SEEZGKQBKS, symbol AAA3528SEEZGKQBKS:AAA3528SEEZGKQBKS
- removed LED71: ENTER, mouser_AAA3528SEEZGKQBKS:AAA3528SEEZGKQBKS, symbol AAA3528SEEZGKQBKS:AAA3528SEEZGKQBKS
- removed LED72: PAD_4, mouser_AAA3528SEEZGKQBKS:AAA3528SEEZGKQBKS, symbol AAA3528SEEZGKQBKS:AAA3528SEEZGKQBKS
- removed LED73: PAD_5, mouser_AAA3528SEEZGKQBKS:AAA3528SEEZGKQBKS, symbol AAA3528SEEZGKQBKS:AAA3528SEEZGKQBKS
- removed LED74: PAD_6, mouser_AAA3528SEEZGKQBKS:AAA3528SEEZGKQBKS, symbol AAA3528SEEZGKQBKS:AAA3528SEEZGKQBKS
- removed LED75: L_SHIFT, mouser_AAA3528SEEZGKQBKS:AAA3528SEEZGKQBKS, symbol AAA3528SEEZGKQBKS:AAA3528SEEZGKQBKS
- removed LED76: Z, mouser_AAA3528SEEZGKQBKS:AAA3528SEEZGKQBKS, symbol AAA3528SEEZGKQBKS:AAA3528SEEZGKQBKS
- removed LED77: X, mouser_AAA3528SEEZGKQBKS:AAA3528SEEZGKQBKS, symbol AAA3528SEEZGKQBKS:AAA3528SEEZGKQBKS
- removed LED78: C, mouser_AAA3528SEEZGKQBKS:AAA3528SEEZGKQBKS, symbol AAA3528SEEZGKQBKS:AAA3528SEEZGKQBKS
- removed LED79: V, mouser_AAA3528SEEZGKQBKS:AAA3528SEEZGKQBKS, symbol AAA3528SEEZGKQBKS:AAA3528SEEZGKQBKS
- removed LED8: F7, mouser_AAA3528SEEZGKQBKS:AAA3528SEEZGKQBKS, symbol AAA3528SEEZGKQBKS:AAA3528SEEZGKQBKS
- removed LED80: B, mouser_AAA3528SEEZGKQBKS:AAA3528SEEZGKQBKS, symbol AAA3528SEEZGKQBKS:AAA3528SEEZGKQBKS
- removed LED81: N, mouser_AAA3528SEEZGKQBKS:AAA3528SEEZGKQBKS, symbol AAA3528SEEZGKQBKS:AAA3528SEEZGKQBKS
- removed LED82: M, mouser_AAA3528SEEZGKQBKS:AAA3528SEEZGKQBKS, symbol AAA3528SEEZGKQBKS:AAA3528SEEZGKQBKS
- removed LED83: ,, mouser_AAA3528SEEZGKQBKS:AAA3528SEEZGKQBKS, symbol AAA3528SEEZGKQBKS:AAA3528SEEZGKQBKS
- removed LED84: ., mouser_AAA3528SEEZGKQBKS:AAA3528SEEZGKQBKS, symbol AAA3528SEEZGKQBKS:AAA3528SEEZGKQBKS
- removed LED85: /, mouser_AAA3528SEEZGKQBKS:AAA3528SEEZGKQBKS, symbol AAA3528SEEZGKQBKS:AAA3528SEEZGKQBKS
- removed LED86: R_SHIFT, mouser_AAA3528SEEZGKQBKS:AAA3528SEEZGKQBKS, symbol AAA3528SEEZGKQBKS:AAA3528SEEZGKQBKS
- removed LED87: UP_ARROW, mouser_AAA3528SEEZGKQBKS:AAA3528SEEZGKQBKS, symbol AAA3528SEEZGKQBKS:AAA3528SEEZGKQBKS
- removed LED88: PAD_1, mouser_AAA3528SEEZGKQBKS:AAA3528SEEZGKQBKS, symbol AAA3528SEEZGKQBKS:AAA3528SEEZGKQBKS
- removed LED89: PAD_2, mouser_AAA3528SEEZGKQBKS:AAA3528SEEZGKQBKS, symbol AAA3528SEEZGKQBKS:AAA3528SEEZGKQBKS
- removed LED9: F8, mouser_AAA3528SEEZGKQBKS:AAA3528SEEZGKQBKS, symbol AAA3528SEEZGKQBKS:AAA3528SEEZGKQBKS
- removed LED90: PAD_3, mouser_AAA3528SEEZGKQBKS:AAA3528SEEZGKQBKS, symbol AAA3528SEEZGKQBKS:AAA3528SEEZGKQBKS
- removed LED91: CTRL, mouser_AAA3528SEEZGKQBKS:AAA3528SEEZGKQBKS, symbol AAA3528SEEZGKQBKS:AAA3528SEEZGKQBKS
- removed LED92: OS, mouser_AAA3528SEEZGKQBKS:AAA3528SEEZGKQBKS, symbol AAA3528SEEZGKQBKS:AAA3528SEEZGKQBKS
- removed LED93: L_ALT, mouser_AAA3528SEEZGKQBKS:AAA3528SEEZGKQBKS, symbol AAA3528SEEZGKQBKS:AAA3528SEEZGKQBKS
- removed LED94: SPACE_L, mouser_AAA3528SEEZGKQBKS:AAA3528SEEZGKQBKS, symbol AAA3528SEEZGKQBKS:AAA3528SEEZGKQBKS
- removed LED95: SPACE, mouser_AAA3528SEEZGKQBKS:AAA3528SEEZGKQBKS, symbol AAA3528SEEZGKQBKS:AAA3528SEEZGKQBKS
- removed LED96: SPACE_R, mouser_AAA3528SEEZGKQBKS:AAA3528SEEZGKQBKS, symbol AAA3528SEEZGKQBKS:AAA3528SEEZGKQBKS
- removed LED97: R_ALT, mouser_AAA3528SEEZGKQBKS:AAA3528SEEZGKQBKS, symbol AAA3528SEEZGKQBKS:AAA3528SEEZGKQBKS
- removed LED98: FN, mouser_AAA3528SEEZGKQBKS:AAA3528SEEZGKQBKS, symbol AAA3528SEEZGKQBKS:AAA3528SEEZGKQBKS
- removed LED99: MENU, mouser_AAA3528SEEZGKQBKS:AAA3528SEEZGKQBKS, symbol AAA3528SEEZGKQBKS:AAA3528SEEZGKQBKS
- added LED1: ESC, XZMDKCBDDG45S-9:PLCC4_SMD-LED_3p2X2p8_SLD, symbol XZMDKCBDDG45S-9:XZMDKCBDDG45S-9
- added LED10: TILDE, XZMDKCBDDG45S-9:PLCC4_SMD-LED_3p2X2p8_SLD, symbol XZMDKCBDDG45S-9:XZMDKCBDDG45S-9
- added LED100: R_CTRL, XZMDKCBDDG45S-9:PLCC4_SMD-LED_3p2X2p8_SLD, symbol XZMDKCBDDG45S-9:XZMDKCBDDG45S-9
- added LED101: L_ARROW, XZMDKCBDDG45S-9:PLCC4_SMD-LED_3p2X2p8_SLD, symbol XZMDKCBDDG45S-9:XZMDKCBDDG45S-9
- added LED102: D_ARROW, XZMDKCBDDG45S-9:PLCC4_SMD-LED_3p2X2p8_SLD, symbol XZMDKCBDDG45S-9:XZMDKCBDDG45S-9
- added LED103: R_ARROW, XZMDKCBDDG45S-9:PLCC4_SMD-LED_3p2X2p8_SLD, symbol XZMDKCBDDG45S-9:XZMDKCBDDG45S-9
- added LED104: PAD_0, XZMDKCBDDG45S-9:PLCC4_SMD-LED_3p2X2p8_SLD, symbol XZMDKCBDDG45S-9:XZMDKCBDDG45S-9
- added LED105: PAD_., XZMDKCBDDG45S-9:PLCC4_SMD-LED_3p2X2p8_SLD, symbol XZMDKCBDDG45S-9:XZMDKCBDDG45S-9
- added LED106: PAD_ENTER, XZMDKCBDDG45S-9:PLCC4_SMD-LED_3p2X2p8_SLD, symbol XZMDKCBDDG45S-9:XZMDKCBDDG45S-9
- added LED107: MENU, XZMDKCBDDG45S-9:PLCC4_SMD-LED_3p2X2p8_SLD, symbol XZMDKCBDDG45S-9:XZMDKCBDDG45S-9
- added LED11: 1, XZMDKCBDDG45S-9:PLCC4_SMD-LED_3p2X2p8_SLD, symbol XZMDKCBDDG45S-9:XZMDKCBDDG45S-9
- added LED12: 2, XZMDKCBDDG45S-9:PLCC4_SMD-LED_3p2X2p8_SLD, symbol XZMDKCBDDG45S-9:XZMDKCBDDG45S-9
- added LED13: 3, XZMDKCBDDG45S-9:PLCC4_SMD-LED_3p2X2p8_SLD, symbol XZMDKCBDDG45S-9:XZMDKCBDDG45S-9
- added LED14: 4, XZMDKCBDDG45S-9:PLCC4_SMD-LED_3p2X2p8_SLD, symbol XZMDKCBDDG45S-9:XZMDKCBDDG45S-9
- added LED15: 5, XZMDKCBDDG45S-9:PLCC4_SMD-LED_3p2X2p8_SLD, symbol XZMDKCBDDG45S-9:XZMDKCBDDG45S-9
- added LED16: 6, XZMDKCBDDG45S-9:PLCC4_SMD-LED_3p2X2p8_SLD, symbol XZMDKCBDDG45S-9:XZMDKCBDDG45S-9
- added LED17: 7, XZMDKCBDDG45S-9:PLCC4_SMD-LED_3p2X2p8_SLD, symbol XZMDKCBDDG45S-9:XZMDKCBDDG45S-9
- added LED18: 8, XZMDKCBDDG45S-9:PLCC4_SMD-LED_3p2X2p8_SLD, symbol XZMDKCBDDG45S-9:XZMDKCBDDG45S-9
- added LED19: 9, XZMDKCBDDG45S-9:PLCC4_SMD-LED_3p2X2p8_SLD, symbol XZMDKCBDDG45S-9:XZMDKCBDDG45S-9
- added LED2: F1, XZMDKCBDDG45S-9:PLCC4_SMD-LED_3p2X2p8_SLD, symbol XZMDKCBDDG45S-9:XZMDKCBDDG45S-9
- added LED20: TAB, XZMDKCBDDG45S-9:PLCC4_SMD-LED_3p2X2p8_SLD, symbol XZMDKCBDDG45S-9:XZMDKCBDDG45S-9
- added LED21: Q, XZMDKCBDDG45S-9:PLCC4_SMD-LED_3p2X2p8_SLD, symbol XZMDKCBDDG45S-9:XZMDKCBDDG45S-9
- added LED22: W, XZMDKCBDDG45S-9:PLCC4_SMD-LED_3p2X2p8_SLD, symbol XZMDKCBDDG45S-9:XZMDKCBDDG45S-9
- added LED23: E, XZMDKCBDDG45S-9:PLCC4_SMD-LED_3p2X2p8_SLD, symbol XZMDKCBDDG45S-9:XZMDKCBDDG45S-9
- added LED24: R, XZMDKCBDDG45S-9:PLCC4_SMD-LED_3p2X2p8_SLD, symbol XZMDKCBDDG45S-9:XZMDKCBDDG45S-9
- added LED25: T, XZMDKCBDDG45S-9:PLCC4_SMD-LED_3p2X2p8_SLD, symbol XZMDKCBDDG45S-9:XZMDKCBDDG45S-9
- added LED26: Y, XZMDKCBDDG45S-9:PLCC4_SMD-LED_3p2X2p8_SLD, symbol XZMDKCBDDG45S-9:XZMDKCBDDG45S-9
- added LED27: U, XZMDKCBDDG45S-9:PLCC4_SMD-LED_3p2X2p8_SLD, symbol XZMDKCBDDG45S-9:XZMDKCBDDG45S-9
- added LED28: I, XZMDKCBDDG45S-9:PLCC4_SMD-LED_3p2X2p8_SLD, symbol XZMDKCBDDG45S-9:XZMDKCBDDG45S-9
- added LED29, LED64: O, XZMDKCBDDG45S-9:PLCC4_SMD-LED_3p2X2p8_SLD, symbol XZMDKCBDDG45S-9:XZMDKCBDDG45S-9
- added LED3: F2, XZMDKCBDDG45S-9:PLCC4_SMD-LED_3p2X2p8_SLD, symbol XZMDKCBDDG45S-9:XZMDKCBDDG45S-9
- added LED30: CAPS, XZMDKCBDDG45S-9:PLCC4_SMD-LED_3p2X2p8_SLD, symbol XZMDKCBDDG45S-9:XZMDKCBDDG45S-9
- added LED31: A, XZMDKCBDDG45S-9:PLCC4_SMD-LED_3p2X2p8_SLD, symbol XZMDKCBDDG45S-9:XZMDKCBDDG45S-9
- added LED32: S, XZMDKCBDDG45S-9:PLCC4_SMD-LED_3p2X2p8_SLD, symbol XZMDKCBDDG45S-9:XZMDKCBDDG45S-9
- added LED33: D, XZMDKCBDDG45S-9:PLCC4_SMD-LED_3p2X2p8_SLD, symbol XZMDKCBDDG45S-9:XZMDKCBDDG45S-9
- added LED34: F, XZMDKCBDDG45S-9:PLCC4_SMD-LED_3p2X2p8_SLD, symbol XZMDKCBDDG45S-9:XZMDKCBDDG45S-9
- added LED35: G, XZMDKCBDDG45S-9:PLCC4_SMD-LED_3p2X2p8_SLD, symbol XZMDKCBDDG45S-9:XZMDKCBDDG45S-9
- added LED36: H, XZMDKCBDDG45S-9:PLCC4_SMD-LED_3p2X2p8_SLD, symbol XZMDKCBDDG45S-9:XZMDKCBDDG45S-9
- added LED37: J, XZMDKCBDDG45S-9:PLCC4_SMD-LED_3p2X2p8_SLD, symbol XZMDKCBDDG45S-9:XZMDKCBDDG45S-9
- added LED38: K, XZMDKCBDDG45S-9:PLCC4_SMD-LED_3p2X2p8_SLD, symbol XZMDKCBDDG45S-9:XZMDKCBDDG45S-9
- added LED39: L, XZMDKCBDDG45S-9:PLCC4_SMD-LED_3p2X2p8_SLD, symbol XZMDKCBDDG45S-9:XZMDKCBDDG45S-9
- added LED4: F3, XZMDKCBDDG45S-9:PLCC4_SMD-LED_3p2X2p8_SLD, symbol XZMDKCBDDG45S-9:XZMDKCBDDG45S-9
- added LED40: L_SHIFT, XZMDKCBDDG45S-9:PLCC4_SMD-LED_3p2X2p8_SLD, symbol XZMDKCBDDG45S-9:XZMDKCBDDG45S-9
- added LED41: Z, XZMDKCBDDG45S-9:PLCC4_SMD-LED_3p2X2p8_SLD, symbol XZMDKCBDDG45S-9:XZMDKCBDDG45S-9
- added LED42: X, XZMDKCBDDG45S-9:PLCC4_SMD-LED_3p2X2p8_SLD, symbol XZMDKCBDDG45S-9:XZMDKCBDDG45S-9
- added LED43: C, XZMDKCBDDG45S-9:PLCC4_SMD-LED_3p2X2p8_SLD, symbol XZMDKCBDDG45S-9:XZMDKCBDDG45S-9
- added LED44: V, XZMDKCBDDG45S-9:PLCC4_SMD-LED_3p2X2p8_SLD, symbol XZMDKCBDDG45S-9:XZMDKCBDDG45S-9
- added LED45: B, XZMDKCBDDG45S-9:PLCC4_SMD-LED_3p2X2p8_SLD, symbol XZMDKCBDDG45S-9:XZMDKCBDDG45S-9
- added LED46: N, XZMDKCBDDG45S-9:PLCC4_SMD-LED_3p2X2p8_SLD, symbol XZMDKCBDDG45S-9:XZMDKCBDDG45S-9
- added LED47: M, XZMDKCBDDG45S-9:PLCC4_SMD-LED_3p2X2p8_SLD, symbol XZMDKCBDDG45S-9:XZMDKCBDDG45S-9
- added LED48: ,, XZMDKCBDDG45S-9:PLCC4_SMD-LED_3p2X2p8_SLD, symbol XZMDKCBDDG45S-9:XZMDKCBDDG45S-9
- added LED49: L_CTRL, XZMDKCBDDG45S-9:PLCC4_SMD-LED_3p2X2p8_SLD, symbol XZMDKCBDDG45S-9:XZMDKCBDDG45S-9
- added LED5: F4, XZMDKCBDDG45S-9:PLCC4_SMD-LED_3p2X2p8_SLD, symbol XZMDKCBDDG45S-9:XZMDKCBDDG45S-9
- added LED50: OS, XZMDKCBDDG45S-9:PLCC4_SMD-LED_3p2X2p8_SLD, symbol XZMDKCBDDG45S-9:XZMDKCBDDG45S-9
- added LED51: L_ALT, XZMDKCBDDG45S-9:PLCC4_SMD-LED_3p2X2p8_SLD, symbol XZMDKCBDDG45S-9:XZMDKCBDDG45S-9
- added LED52: L_SPACE, XZMDKCBDDG45S-9:PLCC4_SMD-LED_3p2X2p8_SLD, symbol XZMDKCBDDG45S-9:XZMDKCBDDG45S-9
- added LED53: SPACE, XZMDKCBDDG45S-9:PLCC4_SMD-LED_3p2X2p8_SLD, symbol XZMDKCBDDG45S-9:XZMDKCBDDG45S-9
- added LED54: R_SPACE, XZMDKCBDDG45S-9:PLCC4_SMD-LED_3p2X2p8_SLD, symbol XZMDKCBDDG45S-9:XZMDKCBDDG45S-9
- added LED55: R_ALT, XZMDKCBDDG45S-9:PLCC4_SMD-LED_3p2X2p8_SLD, symbol XZMDKCBDDG45S-9:XZMDKCBDDG45S-9
- added LED56: FN, XZMDKCBDDG45S-9:PLCC4_SMD-LED_3p2X2p8_SLD, symbol XZMDKCBDDG45S-9:XZMDKCBDDG45S-9
- added LED57: F9, XZMDKCBDDG45S-9:PLCC4_SMD-LED_3p2X2p8_SLD, symbol XZMDKCBDDG45S-9:XZMDKCBDDG45S-9
- added LED58: F10, XZMDKCBDDG45S-9:PLCC4_SMD-LED_3p2X2p8_SLD, symbol XZMDKCBDDG45S-9:XZMDKCBDDG45S-9
- added LED59: F11, XZMDKCBDDG45S-9:PLCC4_SMD-LED_3p2X2p8_SLD, symbol XZMDKCBDDG45S-9:XZMDKCBDDG45S-9
- added LED6: F5, XZMDKCBDDG45S-9:PLCC4_SMD-LED_3p2X2p8_SLD, symbol XZMDKCBDDG45S-9:XZMDKCBDDG45S-9
- added LED60: F12, XZMDKCBDDG45S-9:PLCC4_SMD-LED_3p2X2p8_SLD, symbol XZMDKCBDDG45S-9:XZMDKCBDDG45S-9
- added LED61: PRT_SC, XZMDKCBDDG45S-9:PLCC4_SMD-LED_3p2X2p8_SLD, symbol XZMDKCBDDG45S-9:XZMDKCBDDG45S-9
- added LED62: SCR_LK, XZMDKCBDDG45S-9:PLCC4_SMD-LED_3p2X2p8_SLD, symbol XZMDKCBDDG45S-9:XZMDKCBDDG45S-9
- added LED63: PAUSE, XZMDKCBDDG45S-9:PLCC4_SMD-LED_3p2X2p8_SLD, symbol XZMDKCBDDG45S-9:XZMDKCBDDG45S-9
- added LED65: -, XZMDKCBDDG45S-9:PLCC4_SMD-LED_3p2X2p8_SLD, symbol XZMDKCBDDG45S-9:XZMDKCBDDG45S-9
- added LED66: =, XZMDKCBDDG45S-9:PLCC4_SMD-LED_3p2X2p8_SLD, symbol XZMDKCBDDG45S-9:XZMDKCBDDG45S-9
- added LED67: BACKSPACE, XZMDKCBDDG45S-9:PLCC4_SMD-LED_3p2X2p8_SLD, symbol XZMDKCBDDG45S-9:XZMDKCBDDG45S-9
- added LED68: INSERT, XZMDKCBDDG45S-9:PLCC4_SMD-LED_3p2X2p8_SLD, symbol XZMDKCBDDG45S-9:XZMDKCBDDG45S-9
- added LED69: HOME, XZMDKCBDDG45S-9:PLCC4_SMD-LED_3p2X2p8_SLD, symbol XZMDKCBDDG45S-9:XZMDKCBDDG45S-9
- added LED7: F6, XZMDKCBDDG45S-9:PLCC4_SMD-LED_3p2X2p8_SLD, symbol XZMDKCBDDG45S-9:XZMDKCBDDG45S-9
- added LED70: PG_UP, XZMDKCBDDG45S-9:PLCC4_SMD-LED_3p2X2p8_SLD, symbol XZMDKCBDDG45S-9:XZMDKCBDDG45S-9
- added LED71: NUM_LOCK, XZMDKCBDDG45S-9:PLCC4_SMD-LED_3p2X2p8_SLD, symbol XZMDKCBDDG45S-9:XZMDKCBDDG45S-9
- added LED72: PAD_/, XZMDKCBDDG45S-9:PLCC4_SMD-LED_3p2X2p8_SLD, symbol XZMDKCBDDG45S-9:XZMDKCBDDG45S-9
- added LED73: *, XZMDKCBDDG45S-9:PLCC4_SMD-LED_3p2X2p8_SLD, symbol XZMDKCBDDG45S-9:XZMDKCBDDG45S-9
- added LED74: PAD_-, XZMDKCBDDG45S-9:PLCC4_SMD-LED_3p2X2p8_SLD, symbol XZMDKCBDDG45S-9:XZMDKCBDDG45S-9
- added LED75: P, XZMDKCBDDG45S-9:PLCC4_SMD-LED_3p2X2p8_SLD, symbol XZMDKCBDDG45S-9:XZMDKCBDDG45S-9
- added LED76: [, XZMDKCBDDG45S-9:PLCC4_SMD-LED_3p2X2p8_SLD, symbol XZMDKCBDDG45S-9:XZMDKCBDDG45S-9
- added LED77: ], XZMDKCBDDG45S-9:PLCC4_SMD-LED_3p2X2p8_SLD, symbol XZMDKCBDDG45S-9:XZMDKCBDDG45S-9
- added LED78: \, XZMDKCBDDG45S-9:PLCC4_SMD-LED_3p2X2p8_SLD, symbol XZMDKCBDDG45S-9:XZMDKCBDDG45S-9
- added LED79: DEL, XZMDKCBDDG45S-9:PLCC4_SMD-LED_3p2X2p8_SLD, symbol XZMDKCBDDG45S-9:XZMDKCBDDG45S-9
- added LED8: F7, XZMDKCBDDG45S-9:PLCC4_SMD-LED_3p2X2p8_SLD, symbol XZMDKCBDDG45S-9:XZMDKCBDDG45S-9
- added LED80: END, XZMDKCBDDG45S-9:PLCC4_SMD-LED_3p2X2p8_SLD, symbol XZMDKCBDDG45S-9:XZMDKCBDDG45S-9
- added LED81: PG_DN, XZMDKCBDDG45S-9:PLCC4_SMD-LED_3p2X2p8_SLD, symbol XZMDKCBDDG45S-9:XZMDKCBDDG45S-9
- added LED82: PAD_7, XZMDKCBDDG45S-9:PLCC4_SMD-LED_3p2X2p8_SLD, symbol XZMDKCBDDG45S-9:XZMDKCBDDG45S-9
- added LED83: PAD_8, XZMDKCBDDG45S-9:PLCC4_SMD-LED_3p2X2p8_SLD, symbol XZMDKCBDDG45S-9:XZMDKCBDDG45S-9
- added LED84: PAD_9, XZMDKCBDDG45S-9:PLCC4_SMD-LED_3p2X2p8_SLD, symbol XZMDKCBDDG45S-9:XZMDKCBDDG45S-9
- added LED85: +, XZMDKCBDDG45S-9:PLCC4_SMD-LED_3p2X2p8_SLD, symbol XZMDKCBDDG45S-9:XZMDKCBDDG45S-9
- added LED86: ;, XZMDKCBDDG45S-9:PLCC4_SMD-LED_3p2X2p8_SLD, symbol XZMDKCBDDG45S-9:XZMDKCBDDG45S-9
- added LED87: ', XZMDKCBDDG45S-9:PLCC4_SMD-LED_3p2X2p8_SLD, symbol XZMDKCBDDG45S-9:XZMDKCBDDG45S-9
- added LED88: ENTER, XZMDKCBDDG45S-9:PLCC4_SMD-LED_3p2X2p8_SLD, symbol XZMDKCBDDG45S-9:XZMDKCBDDG45S-9
- added LED89: PAD_4, XZMDKCBDDG45S-9:PLCC4_SMD-LED_3p2X2p8_SLD, symbol XZMDKCBDDG45S-9:XZMDKCBDDG45S-9
- added LED9: F8, XZMDKCBDDG45S-9:PLCC4_SMD-LED_3p2X2p8_SLD, symbol XZMDKCBDDG45S-9:XZMDKCBDDG45S-9
- added LED90: PAD_5, XZMDKCBDDG45S-9:PLCC4_SMD-LED_3p2X2p8_SLD, symbol XZMDKCBDDG45S-9:XZMDKCBDDG45S-9
- added LED91: PAD_6, XZMDKCBDDG45S-9:PLCC4_SMD-LED_3p2X2p8_SLD, symbol XZMDKCBDDG45S-9:XZMDKCBDDG45S-9
- added LED92: ., XZMDKCBDDG45S-9:PLCC4_SMD-LED_3p2X2p8_SLD, symbol XZMDKCBDDG45S-9:XZMDKCBDDG45S-9
- added LED93: /, XZMDKCBDDG45S-9:PLCC4_SMD-LED_3p2X2p8_SLD, symbol XZMDKCBDDG45S-9:XZMDKCBDDG45S-9
- added LED94: R_SHIFT, XZMDKCBDDG45S-9:PLCC4_SMD-LED_3p2X2p8_SLD, symbol XZMDKCBDDG45S-9:XZMDKCBDDG45S-9
- added LED95: U_ARROW, XZMDKCBDDG45S-9:PLCC4_SMD-LED_3p2X2p8_SLD, symbol XZMDKCBDDG45S-9:XZMDKCBDDG45S-9
- added LED96: PAD_1, XZMDKCBDDG45S-9:PLCC4_SMD-LED_3p2X2p8_SLD, symbol XZMDKCBDDG45S-9:XZMDKCBDDG45S-9
- added LED97: PAD_2, XZMDKCBDDG45S-9:PLCC4_SMD-LED_3p2X2p8_SLD, symbol XZMDKCBDDG45S-9:XZMDKCBDDG45S-9
- added LED98: PAD_3, XZMDKCBDDG45S-9:PLCC4_SMD-LED_3p2X2p8_SLD, symbol XZMDKCBDDG45S-9:XZMDKCBDDG45S-9
Connections:
- net CS10 is gone; now on net CS1: R_G4.1
- net CS11 is gone; now on net CS2: R_R4.1
- net CS12 is gone; now on net CS3: R_B4.1
- net CS13 is gone; now on net CS1: R_G5.1
- net CS14 is gone; now on net CS2: R_R5.1
- net CS15 is gone; now on net CS3: R_B5.1
- net CS16 is gone; now on net CS1: R_G6.1
- net CS17 is gone; now on net CS2: R_R6.1
- net CS18 is gone; now on net CS3: R_B6.1
- net CS19 is gone; now on net CS1: R_G7.1
- net CS20 is gone; now on net CS2: R_R7.1
- net CS21 is gone; now on net CS3: R_B7.1
- net CS22 is gone; now on net CS1: R_G8.1
- net CS23 is gone; now on net CS2: R_R8.1
- net CS24 is gone; now on net CS3: R_B8.1
- net CS25 is gone; now on net CS1: R_G9.1
- net CS26 is gone; now on net CS2: R_R9.1
- net CS27 is gone; now on net CS3: R_B9.1
- net CS28 is gone; now on net CS1: R_G10.1
- net CS29 is gone; now on net CS2: R_R10.1
- net CS30 is gone; now on net CS3: R_B10.1
- net CS31 is gone; now on net CS1: R_G11.1
- net CS32 is gone; now on net CS2: R_R11.1
- net CS33 is gone; now on net CS3: R_B11.1
- net CS34 is gone; now on net CS1: R_G12.1
- net CS35 is gone; now on net CS2: R_R12.1
- net CS36 is gone; now on net CS3: R_B12.1
- net CS37 is gone; now on net CS1: R_G13.1
- net CS38 is gone; now on net CS2: R_R13.1
- net CS39 is gone; now on net CS3: R_B13.1
- net CS40 is gone; now on net CS1: R_G14.1
- net CS41 is gone; now on net CS2: R_R14.1
- net CS42 is gone; now on net CS3: R_B14.1
- net CS43 is gone; now on net CS1: R_G15.1
- net CS44 is gone; now on net CS2: R_R15.1
- net CS45 is gone; now on net CS3: R_B15.1
- net CS46 is gone; now on net CS1: R_G16.1
- net CS47 is gone; now on net CS2: R_R16.1
- net CS48 is gone; now on net CS3: R_B16.1
- net CS49 is gone; now on net CS1: R_G17.1
- net CS50 is gone; now on net CS2: R_R17.1
- net CS51 is gone; now on net CS3: R_B17.1
- net CS52 is gone; now on net CS1: R_G18.1
- net CS53 is gone; now on net CS2: R_R18.1
- net CS54 is gone; now on net CS3: R_B18.1
- net CS55 is gone; now on net CS1: R_G19.1
- net CS56 is gone; now on net CS2: R_R19.1
- net CS57 is gone; now on net CS3: R_B19.1
- net CS58 is gone; now on net CS1: R_G20.1
- net CS59 is gone; now on net CS2: R_R20.1
- net CS60 is gone; now on net CS3: R_B20.1
- net CS7 is gone; now on net CS1: R_G3.1
- net CS8 is gone; now on net CS2: R_R3.1
- net CS9 is gone; now on net CS3: R_B3.1
- net SW1: now also LED1.2 (IN), LED2.2 (IN), LED3.2 (IN), LED4.2 (IN), LED5.2 (IN), LED6.2 (IN), LED7.2 (IN), LED8.2 (IN), LED9.2 (IN)
- net SW10: now also LED86.2 (IN), LED87.2 (IN), LED88.2 (IN), LED89.2 (IN), LED90.2 (IN), LED91.2 (IN)
- net SW11: now also LED92.2 (IN), LED93.2 (IN), LED94.2 (IN), LED95.2 (IN), LED96.2 (IN), LED97.2 (IN), LED98.2 (IN)
- net SW12: now also LED100.2 (IN), LED101.2 (IN), LED102.2 (IN), LED103.2 (IN), LED104.2 (IN), LED105.2 (IN), LED106.2 (IN), LED107.2 (IN), LED56.2 (IN)
- net SW2: now also LED10.2 (IN), LED11.2 (IN), LED12.2 (IN), LED13.2 (IN), LED14.2 (IN), LED15.2 (IN), LED16.2 (IN), LED17.2 (IN), LED18.2 (IN), LED19.2 (IN)
- net SW3: now also LED20.2 (IN), LED21.2 (IN), LED22.2 (IN), LED23.2 (IN), LED24.2 (IN), LED25.2 (IN), LED26.2 (IN), LED27.2 (IN), LED28.2 (IN), LED29.2 (IN)
- net SW4: now also LED30.2 (IN), LED31.2 (IN), LED32.2 (IN), LED33.2 (IN), LED34.2 (IN), LED35.2 (IN), LED36.2 (IN), LED37.2 (IN), LED38.2 (IN), LED39.2 (IN)
- net SW5: now also LED40.2 (IN), LED41.2 (IN), LED42.2 (IN), LED43.2 (IN), LED44.2 (IN), LED45.2 (IN), LED46.2 (IN), LED47.2 (IN), LED48.2 (IN)
- net SW6: now also LED49.2 (IN), LED50.2 (IN), LED51.2 (IN), LED52.2 (IN), LED53.2 (IN), LED54.2 (IN), LED55.2 (IN)
- net SW7: now also LED57.2 (IN), LED58.2 (IN), LED59.2 (IN), LED60.2 (IN), LED61.2 (IN), LED62.2 (IN), LED63.2 (IN), LED73.2 (IN), LED74.2 (IN)
- net SW8: now also LED64.2 (IN), LED65.2 (IN), LED66.2 (IN), LED67.2 (IN), LED68.2 (IN), LED69.2 (IN), LED70.2 (IN), LED71.2 (IN), LED72.2 (IN), LED85.2 (IN)
- net SW9: now also LED75.2 (IN), LED76.2 (IN), LED77.2 (IN), LED78.2 (IN), LED79.2 (IN), LED80.2 (IN), LED81.2 (IN), LED82.2 (IN), LED83.2 (IN), LED84.2 (IN)
- net at R_B7.2: now also LED16.3 (B), LED26.3 (B), LED36.3 (B), LED45.3 (B), LED6.3 (B)
- net at R_B1.2: now also LED1.3 (B), LED10.3 (B), LED20.3 (B), LED30.3 (B), LED40.3 (B), LED49.3 (B)
- net at R_G1.2: now also LED1.4 (G), LED10.4 (G), LED20.4 (G), LED30.4 (G), LED40.4 (G), LED49.4 (G)
- net at R_R1.2: now also LED1.1 (R), LED10.1 (R), LED20.1 (R), LED30.1 (R), LED40.1 (R), LED49.1 (R)
- net at R_B4.2: now also LED13.3 (B), LED23.3 (B), LED3.3 (B), LED33.3 (B), LED42.3 (B), LED52.3 (B)
- net at R_G4.2: now also LED13.4 (G), LED23.4 (G), LED3.4 (G), LED33.4 (G), LED42.4 (G), LED52.4 (G)
- net at R_R4.2: now also LED13.1 (R), LED23.1 (R), LED3.1 (R), LED33.1 (R), LED42.1 (R), LED52.1 (R)
- net at R_B16.2: now also LED102.3 (B), LED62.3 (B), LED69.3 (B), LED80.3 (B), LED95.3 (B)
- net at R_G16.2: now also LED102.4 (G), LED62.4 (G), LED69.4 (G), LED80.4 (G), LED95.4 (G)
- net at R_R16.2: now also LED102.1 (R), LED62.1 (R), LED69.1 (R), LED80.1 (R), LED95.1 (R)
- net at R_R2.2: now also LED11.1 (R), LED21.1 (R), LED31.1 (R), LED50.1 (R)
- net at R_B19.2: now also LED105.3 (B), LED72.3 (B), LED73.3 (B), LED83.3 (B), LED90.3 (B), LED97.3 (B)
- net at R_G19.2: now also LED105.4 (G), LED72.4 (G), LED73.4 (G), LED83.4 (G), LED90.4 (G), LED97.4 (G)
- net at R_R19.2: now also LED105.1 (R), LED72.1 (R), LED73.1 (R), LED83.1 (R), LED90.1 (R), LED97.1 (R)
- net at R_B2.2: now also LED11.3 (B), LED21.3 (B), LED31.3 (B), LED50.3 (B)
- net at R_G2.2: now also LED11.4 (G), LED21.4 (G), LED31.4 (G), LED50.4 (G)
- net at R_B18.2: now also LED104.3 (B), LED71.3 (B), LED82.3 (B), LED89.3 (B), LED96.3 (B)
- net at R_G18.2: now also LED104.4 (G), LED71.4 (G), LED82.4 (G), LED89.4 (G), LED96.4 (G)
- net at R_R18.2: now also LED104.1 (R), LED71.1 (R), LED82.1 (R), LED89.1 (R), LED96.1 (R)
- net at R_B9.2: now also LED18.3 (B), LED28.3 (B), LED38.3 (B), LED47.3 (B), LED55.3 (B), LED8.3 (B)
- net at R_G9.2: now also LED18.4 (G), LED28.4 (G), LED38.4 (G), LED47.4 (G), LED55.4 (G), LED8.4 (G)
- net at R_R9.2: now also LED18.1 (R), LED28.1 (R), LED38.1 (R), LED47.1 (R), LED55.1 (R), LED8.1 (R)
- net at R_B3.2: now also LED12.3 (B), LED2.3 (B), LED22.3 (B), LED32.3 (B), LED41.3 (B), LED51.3 (B)
- net at R_G3.2: now also LED12.4 (G), LED2.4 (G), LED22.4 (G), LED32.4 (G), LED41.4 (G), LED51.4 (G)
- net at R_R3.2: now also LED12.1 (R), LED2.1 (R), LED22.1 (R), LED32.1 (R), LED41.1 (R), LED51.1 (R)
- net at R_G17.2: now also LED103.4 (G), LED63.4 (G), LED70.4 (G), LED81.4 (G)
- net at R_B11.2: now also LED56.3 (B), LED57.3 (B), LED64.3 (B), LED75.3 (B), LED86.3 (B), LED92.3 (B)
- net at R_B14.2: now also R_G14.2, R_R14.2, LED100.1 (R), LED100.3 (B), LED100.4 (G), LED60.1 (R), LED60.3 (B), LED60.4 (G), LED67.1 (R), LED67.3 (B), LED67.4 (G), LED78.1 (R), LED78.3 (B), LED78.4 (G), LED88.1 (R), LED88.3 (B), LED88.4 (G), LED94.1 (R), LED94.3 (B), LED94.4 (G)
- net at R_G11.2: now also LED56.4 (G), LED57.4 (G), LED64.4 (G), LED75.4 (G), LED86.4 (G), LED92.4 (G)
- net at R_R7.2: now also LED16.1 (R), LED26.1 (R), LED36.1 (R), LED45.1 (R), LED6.1 (R)
- net at R_B10.2: now also LED19.3 (B), LED29.3 (B), LED39.3 (B), LED48.3 (B), LED9.3 (B)
- net at R_G10.2: now also LED19.4 (G), LED29.4 (G), LED39.4 (G), LED48.4 (G), LED9.4 (G)
- net at R_R10.2: now also LED19.1 (R), LED29.1 (R), LED39.1 (R), LED48.1 (R), LED9.1 (R)
- net at R_G13.2: now also LED59.4 (G), LED66.4 (G), LED77.4 (G)
- net at R_B20.2: now also LED106.3 (B), LED74.3 (B), LED84.3 (B), LED85.3 (B), LED91.3 (B), LED98.3 (B)
- net at R_G20.2: now also LED106.4 (G), LED74.4 (G), LED84.4 (G), LED85.4 (G), LED91.4 (G), LED98.4 (G)
- net at R_R20.2: now also LED106.1 (R), LED74.1 (R), LED84.1 (R), LED85.1 (R), LED91.1 (R), LED98.1 (R)
- net at R_R11.2: now also LED56.1 (R), LED57.1 (R), LED64.1 (R), LED75.1 (R), LED86.1 (R), LED92.1 (R)
- net at R_B5.2: now also LED14.3 (B), LED24.3 (B), LED34.3 (B), LED4.3 (B), LED43.3 (B)
- net at R_G5.2: now also LED14.4 (G), LED24.4 (G), LED34.4 (G), LED4.4 (G), LED43.4 (G)
- net at R_R5.2: now also LED14.1 (R), LED24.1 (R), LED34.1 (R), LED4.1 (R), LED43.1 (R)
- net at R_B8.2: now also LED17.3 (B), LED27.3 (B), LED37.3 (B), LED46.3 (B), LED54.3 (B), LED7.3 (B)
- net at R_G8.2: now also LED17.4 (G), LED27.4 (G), LED37.4 (G), LED46.4 (G), LED54.4 (G), LED7.4 (G)
- net at R_R8.2: now also LED17.1 (R), LED27.1 (R), LED37.1 (R), LED46.1 (R), LED54.1 (R), LED7.1 (R)
- net at R_B15.2: now also LED101.3 (B), LED61.3 (B), LED68.3 (B), LED79.3 (B)
- net at R_G15.2: now also LED101.4 (G), LED61.4 (G), LED68.4 (G), LED79.4 (G)
- net at R_R15.2: now also LED101.1 (R), LED61.1 (R), LED68.1 (R), LED79.1 (R)
- net at R_R6.2: now also LED15.1 (R), LED25.1 (R), LED35.1 (R), LED44.1 (R), LED5.1 (R), LED53.1 (R)
- net at R_B6.2: now also LED15.3 (B), LED25.3 (B), LED35.3 (B), LED44.3 (B), LED5.3 (B), LED53.3 (B)
- net at R_G6.2: now also LED15.4 (G), LED25.4 (G), LED35.4 (G), LED44.4 (G), LED5.4 (G), LED53.4 (G)
- net at R_G7.2: now also LED16.4 (G), LED26.4 (G), LED36.4 (G), LED45.4 (G), LED6.4 (G)
- net at R_B12.2: now also LED107.3 (B), LED58.3 (B), LED65.3 (B), LED76.3 (B), LED87.3 (B), LED93.3 (B)
- net at R_G12.2: now also LED107.4 (G), LED58.4 (G), LED65.4 (G), LED76.4 (G), LED87.4 (G), LED93.4 (G)
- net at R_R12.2: now also LED107.1 (R), LED58.1 (R), LED65.1 (R), LED76.1 (R), LED87.1 (R), LED93.1 (R)
- net at R_R17.2: now also LED103.1 (R), LED63.1 (R), LED70.1 (R), LED81.1 (R)
- net at R_B17.2: now also LED103.3 (B), LED63.3 (B), LED70.3 (B), LED81.3 (B)
- net at R_B13.2: now also LED59.3 (B), LED66.3 (B), LED77.3 (B)
- net at R_R13.2: now also LED59.1 (R), LED66.1 (R), LED77.1 (R)
Other:
- moved on the sheet: R_B1, R_G1, R_R1

Commit message: MCU pins all routed
Just need to finish led drivers and connect matrix
Connections:
- net CS1: no longer R_G10.1, R_G11.1, R_G12.1, R_G13.1, R_G14.1, R_G15.1, R_G16.1, R_G17.1, R_G18.1, R_G19.1, R_G20.1, R_G3.1, R_G4.1, R_G5.1, R_G6.1, R_G7.1, R_G8.1, R_G9.1
- net CS2: no longer R_R10.1, R_R11.1, R_R12.1, R_R13.1, R_R14.1, R_R15.1, R_R16.1, R_R17.1, R_R18.1, R_R19.1, R_R20.1, R_R3.1, R_R4.1, R_R5.1, R_R6.1, R_R7.1, R_R8.1, R_R9.1
- net CS3: no longer R_B10.1, R_B11.1, R_B12.1, R_B13.1, R_B14.1, R_B15.1, R_B16.1, R_B17.1, R_B18.1, R_B19.1, R_B20.1, R_B3.1, R_B4.1, R_B5.1, R_B6.1, R_B7.1, R_B8.1, R_B9.1
- new net CS10: R_G4.1
- new net CS11: R_R4.1
- new net CS12: R_B4.1
- new net CS13: R_G5.1
- new net CS14: R_R5.1
- new net CS15: R_B5.1
- new net CS16: R_G6.1
- new net CS17: R_R6.1
- new net CS18: R_B6.1
- new net CS19: R_G7.1
- new net CS20: R_R7.1
- new net CS21: R_B7.1
- new net CS22: R_G8.1
- new net CS23: R_R8.1
- new net CS24: R_B8.1
- new net CS25: R_G9.1
- new net CS26: R_R9.1
- new net CS27: R_B9.1
- new net CS28: R_G10.1
- new net CS29: R_R10.1
- new net CS30: R_B10.1
- new net CS31: R_G11.1
- new net CS32: R_R11.1
- new net CS33: R_B11.1
- new net CS34: R_G12.1
- new net CS35: R_R12.1
- new net CS36: R_B12.1
- new net CS37: R_G13.1
- new net CS38: R_R13.1
- new net CS39: R_B13.1
- new net CS40: R_G14.1
- new net CS41: R_R14.1
- new net CS42: R_B14.1
- new net CS43: R_G15.1
- new net CS44: R_R15.1
- new net CS45: R_B15.1
- new net CS46: R_G16.1
- new net CS47: R_R16.1
- new net CS48: R_B16.1
- new net CS49: R_G17.1
- new net CS50: R_R17.1
- new net CS51: R_B17.1
- new net CS52: R_G18.1
- new net CS53: R_R18.1
- new net CS54: R_B18.1
- new net CS55: R_G19.1
- new net CS56: R_R19.1
- new net CS57: R_B19.1
- new net CS58: R_G20.1
- new net CS59: R_R20.1
- new net CS60: R_B20.1
- new net CS7: R_G3.1
- new net CS8: R_R3.1
- new net CS9: R_B3.1

Commit message: Began Routing Columns and Rows
Parts:
- removed LED107: MENU, XZMDKCBDDG45S-9:PLCC4_SMD-LED_3p2X2p8_SLD, symbol XZMDKCBDDG45S-9:XZMDKCBDDG45S-9
- removed LED53: SPACE, XZMDKCBDDG45S-9:PLCC4_SMD-LED_3p2X2p8_SLD, symbol XZMDKCBDDG45S-9:XZMDKCBDDG45S-9
- removed LED56: FN, XZMDKCBDDG45S-9:PLCC4_SMD-LED_3p2X2p8_SLD, symbol XZMDKCBDDG45S-9:XZMDKCBDDG45S-9
- added LED49: SPACE, XZMDKCBDDG45S-9:PLCC4_SMD-LED_3p2X2p8_SLD, symbol XZMDKCBDDG45S-9:XZMDKCBDDG45S-9
- added LED98: FN, XZMDKCBDDG45S-9:PLCC4_SMD-LED_3p2X2p8_SLD, symbol XZMDKCBDDG45S-9:XZMDKCBDDG45S-9
- added LED99: MENU, XZMDKCBDDG45S-9:PLCC4_SMD-LED_3p2X2p8_SLD, symbol XZMDKCBDDG45S-9:XZMDKCBDDG45S-9
- renumbered LED49 to LED50, LED50 to LED51, LED51 to LED52, LED52 to LED53, LED57 to LED56, LED58 to LED57, LED59 to LED58, LED60 to LED59, LED61 to LED60, LED62 to LED61, LED63 to LED62, LED64 to LED63, LED65 to LED64, LED66 to LED65, LED67 to LED66, LED68 to LED67, LED69 to LED68, LED70 to LED69, LED71 to LED70, LED72 to LED71, LED73 to LED72, LED74 to LED73, LED75 to LED74, LED76 to LED75, LED77 to LED76, LED78 to LED77, LED79 to LED78, LED80 to LED79, LED81 to LED80, LED82 to LED81, LED83 to LED82, LED84 to LED83, LED85 to LED84, LED86 to LED85, LED87 to LED86, LED88 to LED87, LED89 to LED88, LED90 to LED89, LED91 to LED90, LED92 to LED91, LED93 to LED92, LED94 to LED93, LED95 to LED94, LED96 to LED95, LED97 to LED96, LED98 to LED97
Connections:
- net CS31: now also R_B18.1; no longer R_G11.1
- net CS32: now also R_R18.1; no longer R_R11.1
- net CS33: now also R_G18.1; no longer R_B11.1
- net CS34: now also R_B19.1; no longer R_G12.1
- net CS35: now also R_R19.1; no longer R_R12.1
- net CS36: now also R_G19.1; no longer R_B12.1
- net CS37: now also R_R20.1; no longer R_G13.1
- net CS38: now also R_G20.1; no longer R_R13.1
- net CS39: now also R_B20.1; no longer R_B13.1
- net CS40: now also R_G17.1; no longer R_G14.1
- net CS41: now also R_R17.1; no longer R_R14.1
- net CS42: now also R_B17.1; no longer R_B14.1
- net CS43: now also R_G16.1; no longer R_G15.1
- net CS44: now also R_R16.1; no longer R_R15.1
- net CS45: now also R_B16.1; no longer R_B15.1
- net CS46: now also R_G15.1; no longer R_G16.1
- net CS47: now also R_R15.1; no longer R_R16.1
- net CS48: now also R_B15.1; no longer R_B16.1
- net CS49: now also R_G14.1; no longer R_G17.1
- net CS50: now also R_R14.1; no longer R_R17.1
- net CS51: now also R_B14.1; no longer R_B17.1
- net CS52: now also R_G13.1; no longer R_G18.1
- net CS53: now also R_R13.1; no longer R_R18.1
- net CS54: now also R_B13.1; no longer R_B18.1
- net CS55: now also R_G12.1; no longer R_G19.1
- net CS56: now also R_R12.1; no longer R_R19.1
- net CS57: now also R_B12.1; no longer R_B19.1
- net CS58: now also R_G11.1; no longer R_G20.1
- net CS59: now also R_R11.1; no longer R_R20.1
- net CS60: now also R_B11.1; no longer R_B20.1
- net SW12: now also LED55.2 (IN), LED98.2 (IN), LED99.2 (IN)
- net SW6: now also LED49.2 (IN); no longer LED55.2 (IN)
- net at LED57.4 (G), LED64.4 (G), LED75.4 (G)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: now also LED98.4 (G)
- net at LED18.1 (R), LED28.1 (R), LED38.1 (R)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: now also LED54.1 (R); no longer LED55.1 (R)
- net at LED18.3 (B), LED28.3 (B), LED38.3 (B)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: now also LED54.3 (B); no longer LED55.3 (B)
- net at LED18.4 (G), LED28.4 (G), LED38.4 (G)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: now also LED54.4 (G); no longer LED55.4 (G)
- net at LED56.1 (R), LED63.1 (R), LED74.1 (R)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: now also LED55.1 (R)
- net at LED57.3 (B), LED64.3 (B), LED75.3 (B)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: now also LED98.3 (B)
- net at LED16.1 (R), LED26.1 (R), LED36.1 (R)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: now also LED49.1 (R)
- net at LED16.3 (B), LED26.3 (B), LED36.3 (B)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: now also LED49.3 (B)
- net at LED16.4 (G), LED26.4 (G), LED36.4 (G)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: now also LED49.4 (G)
- net at LED57.1 (R), LED64.1 (R), LED75.1 (R)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: now also LED98.1 (R)
- net at LED17.1 (R), LED27.1 (R), LED37.1 (R)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: no longer LED54.1 (R)
- net at LED56.3 (B), LED63.3 (B), LED74.3 (B)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: now also LED55.3 (B)
- net at LED56.4 (G), LED63.4 (G), LED74.4 (G)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: now also LED55.4 (G)
- net at LED17.3 (B), LED27.3 (B), LED37.3 (B)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: no longer LED54.3 (B)
- net at LED17.4 (G), LED27.4 (G), LED37.4 (G)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: no longer LED54.4 (G)
- net at LED58.1 (R), LED65.1 (R), LED76.1 (R)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: now also LED99.1 (R)
- net at LED58.3 (B), LED65.3 (B), LED76.3 (B)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: now also LED99.3 (B)
- net at LED58.4 (G), LED65.4 (G), LED76.4 (G)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: now also LED99.4 (G)
- new net: LED100.1 (R), LED59.1 (R), LED66.1 (R), LED77.1 (R), LED87.1 (R), LED93.1 (R), R_R14.2
- new net: LED100.3 (B), LED59.3 (B), LED66.3 (B), LED77.3 (B), LED87.3 (B), LED93.3 (B), R_B14.2
- new net: LED100.4 (G), LED59.4 (G), LED66.4 (G), LED77.4 (G), LED87.4 (G), LED93.4 (G), R_G14.2
Other:
- moved on the sheet: R_G14
