File: rgbMatrix.kicad_sch (KiCad schematic)
At the start: 195 parts

Commit message: Began changing out backlight for better components
Parts:
- removed C39: 104, Capacitor_SMD:C_0805_2012Metric_Pad1.18x1.45mm_HandSolder, symbol Device:C_Small
- removed LED1: ESC, XZMDKCBDDG45S-9:PLCC4_SMD-LED_3p2X2p8_SLD, symbol XZMDKCBDDG45S-9:XZMDKCBDDG45S-9
- removed LED10: TILDE, XZMDKCBDDG45S-9:PLCC4_SMD-LED_3p2X2p8_SLD, symbol XZMDKCBDDG45S-9:XZMDKCBDDG45S-9
- removed LED100: R_CTRL, XZMDKCBDDG45S-9:PLCC4_SMD-LED_3p2X2p8_SLD, symbol XZMDKCBDDG45S-9:XZMDKCBDDG45S-9
- removed LED101: L_ARROW, XZMDKCBDDG45S-9:PLCC4_SMD-LED_3p2X2p8_SLD, symbol XZMDKCBDDG45S-9:XZMDKCBDDG45S-9
- removed LED102: D_ARROW, XZMDKCBDDG45S-9:PLCC4_SMD-LED_3p2X2p8_SLD, symbol XZMDKCBDDG45S-9:XZMDKCBDDG45S-9
- removed LED103: R_ARROW, XZMDKCBDDG45S-9:PLCC4_SMD-LED_3p2X2p8_SLD, symbol XZMDKCBDDG45S-9:XZMDKCBDDG45S-9
- removed LED104: PAD_0, XZMDKCBDDG45S-9:PLCC4_SMD-LED_3p2X2p8_SLD, symbol XZMDKCBDDG45S-9:XZMDKCBDDG45S-9
- removed LED105: PAD_., XZMDKCBDDG45S-9:PLCC4_SMD-LED_3p2X2p8_SLD, symbol XZMDKCBDDG45S-9:XZMDKCBDDG45S-9
- removed LED106: PAD_ENTER, XZMDKCBDDG45S-9:PLCC4_SMD-LED_3p2X2p8_SLD, symbol XZMDKCBDDG45S-9:XZMDKCBDDG45S-9
- removed LED107, LED108, LED109, LED110, LED111, LED112, LED113, LED114, LED115, LED116, LED117, LED118, LED119, LED120: IN-PI55TATPRPGPB, ul_IN-PI55TATPRPGPB:IN-PI55TATPRPGPB, symbol ul_IN-PI55TATPRPGPB:IN-PI55TATPRPGPB
- removed LED11: 1, XZMDKCBDDG45S-9:PLCC4_SMD-LED_3p2X2p8_SLD, symbol XZMDKCBDDG45S-9:XZMDKCBDDG45S-9
- removed LED12: 2, XZMDKCBDDG45S-9:PLCC4_SMD-LED_3p2X2p8_SLD, symbol XZMDKCBDDG45S-9:XZMDKCBDDG45S-9
- removed LED13: 3, XZMDKCBDDG45S-9:PLCC4_SMD-LED_3p2X2p8_SLD, symbol XZMDKCBDDG45S-9:XZMDKCBDDG45S-9
- removed LED14: 4, XZMDKCBDDG45S-9:PLCC4_SMD-LED_3p2X2p8_SLD, symbol XZMDKCBDDG45S-9:XZMDKCBDDG45S-9
- removed LED15: 5, XZMDKCBDDG45S-9:PLCC4_SMD-LED_3p2X2p8_SLD, symbol XZMDKCBDDG45S-9:XZMDKCBDDG45S-9
- removed LED16: 6, XZMDKCBDDG45S-9:PLCC4_SMD-LED_3p2X2p8_SLD, symbol XZMDKCBDDG45S-9:XZMDKCBDDG45S-9
- removed LED17: 7, XZMDKCBDDG45S-9:PLCC4_SMD-LED_3p2X2p8_SLD, symbol XZMDKCBDDG45S-9:XZMDKCBDDG45S-9
- removed LED18: 8, XZMDKCBDDG45S-9:PLCC4_SMD-LED_3p2X2p8_SLD, symbol XZMDKCBDDG45S-9:XZMDKCBDDG45S-9
- removed LED19: 9, XZMDKCBDDG45S-9:PLCC4_SMD-LED_3p2X2p8_SLD, symbol XZMDKCBDDG45S-9:XZMDKCBDDG45S-9
- removed LED2: F1, XZMDKCBDDG45S-9:PLCC4_SMD-LED_3p2X2p8_SLD, symbol XZMDKCBDDG45S-9:XZMDKCBDDG45S-9
- removed LED20: TAB, XZMDKCBDDG45S-9:PLCC4_SMD-LED_3p2X2p8_SLD, symbol XZMDKCBDDG45S-9:XZMDKCBDDG45S-9
- removed LED21: Q, XZMDKCBDDG45S-9:PLCC4_SMD-LED_3p2X2p8_SLD, symbol XZMDKCBDDG45S-9:XZMDKCBDDG45S-9
- removed LED22: W, XZMDKCBDDG45S-9:PLCC4_SMD-LED_3p2X2p8_SLD, symbol XZMDKCBDDG45S-9:XZMDKCBDDG45S-9
- removed LED23: E, XZMDKCBDDG45S-9:PLCC4_SMD-LED_3p2X2p8_SLD, symbol XZMDKCBDDG45S-9:XZMDKCBDDG45S-9
- removed LED24: R, XZMDKCBDDG45S-9:PLCC4_SMD-LED_3p2X2p8_SLD, symbol XZMDKCBDDG45S-9:XZMDKCBDDG45S-9
- removed LED25: T, XZMDKCBDDG45S-9:PLCC4_SMD-LED_3p2X2p8_SLD, symbol XZMDKCBDDG45S-9:XZMDKCBDDG45S-9
- removed LED26: Y, XZMDKCBDDG45S-9:PLCC4_SMD-LED_3p2X2p8_SLD, symbol XZMDKCBDDG45S-9:XZMDKCBDDG45S-9
- removed LED27: U, XZMDKCBDDG45S-9:PLCC4_SMD-LED_3p2X2p8_SLD, symbol XZMDKCBDDG45S-9:XZMDKCBDDG45S-9
- removed LED28: I, XZMDKCBDDG45S-9:PLCC4_SMD-LED_3p2X2p8_SLD, symbol XZMDKCBDDG45S-9:XZMDKCBDDG45S-9
- removed LED29, LED63: O, XZMDKCBDDG45S-9:PLCC4_SMD-LED_3p2X2p8_SLD, symbol XZMDKCBDDG45S-9:XZMDKCBDDG45S-9
- removed LED3: F2, XZMDKCBDDG45S-9:PLCC4_SMD-LED_3p2X2p8_SLD, symbol XZMDKCBDDG45S-9:XZMDKCBDDG45S-9
- removed LED30: CAPS, XZMDKCBDDG45S-9:PLCC4_SMD-LED_3p2X2p8_SLD, symbol XZMDKCBDDG45S-9:XZMDKCBDDG45S-9
- removed LED31: A, XZMDKCBDDG45S-9:PLCC4_SMD-LED_3p2X2p8_SLD, symbol XZMDKCBDDG45S-9:XZMDKCBDDG45S-9
- removed LED32: S, XZMDKCBDDG45S-9:PLCC4_SMD-LED_3p2X2p8_SLD, symbol XZMDKCBDDG45S-9:XZMDKCBDDG45S-9
- removed LED33: D, XZMDKCBDDG45S-9:PLCC4_SMD-LED_3p2X2p8_SLD, symbol XZMDKCBDDG45S-9:XZMDKCBDDG45S-9
- removed LED34: F, XZMDKCBDDG45S-9:PLCC4_SMD-LED_3p2X2p8_SLD, symbol XZMDKCBDDG45S-9:XZMDKCBDDG45S-9
- removed LED35: G, XZMDKCBDDG45S-9:PLCC4_SMD-LED_3p2X2p8_SLD, symbol XZMDKCBDDG45S-9:XZMDKCBDDG45S-9
- removed LED36: H, XZMDKCBDDG45S-9:PLCC4_SMD-LED_3p2X2p8_SLD, symbol XZMDKCBDDG45S-9:XZMDKCBDDG45S-9
- removed LED37: J, XZMDKCBDDG45S-9:PLCC4_SMD-LED_3p2X2p8_SLD, symbol XZMDKCBDDG45S-9:XZMDKCBDDG45S-9
- removed LED38: K, XZMDKCBDDG45S-9:PLCC4_SMD-LED_3p2X2p8_SLD, symbol XZMDKCBDDG45S-9:XZMDKCBDDG45S-9
- removed LED39: L, XZMDKCBDDG45S-9:PLCC4_SMD-LED_3p2X2p8_SLD, symbol XZMDKCBDDG45S-9:XZMDKCBDDG45S-9
- removed LED4: F3, XZMDKCBDDG45S-9:PLCC4_SMD-LED_3p2X2p8_SLD, symbol XZMDKCBDDG45S-9:XZMDKCBDDG45S-9
- removed LED40: L_SHIFT, XZMDKCBDDG45S-9:PLCC4_SMD-LED_3p2X2p8_SLD, symbol XZMDKCBDDG45S-9:XZMDKCBDDG45S-9
- removed LED41: Z, XZMDKCBDDG45S-9:PLCC4_SMD-LED_3p2X2p8_SLD, symbol XZMDKCBDDG45S-9:XZMDKCBDDG45S-9
- removed LED42: X, XZMDKCBDDG45S-9:PLCC4_SMD-LED_3p2X2p8_SLD, symbol XZMDKCBDDG45S-9:XZMDKCBDDG45S-9
- removed LED43: C, XZMDKCBDDG45S-9:PLCC4_SMD-LED_3p2X2p8_SLD, symbol XZMDKCBDDG45S-9:XZMDKCBDDG45S-9
- removed LED44: V, XZMDKCBDDG45S-9:PLCC4_SMD-LED_3p2X2p8_SLD, symbol XZMDKCBDDG45S-9:XZMDKCBDDG45S-9
- removed LED45: B, XZMDKCBDDG45S-9:PLCC4_SMD-LED_3p2X2p8_SLD, symbol XZMDKCBDDG45S-9:XZMDKCBDDG45S-9
- removed LED46: N, XZMDKCBDDG45S-9:PLCC4_SMD-LED_3p2X2p8_SLD, symbol XZMDKCBDDG45S-9:XZMDKCBDDG45S-9
- removed LED47: M, XZMDKCBDDG45S-9:PLCC4_SMD-LED_3p2X2p8_SLD, symbol XZMDKCBDDG45S-9:XZMDKCBDDG45S-9
- removed LED48: ,, XZMDKCBDDG45S-9:PLCC4_SMD-LED_3p2X2p8_SLD, symbol XZMDKCBDDG45S-9:XZMDKCBDDG45S-9
- removed LED49: SPACE, XZMDKCBDDG45S-9:PLCC4_SMD-LED_3p2X2p8_SLD, symbol XZMDKCBDDG45S-9:XZMDKCBDDG45S-9
- removed LED5: F4, XZMDKCBDDG45S-9:PLCC4_SMD-LED_3p2X2p8_SLD, symbol XZMDKCBDDG45S-9:XZMDKCBDDG45S-9
- removed LED50: L_CTRL, XZMDKCBDDG45S-9:PLCC4_SMD-LED_3p2X2p8_SLD, symbol XZMDKCBDDG45S-9:XZMDKCBDDG45S-9
- removed LED51: OS, XZMDKCBDDG45S-9:PLCC4_SMD-LED_3p2X2p8_SLD, symbol XZMDKCBDDG45S-9:XZMDKCBDDG45S-9
- removed LED52: L_ALT, XZMDKCBDDG45S-9:PLCC4_SMD-LED_3p2X2p8_SLD, symbol XZMDKCBDDG45S-9:XZMDKCBDDG45S-9
- removed LED53: L_SPACE, XZMDKCBDDG45S-9:PLCC4_SMD-LED_3p2X2p8_SLD, symbol XZMDKCBDDG45S-9:XZMDKCBDDG45S-9
- removed LED54: R_SPACE, XZMDKCBDDG45S-9:PLCC4_SMD-LED_3p2X2p8_SLD, symbol XZMDKCBDDG45S-9:XZMDKCBDDG45S-9
- removed LED55: R_ALT, XZMDKCBDDG45S-9:PLCC4_SMD-LED_3p2X2p8_SLD, symbol XZMDKCBDDG45S-9:XZMDKCBDDG45S-9
- removed LED56: F9, XZMDKCBDDG45S-9:PLCC4_SMD-LED_3p2X2p8_SLD, symbol XZMDKCBDDG45S-9:XZMDKCBDDG45S-9
- removed LED57: F10, XZMDKCBDDG45S-9:PLCC4_SMD-LED_3p2X2p8_SLD, symbol XZMDKCBDDG45S-9:XZMDKCBDDG45S-9
- removed LED58: F11, XZMDKCBDDG45S-9:PLCC4_SMD-LED_3p2X2p8_SLD, symbol XZMDKCBDDG45S-9:XZMDKCBDDG45S-9
- removed LED59: F12, XZMDKCBDDG45S-9:PLCC4_SMD-LED_3p2X2p8_SLD, symbol XZMDKCBDDG45S-9:XZMDKCBDDG45S-9
- removed LED6: F5, XZMDKCBDDG45S-9:PLCC4_SMD-LED_3p2X2p8_SLD, symbol XZMDKCBDDG45S-9:XZMDKCBDDG45S-9
- removed LED60: PRT_SC, XZMDKCBDDG45S-9:PLCC4_SMD-LED_3p2X2p8_SLD, symbol XZMDKCBDDG45S-9:XZMDKCBDDG45S-9
- removed LED61: SCR_LK, XZMDKCBDDG45S-9:PLCC4_SMD-LED_3p2X2p8_SLD, symbol XZMDKCBDDG45S-9:XZMDKCBDDG45S-9
- removed LED62: PAUSE, XZMDKCBDDG45S-9:PLCC4_SMD-LED_3p2X2p8_SLD, symbol XZMDKCBDDG45S-9:XZMDKCBDDG45S-9
- removed LED64: -, XZMDKCBDDG45S-9:PLCC4_SMD-LED_3p2X2p8_SLD, symbol XZMDKCBDDG45S-9:XZMDKCBDDG45S-9
- removed LED65: =, XZMDKCBDDG45S-9:PLCC4_SMD-LED_3p2X2p8_SLD, symbol XZMDKCBDDG45S-9:XZMDKCBDDG45S-9
- removed LED66: BACKSPACE, XZMDKCBDDG45S-9:PLCC4_SMD-LED_3p2X2p8_SLD, symbol XZMDKCBDDG45S-9:XZMDKCBDDG45S-9
- removed LED67: INSERT, XZMDKCBDDG45S-9:PLCC4_SMD-LED_3p2X2p8_SLD, symbol XZMDKCBDDG45S-9:XZMDKCBDDG45S-9
- removed LED68: HOME, XZMDKCBDDG45S-9:PLCC4_SMD-LED_3p2X2p8_SLD, symbol XZMDKCBDDG45S-9:XZMDKCBDDG45S-9
- removed LED69: PG_UP, XZMDKCBDDG45S-9:PLCC4_SMD-LED_3p2X2p8_SLD, symbol XZMDKCBDDG45S-9:XZMDKCBDDG45S-9
- removed LED7: F6, XZMDKCBDDG45S-9:PLCC4_SMD-LED_3p2X2p8_SLD, symbol XZMDKCBDDG45S-9:XZMDKCBDDG45S-9
- removed LED70: NUM_LOCK, XZMDKCBDDG45S-9:PLCC4_SMD-LED_3p2X2p8_SLD, symbol XZMDKCBDDG45S-9:XZMDKCBDDG45S-9
- removed LED71: PAD_/, XZMDKCBDDG45S-9:PLCC4_SMD-LED_3p2X2p8_SLD, symbol XZMDKCBDDG45S-9:XZMDKCBDDG45S-9
- removed LED72: *, XZMDKCBDDG45S-9:PLCC4_SMD-LED_3p2X2p8_SLD, symbol XZMDKCBDDG45S-9:XZMDKCBDDG45S-9
- removed LED73: PAD_-, XZMDKCBDDG45S-9:PLCC4_SMD-LED_3p2X2p8_SLD, symbol XZMDKCBDDG45S-9:XZMDKCBDDG45S-9
- removed LED74: P, XZMDKCBDDG45S-9:PLCC4_SMD-LED_3p2X2p8_SLD, symbol XZMDKCBDDG45S-9:XZMDKCBDDG45S-9
- removed LED75: [, XZMDKCBDDG45S-9:PLCC4_SMD-LED_3p2X2p8_SLD, symbol XZMDKCBDDG45S-9:XZMDKCBDDG45S-9
- removed LED76: ], XZMDKCBDDG45S-9:PLCC4_SMD-LED_3p2X2p8_SLD, symbol XZMDKCBDDG45S-9:XZMDKCBDDG45S-9
- removed LED77: \, XZMDKCBDDG45S-9:PLCC4_SMD-LED_3p2X2p8_SLD, symbol XZMDKCBDDG45S-9:XZMDKCBDDG45S-9
- removed LED78: DEL, XZMDKCBDDG45S-9:PLCC4_SMD-LED_3p2X2p8_SLD, symbol XZMDKCBDDG45S-9:XZMDKCBDDG45S-9
- removed LED79: END, XZMDKCBDDG45S-9:PLCC4_SMD-LED_3p2X2p8_SLD, symbol XZMDKCBDDG45S-9:XZMDKCBDDG45S-9
- removed LED8: F7, XZMDKCBDDG45S-9:PLCC4_SMD-LED_3p2X2p8_SLD, symbol XZMDKCBDDG45S-9:XZMDKCBDDG45S-9
- removed LED80: PG_DN, XZMDKCBDDG45S-9:PLCC4_SMD-LED_3p2X2p8_SLD, symbol XZMDKCBDDG45S-9:XZMDKCBDDG45S-9
- removed LED81: PAD_7, XZMDKCBDDG45S-9:PLCC4_SMD-LED_3p2X2p8_SLD, symbol XZMDKCBDDG45S-9:XZMDKCBDDG45S-9
- removed LED82: PAD_8, XZMDKCBDDG45S-9:PLCC4_SMD-LED_3p2X2p8_SLD, symbol XZMDKCBDDG45S-9:XZMDKCBDDG45S-9
- removed LED83: PAD_9, XZMDKCBDDG45S-9:PLCC4_SMD-LED_3p2X2p8_SLD, symbol XZMDKCBDDG45S-9:XZMDKCBDDG45S-9
- removed LED84: +, XZMDKCBDDG45S-9:PLCC4_SMD-LED_3p2X2p8_SLD, symbol XZMDKCBDDG45S-9:XZMDKCBDDG45S-9
- removed LED85: ;, XZMDKCBDDG45S-9:PLCC4_SMD-LED_3p2X2p8_SLD, symbol XZMDKCBDDG45S-9:XZMDKCBDDG45S-9
- removed LED86: ', XZMDKCBDDG45S-9:PLCC4_SMD-LED_3p2X2p8_SLD, symbol XZMDKCBDDG45S-9:XZMDKCBDDG45S-9
- removed LED87: ENTER, XZMDKCBDDG45S-9:PLCC4_SMD-LED_3p2X2p8_SLD, symbol XZMDKCBDDG45S-9:XZMDKCBDDG45S-9
- removed LED88: PAD_4, XZMDKCBDDG45S-9:PLCC4_SMD-LED_3p2X2p8_SLD, symbol XZMDKCBDDG45S-9:XZMDKCBDDG45S-9
- removed LED89: PAD_5, XZMDKCBDDG45S-9:PLCC4_SMD-LED_3p2X2p8_SLD, symbol XZMDKCBDDG45S-9:XZMDKCBDDG45S-9
- removed LED9: F8, XZMDKCBDDG45S-9:PLCC4_SMD-LED_3p2X2p8_SLD, symbol XZMDKCBDDG45S-9:XZMDKCBDDG45S-9
- removed LED90: PAD_6, XZMDKCBDDG45S-9:PLCC4_SMD-LED_3p2X2p8_SLD, symbol XZMDKCBDDG45S-9:XZMDKCBDDG45S-9
- removed LED91: ., XZMDKCBDDG45S-9:PLCC4_SMD-LED_3p2X2p8_SLD, symbol XZMDKCBDDG45S-9:XZMDKCBDDG45S-9
- removed LED92: /, XZMDKCBDDG45S-9:PLCC4_SMD-LED_3p2X2p8_SLD, symbol XZMDKCBDDG45S-9:XZMDKCBDDG45S-9
- removed LED93: R_SHIFT, XZMDKCBDDG45S-9:PLCC4_SMD-LED_3p2X2p8_SLD, symbol XZMDKCBDDG45S-9:XZMDKCBDDG45S-9
- removed LED94: U_ARROW, XZMDKCBDDG45S-9:PLCC4_SMD-LED_3p2X2p8_SLD, symbol XZMDKCBDDG45S-9:XZMDKCBDDG45S-9
- removed LED95: PAD_1, XZMDKCBDDG45S-9:PLCC4_SMD-LED_3p2X2p8_SLD, symbol XZMDKCBDDG45S-9:XZMDKCBDDG45S-9
- removed LED96: PAD_2, XZMDKCBDDG45S-9:PLCC4_SMD-LED_3p2X2p8_SLD, symbol XZMDKCBDDG45S-9:XZMDKCBDDG45S-9
- removed LED97: PAD_3, XZMDKCBDDG45S-9:PLCC4_SMD-LED_3p2X2p8_SLD, symbol XZMDKCBDDG45S-9:XZMDKCBDDG45S-9
- removed LED98: FN, XZMDKCBDDG45S-9:PLCC4_SMD-LED_3p2X2p8_SLD, symbol XZMDKCBDDG45S-9:XZMDKCBDDG45S-9
- removed LED99: MENU, XZMDKCBDDG45S-9:PLCC4_SMD-LED_3p2X2p8_SLD, symbol XZMDKCBDDG45S-9:XZMDKCBDDG45S-9
- added LED1: ESC, E6CC1205RGBC3UDA:LED__RBG_1206_3216Metric_ReverseMount_Hole2.2x2.2mm, symbol Device:LED_RAGB
- added LED10: TILDE, E6CC1205RGBC3UDA:LED__RBG_1206_3216Metric_ReverseMount_Hole2.2x2.2mm, symbol Device:LED_RAGB
- added LED100: R_CTRL, E6CC1205RGBC3UDA:LED__RBG_1206_3216Metric_ReverseMount_Hole2.2x2.2mm, symbol Device:LED_RAGB
- added LED101: L_ARROW, E6CC1205RGBC3UDA:LED__RBG_1206_3216Metric_ReverseMount_Hole2.2x2.2mm, symbol Device:LED_RAGB
- added LED102: DN_ARROW, E6CC1205RGBC3UDA:LED__RBG_1206_3216Metric_ReverseMount_Hole2.2x2.2mm, symbol Device:LED_RAGB
- added LED103: R_ARROW, E6CC1205RGBC3UDA:LED__RBG_1206_3216Metric_ReverseMount_Hole2.2x2.2mm, symbol Device:LED_RAGB
- added LED104: PAD_0, E6CC1205RGBC3UDA:LED__RBG_1206_3216Metric_ReverseMount_Hole2.2x2.2mm, symbol Device:LED_RAGB
- added LED105: PAD_., E6CC1205RGBC3UDA:LED__RBG_1206_3216Metric_ReverseMount_Hole2.2x2.2mm, symbol Device:LED_RAGB
- added LED106: PAD_ENTER, E6CC1205RGBC3UDA:LED__RBG_1206_3216Metric_ReverseMount_Hole2.2x2.2mm, symbol Device:LED_RAGB
- added LED107, LED108, LED109, LED110, LED111, LED112, LED113, LED114, LED115, LED116, LED117, LED118, LED119: WS2812B, LED_SMD:LED_WS2812B_PLCC4_5.0x5.0mm_P3.2mm, symbol LED:WS2812B
- added LED11: 1, E6CC1205RGBC3UDA:LED__RBG_1206_3216Metric_ReverseMount_Hole2.2x2.2mm, symbol Device:LED_RAGB
- added LED12: 2, E6CC1205RGBC3UDA:LED__RBG_1206_3216Metric_ReverseMount_Hole2.2x2.2mm, symbol Device:LED_RAGB
- added LED13: 3, E6CC1205RGBC3UDA:LED__RBG_1206_3216Metric_ReverseMount_Hole2.2x2.2mm, symbol Device:LED_RAGB
- added LED14: 4, E6CC1205RGBC3UDA:LED__RBG_1206_3216Metric_ReverseMount_Hole2.2x2.2mm, symbol Device:LED_RAGB
- added LED15: 5, E6CC1205RGBC3UDA:LED__RBG_1206_3216Metric_ReverseMount_Hole2.2x2.2mm, symbol Device:LED_RAGB
- added LED16: 6, E6CC1205RGBC3UDA:LED__RBG_1206_3216Metric_ReverseMount_Hole2.2x2.2mm, symbol Device:LED_RAGB
- added LED17: 7, E6CC1205RGBC3UDA:LED__RBG_1206_3216Metric_ReverseMount_Hole2.2x2.2mm, symbol Device:LED_RAGB
- added LED18: 8, E6CC1205RGBC3UDA:LED__RBG_1206_3216Metric_ReverseMount_Hole2.2x2.2mm, symbol Device:LED_RAGB
- added LED19: 9, E6CC1205RGBC3UDA:LED__RBG_1206_3216Metric_ReverseMount_Hole2.2x2.2mm, symbol Device:LED_RAGB
- added LED2: F1, E6CC1205RGBC3UDA:LED__RBG_1206_3216Metric_ReverseMount_Hole2.2x2.2mm, symbol Device:LED_RAGB
- added LED20: TAB, E6CC1205RGBC3UDA:LED__RBG_1206_3216Metric_ReverseMount_Hole2.2x2.2mm, symbol Device:LED_RAGB
- added LED21: Q, E6CC1205RGBC3UDA:LED__RBG_1206_3216Metric_ReverseMount_Hole2.2x2.2mm, symbol Device:LED_RAGB
- added LED22: W, E6CC1205RGBC3UDA:LED__RBG_1206_3216Metric_ReverseMount_Hole2.2x2.2mm, symbol Device:LED_RAGB
- added LED23: E, E6CC1205RGBC3UDA:LED__RBG_1206_3216Metric_ReverseMount_Hole2.2x2.2mm, symbol Device:LED_RAGB
- added LED24: R, E6CC1205RGBC3UDA:LED__RBG_1206_3216Metric_ReverseMount_Hole2.2x2.2mm, symbol Device:LED_RAGB
- added LED25: T, E6CC1205RGBC3UDA:LED__RBG_1206_3216Metric_ReverseMount_Hole2.2x2.2mm, symbol Device:LED_RAGB
- added LED26: Y, E6CC1205RGBC3UDA:LED__RBG_1206_3216Metric_ReverseMount_Hole2.2x2.2mm, symbol Device:LED_RAGB
- added LED27: U, E6CC1205RGBC3UDA:LED__RBG_1206_3216Metric_ReverseMount_Hole2.2x2.2mm, symbol Device:LED_RAGB
- added LED28: I, E6CC1205RGBC3UDA:LED__RBG_1206_3216Metric_ReverseMount_Hole2.2x2.2mm, symbol Device:LED_RAGB
- added LED29: O, E6CC1205RGBC3UDA:LED__RBG_1206_3216Metric_ReverseMount_Hole2.2x2.2mm, symbol Device:LED_RAGB
- added LED3: F2, E6CC1205RGBC3UDA:LED__RBG_1206_3216Metric_ReverseMount_Hole2.2x2.2mm, symbol Device:LED_RAGB
- added LED30: CAPS, E6CC1205RGBC3UDA:LED__RBG_1206_3216Metric_ReverseMount_Hole2.2x2.2mm, symbol Device:LED_RAGB
- added LED31: A, E6CC1205RGBC3UDA:LED__RBG_1206_3216Metric_ReverseMount_Hole2.2x2.2mm, symbol Device:LED_RAGB
- added LED32: S, E6CC1205RGBC3UDA:LED__RBG_1206_3216Metric_ReverseMount_Hole2.2x2.2mm, symbol Device:LED_RAGB
- added LED33: D, E6CC1205RGBC3UDA:LED__RBG_1206_3216Metric_ReverseMount_Hole2.2x2.2mm, symbol Device:LED_RAGB
- added LED34: F, E6CC1205RGBC3UDA:LED__RBG_1206_3216Metric_ReverseMount_Hole2.2x2.2mm, symbol Device:LED_RAGB
- added LED35: G, E6CC1205RGBC3UDA:LED__RBG_1206_3216Metric_ReverseMount_Hole2.2x2.2mm, symbol Device:LED_RAGB
- added LED36: H, E6CC1205RGBC3UDA:LED__RBG_1206_3216Metric_ReverseMount_Hole2.2x2.2mm, symbol Device:LED_RAGB
- added LED37: J, E6CC1205RGBC3UDA:LED__RBG_1206_3216Metric_ReverseMount_Hole2.2x2.2mm, symbol Device:LED_RAGB
- added LED38: K, E6CC1205RGBC3UDA:LED__RBG_1206_3216Metric_ReverseMount_Hole2.2x2.2mm, symbol Device:LED_RAGB
- added LED39: L, E6CC1205RGBC3UDA:LED__RBG_1206_3216Metric_ReverseMount_Hole2.2x2.2mm, symbol Device:LED_RAGB
- added LED4: F3, E6CC1205RGBC3UDA:LED__RBG_1206_3216Metric_ReverseMount_Hole2.2x2.2mm, symbol Device:LED_RAGB
- added LED40: L_SHIFT, E6CC1205RGBC3UDA:LED__RBG_1206_3216Metric_ReverseMount_Hole2.2x2.2mm, symbol Device:LED_RAGB
- added LED41: Z, E6CC1205RGBC3UDA:LED__RBG_1206_3216Metric_ReverseMount_Hole2.2x2.2mm, symbol Device:LED_RAGB
- added LED42: X, E6CC1205RGBC3UDA:LED__RBG_1206_3216Metric_ReverseMount_Hole2.2x2.2mm, symbol Device:LED_RAGB
- added LED43: C, E6CC1205RGBC3UDA:LED__RBG_1206_3216Metric_ReverseMount_Hole2.2x2.2mm, symbol Device:LED_RAGB
- added LED44: V, E6CC1205RGBC3UDA:LED__RBG_1206_3216Metric_ReverseMount_Hole2.2x2.2mm, symbol Device:LED_RAGB
- added LED45: B, E6CC1205RGBC3UDA:LED__RBG_1206_3216Metric_ReverseMount_Hole2.2x2.2mm, symbol Device:LED_RAGB
- added LED46: N, E6CC1205RGBC3UDA:LED__RBG_1206_3216Metric_ReverseMount_Hole2.2x2.2mm, symbol Device:LED_RAGB
- added LED47: M, E6CC1205RGBC3UDA:LED__RBG_1206_3216Metric_ReverseMount_Hole2.2x2.2mm, symbol Device:LED_RAGB
- added LED48: ,, E6CC1205RGBC3UDA:LED__RBG_1206_3216Metric_ReverseMount_Hole2.2x2.2mm, symbol Device:LED_RAGB
- added LED49: L_CTRL, E6CC1205RGBC3UDA:LED__RBG_1206_3216Metric_ReverseMount_Hole2.2x2.2mm, symbol Device:LED_RAGB
- added LED5: F4, E6CC1205RGBC3UDA:LED__RBG_1206_3216Metric_ReverseMount_Hole2.2x2.2mm, symbol Device:LED_RAGB
- added LED50: OS, E6CC1205RGBC3UDA:LED__RBG_1206_3216Metric_ReverseMount_Hole2.2x2.2mm, symbol Device:LED_RAGB
- added LED51: L_ALT, E6CC1205RGBC3UDA:LED__RBG_1206_3216Metric_ReverseMount_Hole2.2x2.2mm, symbol Device:LED_RAGB
- added LED52: L_SPACE, E6CC1205RGBC3UDA:LED__RBG_1206_3216Metric_ReverseMount_Hole2.2x2.2mm, symbol Device:LED_RAGB
- added LED53: SPACE, E6CC1205RGBC3UDA:LED__RBG_1206_3216Metric_ReverseMount_Hole2.2x2.2mm, symbol Device:LED_RAGB
- added LED54: R_SPACE, E6CC1205RGBC3UDA:LED__RBG_1206_3216Metric_ReverseMount_Hole2.2x2.2mm, symbol Device:LED_RAGB
- added LED55: F9, E6CC1205RGBC3UDA:LED__RBG_1206_3216Metric_ReverseMount_Hole2.2x2.2mm, symbol Device:LED_RAGB
- added LED56: F10, E6CC1205RGBC3UDA:LED__RBG_1206_3216Metric_ReverseMount_Hole2.2x2.2mm, symbol Device:LED_RAGB
- added LED57: F11, E6CC1205RGBC3UDA:LED__RBG_1206_3216Metric_ReverseMount_Hole2.2x2.2mm, symbol Device:LED_RAGB
- added LED58: F12, E6CC1205RGBC3UDA:LED__RBG_1206_3216Metric_ReverseMount_Hole2.2x2.2mm, symbol Device:LED_RAGB
- added LED59: PRT_SC, E6CC1205RGBC3UDA:LED__RBG_1206_3216Metric_ReverseMount_Hole2.2x2.2mm, symbol Device:LED_RAGB
- added LED6: F5, E6CC1205RGBC3UDA:LED__RBG_1206_3216Metric_ReverseMount_Hole2.2x2.2mm, symbol Device:LED_RAGB
- added LED60: SC_LCK, E6CC1205RGBC3UDA:LED__RBG_1206_3216Metric_ReverseMount_Hole2.2x2.2mm, symbol Device:LED_RAGB
- added LED61: PAUSE, E6CC1205RGBC3UDA:LED__RBG_1206_3216Metric_ReverseMount_Hole2.2x2.2mm, symbol Device:LED_RAGB
- added LED62: 0, E6CC1205RGBC3UDA:LED__RBG_1206_3216Metric_ReverseMount_Hole2.2x2.2mm, symbol Device:LED_RAGB
- added LED63: -, E6CC1205RGBC3UDA:LED__RBG_1206_3216Metric_ReverseMount_Hole2.2x2.2mm, symbol Device:LED_RAGB
- added LED64: =, E6CC1205RGBC3UDA:LED__RBG_1206_3216Metric_ReverseMount_Hole2.2x2.2mm, symbol Device:LED_RAGB
- added LED65: BACKSPACE, E6CC1205RGBC3UDA:LED__RBG_1206_3216Metric_ReverseMount_Hole2.2x2.2mm, symbol Device:LED_RAGB
- added LED66: INSERT, E6CC1205RGBC3UDA:LED__RBG_1206_3216Metric_ReverseMount_Hole2.2x2.2mm, symbol Device:LED_RAGB
- added LED67: HOME, E6CC1205RGBC3UDA:LED__RBG_1206_3216Metric_ReverseMount_Hole2.2x2.2mm, symbol Device:LED_RAGB
- added LED68: PG_UP, E6CC1205RGBC3UDA:LED__RBG_1206_3216Metric_ReverseMount_Hole2.2x2.2mm, symbol Device:LED_RAGB
- added LED69: NUM_LK, E6CC1205RGBC3UDA:LED__RBG_1206_3216Metric_ReverseMount_Hole2.2x2.2mm, symbol Device:LED_RAGB
- added LED7: F6, E6CC1205RGBC3UDA:LED__RBG_1206_3216Metric_ReverseMount_Hole2.2x2.2mm, symbol Device:LED_RAGB
- added LED70: PAD_/, E6CC1205RGBC3UDA:LED__RBG_1206_3216Metric_ReverseMount_Hole2.2x2.2mm, symbol Device:LED_RAGB
- added LED71: *, E6CC1205RGBC3UDA:LED__RBG_1206_3216Metric_ReverseMount_Hole2.2x2.2mm, symbol Device:LED_RAGB
- added LED72: PAD_-, E6CC1205RGBC3UDA:LED__RBG_1206_3216Metric_ReverseMount_Hole2.2x2.2mm, symbol Device:LED_RAGB
- added LED73: P, E6CC1205RGBC3UDA:LED__RBG_1206_3216Metric_ReverseMount_Hole2.2x2.2mm, symbol Device:LED_RAGB
- added LED74: [, E6CC1205RGBC3UDA:LED__RBG_1206_3216Metric_ReverseMount_Hole2.2x2.2mm, symbol Device:LED_RAGB
- added LED75: }, E6CC1205RGBC3UDA:LED__RBG_1206_3216Metric_ReverseMount_Hole2.2x2.2mm, symbol Device:LED_RAGB
- added LED76: \, E6CC1205RGBC3UDA:LED__RBG_1206_3216Metric_ReverseMount_Hole2.2x2.2mm, symbol Device:LED_RAGB
- added LED77: DEL, E6CC1205RGBC3UDA:LED__RBG_1206_3216Metric_ReverseMount_Hole2.2x2.2mm, symbol Device:LED_RAGB
- added LED78: END, E6CC1205RGBC3UDA:LED__RBG_1206_3216Metric_ReverseMount_Hole2.2x2.2mm, symbol Device:LED_RAGB
- added LED79: PG_DN, E6CC1205RGBC3UDA:LED__RBG_1206_3216Metric_ReverseMount_Hole2.2x2.2mm, symbol Device:LED_RAGB
- added LED8: F7, E6CC1205RGBC3UDA:LED__RBG_1206_3216Metric_ReverseMount_Hole2.2x2.2mm, symbol Device:LED_RAGB
- added LED80: PAD_7, E6CC1205RGBC3UDA:LED__RBG_1206_3216Metric_ReverseMount_Hole2.2x2.2mm, symbol Device:LED_RAGB
- added LED81: PAD_8, E6CC1205RGBC3UDA:LED__RBG_1206_3216Metric_ReverseMount_Hole2.2x2.2mm, symbol Device:LED_RAGB
- added LED82: PAD_9, E6CC1205RGBC3UDA:LED__RBG_1206_3216Metric_ReverseMount_Hole2.2x2.2mm, symbol Device:LED_RAGB
- added LED83: +, E6CC1205RGBC3UDA:LED__RBG_1206_3216Metric_ReverseMount_Hole2.2x2.2mm, symbol Device:LED_RAGB
- added LED84: ;, E6CC1205RGBC3UDA:LED__RBG_1206_3216Metric_ReverseMount_Hole2.2x2.2mm, symbol Device:LED_RAGB
- added LED85: ', E6CC1205RGBC3UDA:LED__RBG_1206_3216Metric_ReverseMount_Hole2.2x2.2mm, symbol Device:LED_RAGB
- added LED86: ENTER, E6CC1205RGBC3UDA:LED__RBG_1206_3216Metric_ReverseMount_Hole2.2x2.2mm, symbol Device:LED_RAGB
- added LED87: PAD_4, E6CC1205RGBC3UDA:LED__RBG_1206_3216Metric_ReverseMount_Hole2.2x2.2mm, symbol Device:LED_RAGB
- added LED88: PAD_5, E6CC1205RGBC3UDA:LED__RBG_1206_3216Metric_ReverseMount_Hole2.2x2.2mm, symbol Device:LED_RAGB
- added LED89: PAD_6, E6CC1205RGBC3UDA:LED__RBG_1206_3216Metric_ReverseMount_Hole2.2x2.2mm, symbol Device:LED_RAGB
- added LED9: F8, E6CC1205RGBC3UDA:LED__RBG_1206_3216Metric_ReverseMount_Hole2.2x2.2mm, symbol Device:LED_RAGB
- added LED90: ., E6CC1205RGBC3UDA:LED__RBG_1206_3216Metric_ReverseMount_Hole2.2x2.2mm, symbol Device:LED_RAGB
- added LED91: /, E6CC1205RGBC3UDA:LED__RBG_1206_3216Metric_ReverseMount_Hole2.2x2.2mm, symbol Device:LED_RAGB
- added LED92: R_SHIFT, E6CC1205RGBC3UDA:LED__RBG_1206_3216Metric_ReverseMount_Hole2.2x2.2mm, symbol Device:LED_RAGB
- added LED93: UP_ARROW, E6CC1205RGBC3UDA:LED__RBG_1206_3216Metric_ReverseMount_Hole2.2x2.2mm, symbol Device:LED_RAGB
- added LED94: PAD_1, E6CC1205RGBC3UDA:LED__RBG_1206_3216Metric_ReverseMount_Hole2.2x2.2mm, symbol Device:LED_RAGB
- added LED95: PAD_2, E6CC1205RGBC3UDA:LED__RBG_1206_3216Metric_ReverseMount_Hole2.2x2.2mm, symbol Device:LED_RAGB
- added LED96: PAD_3, E6CC1205RGBC3UDA:LED__RBG_1206_3216Metric_ReverseMount_Hole2.2x2.2mm, symbol Device:LED_RAGB
- added LED97: R_ALT, E6CC1205RGBC3UDA:LED__RBG_1206_3216Metric_ReverseMount_Hole2.2x2.2mm, symbol Device:LED_RAGB
- added LED98: FN, E6CC1205RGBC3UDA:LED__RBG_1206_3216Metric_ReverseMount_Hole2.2x2.2mm, symbol Device:LED_RAGB
- added LED99: MENU, E6CC1205RGBC3UDA:LED__RBG_1206_3216Metric_ReverseMount_Hole2.2x2.2mm, symbol Device:LED_RAGB
- C18: renamed from C35; value 104 -> 100n
- C32: renamed from C36; value 104 -> 100n
- C34: renamed from C42; value 104 -> 100n
- C35: renamed from C43; value 104 -> 100n
- C36: renamed from C34; value 104 -> 100n
- C37, C40, C41: value 104 -> 100n
- C38: renamed from C18; value 104 -> 100n
- C39: renamed from C38; value 104 -> 100n
- C42: renamed from C44; value 104 -> 100n
- C43: renamed from C32; value 104 -> 100n
- C44: renamed from C45; value 104 -> 100n
Connections:
- net +5V: now also LED107.1 (VDD), LED108.1 (VDD), LED109.1 (VDD), LED110.1 (VDD), LED111.1 (VDD), LED112.1 (VDD), LED113.1 (VDD), LED114.1 (VDD), LED115.1 (VDD), LED116.1 (VDD), LED117.1 (VDD), LED118.1 (VDD), LED119.1 (VDD)
- net GND: now also LED107.3 (VSS), LED108.3 (VSS), LED109.3 (VSS), LED110.3 (VSS), LED111.3 (VSS), LED112.3 (VSS), LED113.3 (VSS), LED114.3 (VSS), LED115.3 (VSS), LED116.3 (VSS), LED117.3 (VSS), LED118.3 (VSS), LED119.3 (VSS)
- net SW1: now also LED1.2 (A), LED2.2 (A), LED3.2 (A), LED4.2 (A), LED5.2 (A), LED6.2 (A), LED7.2 (A), LED8.2 (A), LED9.2 (A)
- net SW10: now also LED84.2 (A), LED85.2 (A), LED86.2 (A), LED87.2 (A), LED88.2 (A), LED89.2 (A)
- net SW11: now also LED90.2 (A), LED91.2 (A), LED92.2 (A), LED93.2 (A), LED94.2 (A), LED95.2 (A), LED96.2 (A)
- net SW12: now also LED100.2 (A), LED101.2 (A), LED102.2 (A), LED103.2 (A), LED104.2 (A), LED105.2 (A), LED106.2 (A), LED97.2 (A), LED98.2 (A), LED99.2 (A)
- net SW2: now also LED10.2 (A), LED11.2 (A), LED12.2 (A), LED13.2 (A), LED14.2 (A), LED15.2 (A), LED16.2 (A), LED17.2 (A), LED18.2 (A), LED19.2 (A)
- net SW3: now also LED20.2 (A), LED21.2 (A), LED22.2 (A), LED23.2 (A), LED24.2 (A), LED25.2 (A), LED26.2 (A), LED27.2 (A), LED28.2 (A), LED29.2 (A)
- net SW4: now also LED30.2 (A), LED31.2 (A), LED32.2 (A), LED33.2 (A), LED34.2 (A), LED35.2 (A), LED36.2 (A), LED37.2 (A), LED38.2 (A), LED39.2 (A)
- net SW5: now also LED40.2 (A), LED41.2 (A), LED42.2 (A), LED43.2 (A), LED44.2 (A), LED45.2 (A), LED46.2 (A), LED47.2 (A), LED48.2 (A)
- net SW6: now also LED49.2 (A), LED50.2 (A), LED51.2 (A), LED52.2 (A), LED53.2 (A), LED54.2 (A)
- net SW7: now also LED55.2 (A), LED56.2 (A), LED57.2 (A), LED58.2 (A), LED59.2 (A), LED60.2 (A), LED61.2 (A), LED71.2 (A), LED72.2 (A)
- net SW8: now also LED62.2 (A), LED63.2 (A), LED64.2 (A), LED65.2 (A), LED66.2 (A), LED67.2 (A), LED68.2 (A), LED69.2 (A), LED70.2 (A), LED83.2 (A)
- net SW9: now also LED73.2 (A), LED74.2 (A), LED75.2 (A), LED76.2 (A), LED77.2 (A), LED78.2 (A), LED79.2 (A), LED80.2 (A), LED81.2 (A), LED82.2 (A)
- net at R_G12.2: now also LED56.3 (GK), LED63.3 (GK), LED74.3 (GK), LED85.3 (GK), LED91.3 (GK), LED98.3 (GK)
- net at R_R11.2: now also LED55.1 (RK), LED62.1 (RK), LED73.1 (RK), LED84.1 (RK), LED90.1 (RK), LED97.1 (RK)
- net at R_R20.2: now also LED106.1 (RK), LED72.1 (RK), LED82.1 (RK), LED83.1 (RK), LED89.1 (RK), LED96.1 (RK)
- net at R_R4.2: now also LED13.1 (RK), LED23.1 (RK), LED3.1 (RK), LED33.1 (RK), LED42.1 (RK), LED52.1 (RK)
- net at R_B4.2: now also LED13.4 (BK), LED23.4 (BK), LED3.4 (BK), LED33.4 (BK), LED42.4 (BK), LED52.4 (BK)
- net at R_G4.2: now also LED13.3 (GK), LED23.3 (GK), LED3.3 (GK), LED33.3 (GK), LED42.3 (GK), LED52.3 (GK)
- net at R_R14.2: now also LED100.1 (RK), LED58.1 (RK), LED65.1 (RK), LED76.1 (RK), LED86.1 (RK), LED92.1 (RK)
- net at R_B14.2: now also LED100.4 (BK), LED58.4 (BK), LED65.4 (BK), LED76.4 (BK), LED86.4 (BK), LED92.4 (BK)
- net at R_G14.2: now also LED100.3 (GK), LED58.3 (GK), LED65.3 (GK), LED76.3 (GK), LED86.3 (GK), LED92.3 (GK)
- net at R_B3.2: now also LED12.4 (BK), LED2.4 (BK), LED22.4 (BK), LED32.4 (BK), LED41.4 (BK), LED51.4 (BK)
- net at R_B12.2: now also LED56.4 (BK), LED63.4 (BK), LED74.4 (BK), LED85.4 (BK), LED91.4 (BK), LED98.4 (BK)
- net at R_R5.2: now also LED14.1 (RK), LED24.1 (RK), LED34.1 (RK), LED4.1 (RK), LED43.1 (RK)
- net at R_B5.2: now also LED14.4 (BK), LED24.4 (BK), LED34.4 (BK), LED4.4 (BK), LED43.4 (BK)
- net at R_G5.2: now also LED14.3 (GK), LED24.3 (GK), LED34.3 (GK), LED4.3 (GK), LED43.3 (GK)
- net at R_R1.2: now also LED1.1 (RK), LED10.1 (RK), LED20.1 (RK), LED30.1 (RK), LED40.1 (RK), LED49.1 (RK)
- net at R_B1.2: now also LED1.4 (BK), LED10.4 (BK), LED20.4 (BK), LED30.4 (BK), LED40.4 (BK), LED49.4 (BK)
- net at R_G1.2: now also LED1.3 (GK), LED10.3 (GK), LED20.3 (GK), LED30.3 (GK), LED40.3 (GK), LED49.3 (GK)
- net at R_B10.2: now also LED19.4 (BK), LED29.4 (BK), LED39.4 (BK), LED48.4 (BK), LED9.4 (BK)
- net at R_R10.2: now also LED19.1 (RK), LED29.1 (RK), LED39.1 (RK), LED48.1 (RK), LED9.1 (RK)
- net at R_G10.2: now also LED19.3 (GK), LED29.3 (GK), LED39.3 (GK), LED48.3 (GK), LED9.3 (GK)
- net at R_B9.2: now also LED18.4 (BK), LED28.4 (BK), LED38.4 (BK), LED47.4 (BK), LED54.4 (BK), LED8.4 (BK)
- net at R_R18.2: now also LED104.1 (RK), LED69.1 (RK), LED80.1 (RK), LED87.1 (RK), LED94.1 (RK)
- net at R_R16.2: now also LED102.1 (RK), LED60.1 (RK), LED67.1 (RK), LED78.1 (RK), LED93.1 (RK)
- net at R_B16.2: now also LED102.4 (BK), LED60.4 (BK), LED67.4 (BK), LED78.4 (BK), LED93.4 (BK)
- net at R_G16.2: now also LED102.3 (GK), LED60.3 (GK), LED67.3 (GK), LED78.3 (GK), LED93.3 (GK)
- net at R_B20.2: now also LED106.4 (BK), LED72.4 (BK), LED82.4 (BK), LED83.4 (BK), LED89.4 (BK), LED96.4 (BK)
- net at R_G20.2: now also LED106.3 (GK), LED72.3 (GK), LED82.3 (GK), LED83.3 (GK), LED89.3 (GK), LED96.3 (GK)
- net at R_R9.2: now also LED18.1 (RK), LED28.1 (RK), LED38.1 (RK), LED47.1 (RK), LED54.1 (RK), LED8.1 (RK)
- net at R_R7.2: now also LED16.1 (RK), LED26.1 (RK), LED36.1 (RK), LED45.1 (RK), LED53.1 (RK), LED6.1 (RK)
- net at R_B7.2: now also LED16.4 (BK), LED26.4 (BK), LED36.4 (BK), LED45.4 (BK), LED53.4 (BK), LED6.4 (BK)
- net at R_G7.2: now also LED16.3 (GK), LED26.3 (GK), LED36.3 (GK), LED45.3 (GK), LED53.3 (GK), LED6.3 (GK)
- net at R_R15.2: now also LED101.1 (RK), LED59.1 (RK), LED66.1 (RK), LED77.1 (RK)
- net at R_R19.2: now also LED105.1 (RK), LED70.1 (RK), LED71.1 (RK), LED81.1 (RK), LED88.1 (RK), LED95.1 (RK)
- net at R_B19.2: now also LED105.4 (BK), LED70.4 (BK), LED71.4 (BK), LED81.4 (BK), LED88.4 (BK), LED95.4 (BK)
- net at R_G19.2: now also LED105.3 (GK), LED70.3 (GK), LED71.3 (GK), LED81.3 (GK), LED88.3 (GK), LED95.3 (GK)
- net at R_R17.2: now also LED103.1 (RK), LED61.1 (RK), LED68.1 (RK), LED79.1 (RK)
- net at R_R12.2: now also LED56.1 (RK), LED63.1 (RK), LED74.1 (RK), LED85.1 (RK), LED91.1 (RK), LED98.1 (RK)
- net at R_R6.2: now also LED15.1 (RK), LED25.1 (RK), LED35.1 (RK), LED44.1 (RK), LED5.1 (RK)
- net at R_B6.2: now also LED15.4 (BK), LED25.4 (BK), LED35.4 (BK), LED44.4 (BK), LED5.4 (BK)
- net at R_G6.2: now also LED15.3 (GK), LED25.3 (GK), LED35.3 (GK), LED44.3 (GK), LED5.3 (GK)
- net at R_R8.2: now also LED17.1 (RK), LED27.1 (RK), LED37.1 (RK), LED46.1 (RK), LED7.1 (RK)
- net at R_G15.2: now also LED101.3 (GK), LED59.3 (GK), LED66.3 (GK), LED77.3 (GK)
- net at R_B11.2: now also LED55.4 (BK), LED62.4 (BK), LED73.4 (BK), LED84.4 (BK), LED90.4 (BK), LED97.4 (BK)
- net at R_G11.2: now also LED55.3 (GK), LED62.3 (GK), LED73.3 (GK), LED84.3 (GK), LED90.3 (GK), LED97.3 (GK)
- net at R_B8.2: now also LED17.4 (BK), LED27.4 (BK), LED37.4 (BK), LED46.4 (BK), LED7.4 (BK)
- net at R_G8.2: now also LED17.3 (GK), LED27.3 (GK), LED37.3 (GK), LED46.3 (GK), LED7.3 (GK)
- net at R_B18.2: now also LED104.4 (BK), LED69.4 (BK), LED80.4 (BK), LED87.4 (BK), LED94.4 (BK)
- net at R_G18.2: now also LED104.3 (GK), LED69.3 (GK), LED80.3 (GK), LED87.3 (GK), LED94.3 (GK)
- net at R_B17.2: now also LED103.4 (BK), LED61.4 (BK), LED68.4 (BK), LED79.4 (BK)
- net at R_G17.2: now also LED103.3 (GK), LED61.3 (GK), LED68.3 (GK), LED79.3 (GK)
- net at R_B15.2: now also LED101.4 (BK), LED59.4 (BK), LED66.4 (BK), LED77.4 (BK)
- net at R_R13.2: now also LED57.1 (RK), LED64.1 (RK), LED75.1 (RK), LED99.1 (RK)
- net at R_B13.2: now also LED57.4 (BK), LED64.4 (BK), LED75.4 (BK), LED99.4 (BK)
- net at R_G13.2: now also LED57.3 (GK), LED64.3 (GK), LED75.3 (GK), LED99.3 (GK)
- net at R_G9.2: now also LED18.3 (GK), LED28.3 (GK), LED38.3 (GK), LED47.3 (GK), LED54.3 (GK), LED8.3 (GK)
- net at R_R2.2: now also LED11.1 (RK), LED21.1 (RK), LED31.1 (RK), LED50.1 (RK)
- net at R_B2.2: now also LED11.4 (BK), LED21.4 (BK), LED31.4 (BK), LED50.4 (BK)
- net at R_G2.2: now also LED11.3 (GK), LED21.3 (GK), LED31.3 (GK), LED50.3 (GK)
- net at R_R3.2: now also LED12.1 (RK), LED2.1 (RK), LED22.1 (RK), LED32.1 (RK), LED41.1 (RK), LED51.1 (RK)
- net at R_G3.2: now also LED12.3 (GK), LED2.3 (GK), LED22.3 (GK), LED32.3 (GK), LED41.3 (GK), LED51.3 (GK)
- net at R3.2: now also LED111.4 (DIN)
- new net: LED107.4 (DIN), LED108.2 (DOUT)
- new net: LED108.4 (DIN), LED109.2 (DOUT)
- new net: LED114.4 (DIN), LED117.2 (DOUT)
- new net: LED116.2 (DOUT), LED117.4 (DIN)
- new net: LED113.2 (DOUT), LED115.4 (DIN)
- new net: LED107.2 (DOUT), LED113.4 (DIN)
- new net: LED109.4 (DIN), LED110.2 (DOUT)
- new net: LED110.4 (DIN), LED111.2 (DOUT)
- new net: LED112.4 (DIN), LED114.2 (DOUT)
- new net: LED115.2 (DOUT), LED118.4 (DIN)
- new net: LED116.4 (DIN), LED119.2 (DOUT)
- new net: LED118.2 (DOUT), LED119.4 (DIN)
Other:
- note added: "Left Side LEDs"
- note added: "Right Side LEDs"
- note removed: "Left Side Of Keyboard"
- note removed: "Right Side of Keyboard"
- note removed: "SW10, COL 20"
- note removed: "SW11 COL 20"
- note removed: "SW12, COL 20"
- note removed: "SW7, COL 19"
- note removed: "SW7, COL 20"
- note removed: "SW8, COL 20"
- note removed: "SW9, COL 20"
