File: KB-pcb-practice.kicad_pcb (KiCad board)
At the start: 2 copper layers, 436 parts, among them J1 ARM 10pin, SW1 Reset, SW10 F7, SW100 R_CTRL, SW101 L_ARROW, SW102 DN_ARROW, SW103 R_ARROW, SW104 PAD_0, SW105 PAD_., SW106 PAD_ENTER, SW11 F8, SW12 F9, SW13 F10, SW14 F11, SW15 F12, SW16 PRT_SC, SW17 SCR_LK, SW18 PAUSE, SW19 TILDE, SW2 Boot, SW20 1, SW21 2, SW22 3, SW23 4, SW24 5, SW25 6, SW26 7, SW27 8, SW28 9, SW29 0, SW3 ESC, SW30 -, SW31 =, SW32 BACKSPACE, SW33 INSERT, SW34 HOME, SW35 PG_UP, SW36 NUM_LK, SW37 PAD_/, SW38 *, SW39 PAD_-, SW4 F1, SW40 TAB, SW41 Q, SW42 W, SW43 E, SW44 R, SW45 T, SW46 Y, SW47 U, SW48 I, SW49 O, SW5 F2, SW50 P, SW51 [, SW52 ], SW53 \, SW54 DEL, SW55 END, SW56 PG_DN, SW57 PAD_7, SW58 PAD_8, SW59 PAD_9, SW6 F3, SW60 +, SW61 CAPS, SW62 A, SW63 S, SW64 D, SW65 F, SW66 G, SW67 H, SW68 J, SW69 K, SW7 F4, SW70 L, SW71 ;, SW72 ', SW73 ENTER, SW74 PAD_4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

Commit message: Changing hotswap switches
Reverse Mount leds not added yet.
Parts:
- C1, C10, C11, C12, C13, C14, C15, C16, C17, C18, C19, C2, C20, C21, C22, C23, C24, C25, C26, C27, C28, C29, C3, C30, C31, C32, C4, C5, C6, C7, C8, C9, D1, D10, D100, D101, D102, D103, D104, D105, D11, D12, D13, D14, D15, D16, D17, D18, D19, D2, D20, D21, D22, D23, D24, D25, D26, D27, D28, D29, D3, D30, D31, D32, D33, D34, D35, D36, D37, D38, D39, D4, D40, D41, D42, D43, D44, D45, D46, D47, D48, D49, D5, D50, D51, D52, D53, D54, D55, D56, D57, D58, D59, D6, D60, D61, D62, D63, D64, D65, D66, D67, D68, D69, D7, D70, D71, D72, D73, D74, D75, D76, D77, D78, D79, D8, D80, D81, D82, D83, D84, D85, D86, D87, D88, D89, D9, D90, D91, D92, D93, D94, D95, D96, D97, D98, D99, F1, F2, J1, R1, R10, R11, R12, R13, R14, R15, R16, R17, R2, R3, R4, R5, R6, R7, R8, R9, R_B1, R_B10, R_B11, R_B12, R_B13, R_B14, R_B15, R_B16, R_B17, R_B18, R_B19, R_B2, R_B20, R_B3, R_B4, R_B5, R_B6, R_B7, R_B8, R_B9, R_G1, R_G10, R_G11, R_G12, R_G13, R_G14, R_G15, R_G16, R_G17, R_G18, R_G19, R_G2, R_G20, R_G3, R_G4, R_G5, R_G6, R_G7, R_G8, R_G9, R_R1, R_R10, R_R11, R_R12, R_R13, R_R14, R_R15, R_R16, R_R17, R_R18, R_R19, R_R2, R_R20, R_R3, R_R4, R_R5, R_R6, R_R7, R_R8, R_R9, SW1, SW2, U1, U2, U3, U4, U5, USB1, Y1: moved to B.Cu
- SW10, SW101, SW102, SW103, SW105, SW11, SW12, SW13, SW14, SW15, SW16, SW17, SW18, SW19, SW20, SW21, SW22, SW23, SW24, SW25, SW26, SW27, SW28, SW29, SW3, SW30, SW31, SW33, SW34, SW35, SW36, SW37, SW38, SW39, SW4, SW41, SW42, SW43, SW44, SW45, SW46, SW47, SW48, SW49, SW5, SW50, SW51, SW52, SW53, SW54, SW55, SW56, SW57, SW58, SW59, SW6, SW60, SW62, SW63, SW64, SW65, SW66, SW67, SW68, SW69, SW7, SW70, SW71, SW72, SW74, SW75, SW76, SW78, SW79, SW8, SW80, SW81, SW82, SW83, SW84, SW85, SW86, SW87, SW89, SW9, SW90, SW91, SW92, SW94, SW98, SW99: footprint Alps_Only:ALPS-1U -> MX_Only:MXOnly-1U-Hotswap
- SW100, SW40, SW93: footprint Alps_Only:ALPS-1.5U -> MX_Only:MXOnly-1.5U-Hotswap
- SW104: footprint Alps_Only:ALPS-2.25U-LED -> MX_Only:MXOnly-2.25U-Hotswap
- SW106, SW73, SW77, SW88: footprint Alps_Only:ALPS-2.25U -> MX_Only:MXOnly-2.25U-Hotswap
- SW32: footprint Alps_Only:ALPS-2U -> MX_Only:MXOnly-2U-Hotswap
- SW61: footprint Alps_Only:ALPS-1.75U -> MX_Only:MXOnly-1.75U-Hotswap
- SW95, SW97: footprint Alps_Only:ALPS-1.25U -> MX_Only:MXOnly-1.25U-Hotswap
- SW96: footprint Alps_Only:ALPS-6.5U -> MX_Only:MXOnly-6.25U-Hotswap
- moved SW100 575.7 mm to (571.4, 183.5)
- moved SW97 486.1 mm to (507.1, 183.5)
- moved SW104 482.6 mm to (543.7, 254.8)
- moved SW98 466.6 mm to (528.5, 183.5)
- moved SW82 434.7 mm to (433.2, 164.5)
- moved D25 427.0 mm to (568.5, 354.3), turned to 180 degrees
- moved D76 427.0 mm to (568.5, 350.9), turned to 180 degrees
- moved SW96 426.7 mm to (435.8, 183.5)
- moved D100 413.1 mm to (559.0, 334.1), turned to 180 degrees
- moved D18 413.1 mm to (559.0, 340.8), turned to 180 degrees
- moved D33 413.1 mm to (559.0, 347.5), turned to 180 degrees
- moved D52 413.1 mm to (559.0, 337.4), turned to 180 degrees
- moved D64 413.1 mm to (559.0, 330.7), turned to 180 degrees
- moved D88 413.1 mm to (559.0, 344.1), turned to 180 degrees
- moved SW99 410.6 mm to (547.6, 183.5)
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
Commit message: Changed to reverse mount rgb leds
Both symbol and footprint were changed accordingly.
Parts:
- LED1, LED10, LED100, LED101, LED102, LED103, LED104, LED105, LED106, LED11, LED12, LED13, LED14, LED15, LED16, LED17, LED18, LED19, LED2, LED20, LED21, LED22, LED23, LED24, LED25, LED26, LED27, LED28, LED29, LED3, LED30, LED31, LED32, LED33, LED34, LED35, LED36, LED37, LED38, LED39, LED4, LED40, LED41, LED42, LED43, LED44, LED45, LED46, LED47, LED48, LED49, LED5, LED50, LED51, LED52, LED53, LED54, LED55, LED56, LED57, LED58, LED59, LED6, LED60, LED61, LED62, LED63, LED64, LED65, LED66, LED67, LED68, LED69, LED7, LED70, LED71, LED72, LED73, LED74, LED75, LED76, LED77, LED78, LED79, LED8, LED80, LED81, LED82, LED83, LED84, LED85, LED87, LED88, LED89, LED9, LED90, LED91, LED92, LED93, LED94, LED95, LED96, LED97, LED98, LED99: footprint mouser_AAA3528SEEZGKQBKS:AAA3528SEEZGKQBKS -> XZMDKCBDDG45S-9:PLCC4_SMD-LED_3p2X2p8_SLD
- LED86: footprint mouser_AAA3528SEEZGKQBKS:AAA3528SEEZGKQBKS -> XZMDKCBDDG45S-9:PLCC4_SMD-LED_3p2X2p8_SLD; moved to B.Cu
- SW100, SW93: footprint MX_Only:MXOnly-1.5U-Hotswap -> MX_Only:MXOnly-1.25U-Hotswap
- SW104, SW106: footprint MX_Only:MXOnly-2.25U-Hotswap -> MX_Only:MXOnly-2U-Hotswap
- SW53: footprint MX_Only:MXOnly-1U-Hotswap -> MX_Only:MXOnly-1.5U-Hotswap
- SW60: footprint MX_Only:MXOnly-1U-Hotswap -> MX_Only:MXOnly-2U-Hotswap
- SW88: footprint MX_Only:MXOnly-2.25U-Hotswap -> MX_Only:MXOnly-2.75U-Hotswap
- SW94, SW98, SW99: footprint MX_Only:MXOnly-1U-Hotswap -> MX_Only:MXOnly-1.25U-Hotswap
- moved SW106 475.6 mm to (509.6, 192.9), turned to 90 degrees
- moved SW37 394.5 mm to (471.5, 126.2)
- moved SW39 392.2 mm to (509.6, 126.2)
- moved SW55 368.6 mm to (404.8, 145.3)
- moved SW36 357.1 mm to (452.4, 126.2)
- moved SW59 328.0 mm to (490.5, 145.3)
- moved SW56 322.0 mm to (423.9, 145.3)
- moved SW57 320.3 mm to (452.4, 145.3)
- moved SW38 319.5 mm to (490.5, 126.2)
- moved SW33 314.1 mm to (385.8, 126.2)
- moved SW105 310.4 mm to (490.5, 202.4)
- moved SW35 303.3 mm to (423.9, 126.2)
- moved SW58 299.6 mm to (471.5, 145.3)
- moved SW17 281.6 mm to (404.8, 102.4)
- moved SW60 272.7 mm to (509.6, 154.8), turned to 90 degrees
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
Commit message: MCU pins all routed
Just need to finish led drivers and connect matrix
Parts:
- removed C32: 100n, Capacitor_SMD:C_0805_2012Metric_Pad1.18x1.45mm_HandSolder
- removed F2: 2.5, Fuse:Fuse_1206_3216Metric_Pad1.42x1.75mm_HandSolder
- removed LED99: MENU, XZMDKCBDDG45S-9:PLCC4_SMD-LED_3p2X2p8_SLD
- added C33: 100n, Capacitor_SMD:C_0805_2012Metric_Pad1.18x1.45mm_HandSolder, B.Cu at (471.9, 113.2)
- added LED107: MENU, XZMDKCBDDG45S-9:PLCC4_SMD-LED_3p2X2p8_SLD, B.Cu at (323.9, 207.5)
- J1: value ARM 10pin -> Conn_01x03; footprint Connector_PinHeader_1.27mm:PinHeader_2x05_P1.27mm_Horizontal -> Connector_PinHeader_2.54mm:PinHeader_1x03_P2.54mm_Vertical
- LED1, LED100, LED101, LED103, LED104, LED105, LED106, LED2, LED3, LED4, LED5, LED6, LED7, LED8, LED9: moved to B.Cu
- LED10: value F9 -> TILDE; moved to B.Cu
- LED102: value DN_ARROW -> D_ARROW; moved to B.Cu
- LED11: value F10 -> 1; moved to B.Cu
- LED12: value F11 -> 2; moved to B.Cu
- LED13: value F12 -> 3; moved to B.Cu
- LED14: value PRT_SC -> 4; moved to B.Cu
- LED15: value SCR_LK -> 5; moved to B.Cu
- LED16: value PAUSE -> 6; moved to B.Cu
- LED17: value TILDE -> 7; moved to B.Cu
- LED18: value 1 -> 8; moved to B.Cu
- LED19: value 2 -> 9; moved to B.Cu
- LED20: value 3 -> TAB; moved to B.Cu
- LED21: value 4 -> Q; moved to B.Cu
- LED22: value 5 -> W; moved to B.Cu
- LED23: value 6 -> E; moved to B.Cu
- LED24: value 7 -> R; moved to B.Cu
- LED25: value 8 -> T; moved to B.Cu
- LED26: value 9 -> Y; moved to B.Cu
- LED27: value 0 -> U; moved to B.Cu
- LED28: value - -> I; moved to B.Cu
- LED29: value = -> O; moved to B.Cu
- LED30: value BACKSPACE -> CAPS; moved to B.Cu
- LED31: value INSERT -> A; moved to B.Cu
- LED32: value HOME -> S; moved to B.Cu
- LED33: value PG_UP -> D; moved to B.Cu
- LED34: value NUM_LK -> F; moved to B.Cu
- LED35: value PAD_/ -> G; moved to B.Cu
- LED36: value * -> H; moved to B.Cu
- LED37: value PAD_- -> J; moved to B.Cu
- LED38: value TAB -> K; moved to B.Cu
- LED39: value Q -> L; moved to B.Cu
- LED40: value W -> L_SHIFT; moved to B.Cu
- LED41: value E -> Z; moved to B.Cu
- LED42: value R -> X; moved to B.Cu
- LED43: value T -> C; moved to B.Cu
- LED44: value Y -> V; moved to B.Cu
- LED45: value U -> B; moved to B.Cu
- LED46: value I -> N; moved to B.Cu
- LED47: value O -> M; moved to B.Cu
- LED48: value P -> ,; moved to B.Cu
- LED49: value [ -> L_CTRL; moved to B.Cu
- LED50: value ] -> OS; moved to B.Cu
- LED51: value \ -> L_ALT; moved to B.Cu
- LED52: value DEL -> L_SPACE; moved to B.Cu
- LED53: value END -> SPACE; moved to B.Cu
- LED54: value PG_DN -> R_SPACE; moved to B.Cu
- LED55: value PAD_7 -> R_ALT; moved to B.Cu
- LED56: value PAD_8 -> FN; moved to B.Cu
- LED57: value PAD_9 -> F9; moved to B.Cu
- LED58: value + -> F10; moved to B.Cu
- LED59: value CAPS -> F11; moved to B.Cu
- LED60: value A -> F12; moved to B.Cu
- LED61: value S -> PRT_SC; moved to B.Cu
- LED62: value D -> SCR_LK; moved to B.Cu
- LED63: value F -> PAUSE; moved to B.Cu
- LED64: value G -> O; moved to B.Cu
- LED65: value H -> -; moved to B.Cu
- LED66: value J -> =; moved to B.Cu
- LED67: value K -> BACKSPACE; moved to B.Cu
- LED68: value L -> INSERT; moved to B.Cu
- LED69: value ; -> HOME; moved to B.Cu
- LED70: value ' -> PG_UP; moved to B.Cu
- LED71: value ENTER -> NUM_LOCK; moved to B.Cu
- LED72: value PAD_4 -> PAD_/; moved to B.Cu
- LED73: value PAD_5 -> *; moved to B.Cu
- LED74: value PAD_6 -> PAD_-; moved to B.Cu
- LED75: value L_SHIFT -> P; moved to B.Cu
- LED76: value Z -> [; moved to B.Cu
- LED77: value X -> ]; moved to B.Cu
- LED78: value C -> \; moved to B.Cu
- LED79: value V -> DEL; moved to B.Cu
- LED80: value B -> END; moved to B.Cu
- LED81: value N -> PG_DN; moved to B.Cu
- LED82: value M -> PAD_7; moved to B.Cu
- LED83: value , -> PAD_8; moved to B.Cu
- LED84: value . -> PAD_9; moved to B.Cu
- LED85: value / -> +; moved to B.Cu
- LED86: value R_SHIFT -> ;
- LED87: value UP_ARROW -> '; moved to B.Cu
- LED88: value PAD_1 -> ENTER; moved to B.Cu
- LED89: value PAD_2 -> PAD_4; moved to B.Cu
- LED90: value PAD_3 -> PAD_5; moved to B.Cu
- LED91: value CTRL -> PAD_6; moved to B.Cu
- LED92: value OS -> .; moved to B.Cu
- LED93: value L_ALT -> /; moved to B.Cu
- LED94: value SPACE_L -> R_SHIFT; moved to B.Cu
- LED95: value SPACE -> U_ARROW; moved to B.Cu
- LED96: value SPACE_R -> PAD_1; moved to B.Cu
- LED97: value R_ALT -> PAD_2; moved to B.Cu
- LED98: value FN -> PAD_3; moved to B.Cu
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Connections:
- net Net-(D1-I/O1) renamed DP
- net Net-(D1-I/O2) renamed DN
- C11 pad 1: +3.3V -> +1V1
- C30 pad 1: Net-(U5-VI) -> +5V
- F1 pad 2: Net-(U5-VI) -> +5V
- J1 pad 1: +3.3V -> SWCLK
- J1 pad 3: GND -> SWD
- LED1 pad 1: Net-(LED1-K_RED) -> Net-(LED1-R)
- LED1 pad 3: Net-(LED1-K_GREEN) -> Net-(LED1-B)
- LED1 pad 4: Net-(LED1-K_BLUE) -> Net-(LED1-G)
- LED10 pad 1: Net-(LED10-K_RED) -> Net-(LED1-R)
- LED10 pad 2: SW7 -> SW2
- LED10 pad 3: Net-(LED10-K_GREEN) -> Net-(LED1-B)
- LED10 pad 4: Net-(LED10-K_BLUE) -> Net-(LED1-G)
- LED100 pad 1: Net-(LED100-K_RED) -> Net-(LED100-B)
- LED100 pad 3: Net-(LED100-K_GREEN) -> Net-(LED100-B)
- LED100 pad 4: Net-(LED100-K_BLUE) -> Net-(LED100-B)
- LED101 pad 1: Net-(LED101-K_RED) -> Net-(LED101-R)
- LED101 pad 3: Net-(LED101-K_GREEN) -> Net-(LED101-B)
- LED101 pad 4: Net-(LED101-K_BLUE) -> Net-(LED101-G)
- LED102 pad 1: Net-(LED102-K_RED) -> Net-(LED102-R)
- LED102 pad 3: Net-(LED102-K_GREEN) -> Net-(LED102-B)
- LED102 pad 4: Net-(LED102-K_BLUE) -> Net-(LED102-G)
- LED103 pad 1: Net-(LED103-K_RED) -> Net-(LED103-R)
- LED103 pad 3: Net-(LED103-K_GREEN) -> Net-(LED103-B)
- LED103 pad 4: Net-(LED103-K_BLUE) -> Net-(LED103-G)
- LED104 pad 1: Net-(LED104-K_RED) -> Net-(LED104-R)
- LED104 pad 3: Net-(LED104-K_GREEN) -> Net-(LED104-B)
- LED104 pad 4: Net-(LED104-K_BLUE) -> Net-(LED104-G)
- LED105 pad 1: Net-(LED105-K_RED) -> Net-(LED105-R)
- LED105 pad 3: Net-(LED105-K_GREEN) -> Net-(LED105-B)
- LED105 pad 4: Net-(LED105-K_BLUE) -> Net-(LED105-G)
- LED106 pad 1: Net-(LED106-K_RED) -> Net-(LED106-R)
- LED106 pad 3: Net-(LED106-K_GREEN) -> Net-(LED106-B)
- LED106 pad 4: Net-(LED106-K_BLUE) -> Net-(LED106-G)
- LED11 pad 1: Net-(LED100-K_RED) -> Net-(LED11-R)
- LED11 pad 2: SW7 -> SW2
- LED11 pad 3: Net-(LED100-K_GREEN) -> Net-(LED11-B)
- LED11 pad 4: Net-(LED100-K_BLUE) -> Net-(LED11-G)
- LED12 pad 1: Net-(LED12-K_RED) -> Net-(LED12-R)
- LED12 pad 2: SW7 -> SW2
- LED12 pad 3: Net-(LED12-K_GREEN) -> Net-(LED12-B)
- LED12 pad 4: Net-(LED12-K_BLUE) -> Net-(LED12-G)
- LED13 pad 1: Net-(LED13-K_RED) -> Net-(LED13-R)
- LED13 pad 2: SW7 -> SW2
- LED13 pad 3: Net-(LED13-K_GREEN) -> Net-(LED13-B)
- LED13 pad 4: Net-(LED13-K_BLUE) -> Net-(LED13-G)
- LED14 pad 1: Net-(LED101-K_RED) -> Net-(LED14-R)
- LED14 pad 2: SW7 -> SW2
- LED14 pad 3: Net-(LED101-K_GREEN) -> Net-(LED14-B)
- LED14 pad 4: Net-(LED101-K_BLUE) -> Net-(LED14-G)
- LED15 pad 1: Net-(LED102-K_RED) -> Net-(LED15-R)
- LED15 pad 2: SW7 -> SW2
- LED15 pad 3: Net-(LED102-K_GREEN) -> Net-(LED15-B)
- LED15 pad 4: Net-(LED102-K_BLUE) -> Net-(LED15-G)
- LED16 pad 1: Net-(LED103-K_RED) -> Net-(LED16-R)
- LED16 pad 2: SW7 -> SW2
- LED16 pad 3: Net-(LED103-K_GREEN) -> Net-(LED16-B)
- LED16 pad 4: Net-(LED103-K_BLUE) -> Net-(LED16-G)
- LED17 pad 1: Net-(LED1-K_RED) -> Net-(LED17-R)
- LED17 pad 3: Net-(LED1-K_GREEN) -> Net-(LED17-B)
- LED17 pad 4: Net-(LED1-K_BLUE) -> Net-(LED17-G)
- LED18 pad 1: Net-(LED18-K_RED) -> Net-(LED18-R)
- LED18 pad 3: Net-(LED18-K_GREEN) -> Net-(LED18-B)
- LED18 pad 4: Net-(LED18-K_BLUE) -> Net-(LED18-G)
- LED19 pad 1: Net-(LED19-K_RED) -> Net-(LED19-R)
- LED19 pad 3: Net-(LED19-K_GREEN) -> Net-(LED19-B)
- LED19 pad 4: Net-(LED19-K_BLUE) -> Net-(LED19-G)
- LED2 pad 1: Net-(LED19-K_RED) -> Net-(LED12-R)
- LED2 pad 3: Net-(LED19-K_GREEN) -> Net-(LED12-B)
- LED2 pad 4: Net-(LED19-K_BLUE) -> Net-(LED12-G)
- LED20 pad 1: Net-(LED20-K_RED) -> Net-(LED1-R)
- LED20 pad 2: SW2 -> SW3
- LED20 pad 3: Net-(LED20-K_GREEN) -> Net-(LED1-B)
- LED20 pad 4: Net-(LED20-K_BLUE) -> Net-(LED1-G)
- LED21 pad 1: Net-(LED21-K_RED) -> Net-(LED11-R)
- LED21 pad 2: SW2 -> SW3
- LED21 pad 3: Net-(LED21-K_GREEN) -> Net-(LED11-B)
- LED21 pad 4: Net-(LED21-K_BLUE) -> Net-(LED11-G)
- LED22 pad 1: Net-(LED22-K_RED) -> Net-(LED12-R)
- LED22 pad 2: SW2 -> SW3
- LED22 pad 3: Net-(LED22-K_GREEN) -> Net-(LED12-B)
- LED22 pad 4: Net-(LED22-K_BLUE) -> Net-(LED12-G)
- LED23 pad 1: Net-(LED23-K_RED) -> Net-(LED13-R)
- LED23 pad 2: SW2 -> SW3
- LED23 pad 3: Net-(LED23-K_GREEN) -> Net-(LED13-B)
- LED23 pad 4: Net-(LED23-K_BLUE) -> Net-(LED13-G)
- LED24 pad 1: Net-(LED24-K_RED) -> Net-(LED14-R)
- LED24 pad 2: SW2 -> SW3
- LED24 pad 3: Net-(LED24-K_GREEN) -> Net-(LED14-B)
- LED24 pad 4: Net-(LED24-K_BLUE) -> Net-(LED14-G)
- LED25 pad 1: Net-(LED25-K_RED) -> Net-(LED15-R)
- LED25 pad 2: SW2 -> SW3
- LED25 pad 3: Net-(LED25-K_GREEN) -> Net-(LED15-B)
- LED25 pad 4: Net-(LED25-K_BLUE) -> Net-(LED15-G)
- LED26 pad 1: Net-(LED26-K_RED) -> Net-(LED16-R)
- LED26 pad 2: SW2 -> SW3
- LED26 pad 3: Net-(LED26-K_GREEN) -> Net-(LED16-B)
- LED26 pad 4: Net-(LED26-K_BLUE) -> Net-(LED16-G)
- LED27 pad 1: Net-(LED10-K_RED) -> Net-(LED17-R)
- LED27 pad 2: SW8 -> SW3
- LED27 pad 3: Net-(LED10-K_GREEN) -> Net-(LED17-B)
- LED27 pad 4: Net-(LED10-K_BLUE) -> Net-(LED17-G)
- LED28 pad 1: Net-(LED100-K_RED) -> Net-(LED18-R)
- LED28 pad 2: SW8 -> SW3
- LED28 pad 3: Net-(LED100-K_GREEN) -> Net-(LED18-B)
- LED28 pad 4: Net-(LED100-K_BLUE) -> Net-(LED18-G)
- LED29 pad 1: Net-(LED12-K_RED) -> Net-(LED19-R)
- LED29 pad 2: SW8 -> SW3
- LED29 pad 3: Net-(LED12-K_GREEN) -> Net-(LED19-B)
- LED29 pad 4: Net-(LED12-K_BLUE) -> Net-(LED19-G)
- LED3 pad 1: Net-(LED20-K_RED) -> Net-(LED13-R)
- LED3 pad 3: Net-(LED20-K_GREEN) -> Net-(LED13-B)
- LED3 pad 4: Net-(LED20-K_BLUE) -> Net-(LED13-G)
- LED30 pad 1: Net-(LED13-K_RED) -> Net-(LED1-R)
- LED30 pad 2: SW8 -> SW4
- LED30 pad 3: Net-(LED13-K_GREEN) -> Net-(LED1-B)
- LED30 pad 4: Net-(LED13-K_BLUE) -> Net-(LED1-G)
- LED31 pad 1: Net-(LED101-K_RED) -> Net-(LED11-R)
- LED31 pad 2: SW8 -> SW4
- LED31 pad 3: Net-(LED101-K_GREEN) -> Net-(LED11-B)
- LED31 pad 4: Net-(LED101-K_BLUE) -> Net-(LED11-G)
- LED32 pad 1: Net-(LED102-K_RED) -> Net-(LED12-R)
- LED32 pad 2: SW8 -> SW4
- LED32 pad 3: Net-(LED102-K_GREEN) -> Net-(LED12-B)
- LED32 pad 4: Net-(LED102-K_BLUE) -> Net-(LED12-G)
- LED33 pad 1: Net-(LED103-K_RED) -> Net-(LED13-R)
- LED33 pad 2: SW8 -> SW4
- LED33 pad 3: Net-(LED103-K_GREEN) -> Net-(LED13-B)
- LED33 pad 4: Net-(LED103-K_BLUE) -> Net-(LED13-G)
- LED34 pad 1: Net-(LED104-K_RED) -> Net-(LED14-R)
- LED34 pad 2: SW8 -> SW4
- LED34 pad 3: Net-(LED104-K_GREEN) -> Net-(LED14-B)
- LED34 pad 4: Net-(LED104-K_BLUE) -> Net-(LED14-G)
- LED35 pad 1: Net-(LED105-K_RED) -> Net-(LED15-R)
- LED35 pad 2: SW8 -> SW4
- LED35 pad 3: Net-(LED105-K_GREEN) -> Net-(LED15-B)
- LED35 pad 4: Net-(LED105-K_BLUE) -> Net-(LED15-G)
- LED36 pad 1: Net-(LED105-K_RED) -> Net-(LED16-R)
- LED36 pad 2: SW7 -> SW4
- LED36 pad 3: Net-(LED105-K_GREEN) -> Net-(LED16-B)
- LED36 pad 4: Net-(LED105-K_BLUE) -> Net-(LED16-G)
- LED37 pad 1: Net-(LED106-K_RED) -> Net-(LED17-R)
- LED37 pad 2: SW7 -> SW4
- LED37 pad 3: Net-(LED106-K_GREEN) -> Net-(LED17-B)
- LED37 pad 4: Net-(LED106-K_BLUE) -> Net-(LED17-G)
- LED38 pad 1: Net-(LED1-K_RED) -> Net-(LED18-R)
- LED38 pad 2: SW3 -> SW4
- LED38 pad 3: Net-(LED1-K_GREEN) -> Net-(LED18-B)
- LED38 pad 4: Net-(LED1-K_BLUE) -> Net-(LED18-G)
- LED39 pad 1: Net-(LED18-K_RED) -> Net-(LED19-R)
- LED39 pad 2: SW3 -> SW4
- LED39 pad 3: Net-(LED18-K_GREEN) -> Net-(LED19-B)
- LED39 pad 4: Net-(LED18-K_BLUE) -> Net-(LED19-G)
- LED4 pad 1: Net-(LED21-K_RED) -> Net-(LED14-R)
- LED4 pad 3: Net-(LED21-K_GREEN) -> Net-(LED14-B)
- LED4 pad 4: Net-(LED21-K_BLUE) -> Net-(LED14-G)
- LED40 pad 1: Net-(LED19-K_RED) -> Net-(LED1-R)
- LED40 pad 2: SW3 -> SW5
- LED40 pad 3: Net-(LED19-K_GREEN) -> Net-(LED1-B)
- LED40 pad 4: Net-(LED19-K_BLUE) -> Net-(LED1-G)
- LED41 pad 1: Net-(LED20-K_RED) -> Net-(LED12-R)
- LED41 pad 2: SW3 -> SW5
- LED41 pad 3: Net-(LED20-K_GREEN) -> Net-(LED12-B)
- LED41 pad 4: Net-(LED20-K_BLUE) -> Net-(LED12-G)
- LED42 pad 1: Net-(LED21-K_RED) -> Net-(LED13-R)
- LED42 pad 2: SW3 -> SW5
- LED42 pad 3: Net-(LED21-K_GREEN) -> Net-(LED13-B)
- LED42 pad 4: Net-(LED21-K_BLUE) -> Net-(LED13-G)
- LED43 pad 1: Net-(LED22-K_RED) -> Net-(LED14-R)
- LED43 pad 2: SW3 -> SW5
- LED43 pad 3: Net-(LED22-K_GREEN) -> Net-(LED14-B)
- LED43 pad 4: Net-(LED22-K_BLUE) -> Net-(LED14-G)
- LED44 pad 1: Net-(LED23-K_RED) -> Net-(LED15-R)
- LED44 pad 2: SW3 -> SW5
- LED44 pad 3: Net-(LED23-K_GREEN) -> Net-(LED15-B)
- LED44 pad 4: Net-(LED23-K_BLUE) -> Net-(LED15-G)
- LED45 pad 1: Net-(LED24-K_RED) -> Net-(LED16-R)
- LED45 pad 2: SW3 -> SW5
- LED45 pad 3: Net-(LED24-K_GREEN) -> Net-(LED16-B)
- LED45 pad 4: Net-(LED24-K_BLUE) -> Net-(LED16-G)
- LED46 pad 1: Net-(LED25-K_RED) -> Net-(LED17-R)
- LED46 pad 2: SW3 -> SW5
- LED46 pad 3: Net-(LED25-K_GREEN) -> Net-(LED17-B)
- LED46 pad 4: Net-(LED25-K_BLUE) -> Net-(LED17-G)
- LED47 pad 1: Net-(LED26-K_RED) -> Net-(LED18-R)
- LED47 pad 2: SW3 -> SW5
- LED47 pad 3: Net-(LED26-K_GREEN) -> Net-(LED18-B)
- LED47 pad 4: Net-(LED26-K_BLUE) -> Net-(LED18-G)
- LED48 pad 1: Net-(LED10-K_RED) -> Net-(LED19-R)
- LED48 pad 2: SW9 -> SW5
- LED48 pad 3: Net-(LED10-K_GREEN) -> Net-(LED19-B)
- LED48 pad 4: Net-(LED10-K_BLUE) -> Net-(LED19-G)
- LED49 pad 1: Net-(LED100-K_RED) -> Net-(LED1-R)
- LED49 pad 2: SW9 -> SW6
- LED49 pad 3: Net-(LED100-K_GREEN) -> Net-(LED1-B)
- LED49 pad 4: Net-(LED100-K_BLUE) -> Net-(LED1-G)
- LED5 pad 1: Net-(LED22-K_RED) -> Net-(LED15-R)
- LED5 pad 3: Net-(LED22-K_GREEN) -> Net-(LED15-B)
- LED5 pad 4: Net-(LED22-K_BLUE) -> Net-(LED15-G)
- LED50 pad 1: Net-(LED12-K_RED) -> Net-(LED11-R)
- LED50 pad 2: SW9 -> SW6
- LED50 pad 3: Net-(LED12-K_GREEN) -> Net-(LED11-B)
- LED50 pad 4: Net-(LED12-K_BLUE) -> Net-(LED11-G)
- LED51 pad 1: Net-(LED13-K_RED) -> Net-(LED12-R)
- LED51 pad 2: SW9 -> SW6
- LED51 pad 3: Net-(LED13-K_GREEN) -> Net-(LED12-B)
- LED51 pad 4: Net-(LED13-K_BLUE) -> Net-(LED12-G)
- LED52 pad 1: Net-(LED101-K_RED) -> Net-(LED13-R)
- LED52 pad 2: SW9 -> SW6
- LED52 pad 3: Net-(LED101-K_GREEN) -> Net-(LED13-B)
- LED52 pad 4: Net-(LED101-K_BLUE) -> Net-(LED13-G)
- LED53 pad 1: Net-(LED102-K_RED) -> Net-(LED15-R)
- LED53 pad 2: SW9 -> SW6
- LED53 pad 3: Net-(LED102-K_GREEN) -> Net-(LED15-B)
- LED53 pad 4: Net-(LED102-K_BLUE) -> Net-(LED15-G)
- LED54 pad 1: Net-(LED103-K_RED) -> Net-(LED17-R)
- LED54 pad 2: SW9 -> SW6
- LED54 pad 3: Net-(LED103-K_GREEN) -> Net-(LED17-B)
- LED54 pad 4: Net-(LED103-K_BLUE) -> Net-(LED17-G)
- LED55 pad 1: Net-(LED104-K_RED) -> Net-(LED18-R)
- LED55 pad 2: SW9 -> SW6
- LED55 pad 3: Net-(LED104-K_GREEN) -> Net-(LED18-B)
- LED55 pad 4: Net-(LED104-K_BLUE) -> Net-(LED18-G)
- LED56 pad 1: Net-(LED105-K_RED) -> Net-(LED56-R)
- LED56 pad 2: SW9 -> SW12
- LED56 pad 3: Net-(LED105-K_GREEN) -> Net-(LED56-B)
- LED56 pad 4: Net-(LED105-K_BLUE) -> Net-(LED56-G)
- LED57 pad 1: Net-(LED106-K_RED) -> Net-(LED56-R)
- LED57 pad 2: SW9 -> SW7
- LED57 pad 3: Net-(LED106-K_GREEN) -> Net-(LED56-B)
- LED57 pad 4: Net-(LED106-K_BLUE) -> Net-(LED56-G)
- LED58 pad 1: Net-(LED106-K_RED) -> Net-(LED107-R)
- LED58 pad 2: SW8 -> SW7
- LED58 pad 3: Net-(LED106-K_GREEN) -> Net-(LED107-B)
- LED58 pad 4: Net-(LED106-K_BLUE) -> Net-(LED107-G)
- LED59 pad 1: Net-(LED1-K_RED) -> Net-(LED59-R)
- LED59 pad 2: SW4 -> SW7
- LED59 pad 3: Net-(LED1-K_GREEN) -> Net-(LED59-B)
- LED59 pad 4: Net-(LED1-K_BLUE) -> Net-(LED59-G)
- LED6 pad 1: Net-(LED23-K_RED) -> Net-(LED16-R)
- LED6 pad 3: Net-(LED23-K_GREEN) -> Net-(LED16-B)
- LED6 pad 4: Net-(LED23-K_BLUE) -> Net-(LED16-G)
- LED60 pad 1: Net-(LED18-K_RED) -> Net-(LED100-B)
- LED60 pad 2: SW4 -> SW7
- LED60 pad 3: Net-(LED18-K_GREEN) -> Net-(LED100-B)
- LED60 pad 4: Net-(LED18-K_BLUE) -> Net-(LED100-B)
- LED61 pad 1: Net-(LED19-K_RED) -> Net-(LED101-R)
- LED61 pad 2: SW4 -> SW7
- LED61 pad 3: Net-(LED19-K_GREEN) -> Net-(LED101-B)
- LED61 pad 4: Net-(LED19-K_BLUE) -> Net-(LED101-G)
- LED62 pad 1: Net-(LED20-K_RED) -> Net-(LED102-R)
- LED62 pad 2: SW4 -> SW7
- LED62 pad 3: Net-(LED20-K_GREEN) -> Net-(LED102-B)
- LED62 pad 4: Net-(LED20-K_BLUE) -> Net-(LED102-G)
- LED63 pad 1: Net-(LED21-K_RED) -> Net-(LED103-R)
- LED63 pad 2: SW4 -> SW7
- LED63 pad 3: Net-(LED21-K_GREEN) -> Net-(LED103-B)
- LED63 pad 4: Net-(LED21-K_BLUE) -> Net-(LED103-G)
- LED64 pad 1: Net-(LED22-K_RED) -> Net-(LED56-R)
- LED64 pad 2: SW4 -> SW8
- LED64 pad 3: Net-(LED22-K_GREEN) -> Net-(LED56-B)
- LED64 pad 4: Net-(LED22-K_BLUE) -> Net-(LED56-G)
- LED65 pad 1: Net-(LED23-K_RED) -> Net-(LED107-R)
- LED65 pad 2: SW4 -> SW8
- LED65 pad 3: Net-(LED23-K_GREEN) -> Net-(LED107-B)
- LED65 pad 4: Net-(LED23-K_BLUE) -> Net-(LED107-G)
- LED66 pad 1: Net-(LED24-K_RED) -> Net-(LED59-R)
- LED66 pad 2: SW4 -> SW8
- LED66 pad 3: Net-(LED24-K_GREEN) -> Net-(LED59-B)
- LED66 pad 4: Net-(LED24-K_BLUE) -> Net-(LED59-G)
- LED67 pad 1: Net-(LED25-K_RED) -> Net-(LED100-B)
- LED67 pad 2: SW4 -> SW8
- LED67 pad 3: Net-(LED25-K_GREEN) -> Net-(LED100-B)
- LED67 pad 4: Net-(LED25-K_BLUE) -> Net-(LED100-B)
- LED68 pad 1: Net-(LED26-K_RED) -> Net-(LED101-R)
- LED68 pad 2: SW4 -> SW8
- LED68 pad 3: Net-(LED26-K_GREEN) -> Net-(LED101-B)
- LED68 pad 4: Net-(LED26-K_BLUE) -> Net-(LED101-G)
- LED69 pad 1: Net-(LED10-K_RED) -> Net-(LED102-R)
- LED69 pad 2: SW10 -> SW8
- LED69 pad 3: Net-(LED10-K_GREEN) -> Net-(LED102-B)
- LED69 pad 4: Net-(LED10-K_BLUE) -> Net-(LED102-G)
- LED7 pad 1: Net-(LED24-K_RED) -> Net-(LED17-R)
- LED7 pad 3: Net-(LED24-K_GREEN) -> Net-(LED17-B)
- LED7 pad 4: Net-(LED24-K_BLUE) -> Net-(LED17-G)
- LED70 pad 1: Net-(LED100-K_RED) -> Net-(LED103-R)
- LED70 pad 2: SW10 -> SW8
- LED70 pad 3: Net-(LED100-K_GREEN) -> Net-(LED103-B)
- LED70 pad 4: Net-(LED100-K_BLUE) -> Net-(LED103-G)
- LED71 pad 1: Net-(LED13-K_RED) -> Net-(LED104-R)
- LED71 pad 2: SW10 -> SW8
- LED71 pad 3: Net-(LED13-K_GREEN) -> Net-(LED104-B)
- LED71 pad 4: Net-(LED13-K_BLUE) -> Net-(LED104-G)
- LED72 pad 1: Net-(LED104-K_RED) -> Net-(LED105-R)
- LED72 pad 2: SW10 -> SW8
- LED72 pad 3: Net-(LED104-K_GREEN) -> Net-(LED105-B)
- LED72 pad 4: Net-(LED104-K_BLUE) -> Net-(LED105-G)
- LED73 pad 1: Net-(LED105-K_RED) -> Net-(LED105-R)
- LED73 pad 2: SW10 -> SW7
- LED73 pad 3: Net-(LED105-K_GREEN) -> Net-(LED105-B)
- LED73 pad 4: Net-(LED105-K_BLUE) -> Net-(LED105-G)
- LED74 pad 1: Net-(LED106-K_RED) -> Net-(LED106-R)
- LED74 pad 2: SW10 -> SW7
- LED74 pad 3: Net-(LED106-K_GREEN) -> Net-(LED106-B)
- LED74 pad 4: Net-(LED106-K_BLUE) -> Net-(LED106-G)
- LED75 pad 1: Net-(LED1-K_RED) -> Net-(LED56-R)
- LED75 pad 2: SW5 -> SW9
- LED75 pad 3: Net-(LED1-K_GREEN) -> Net-(LED56-B)
- LED75 pad 4: Net-(LED1-K_BLUE) -> Net-(LED56-G)
- LED76 pad 1: Net-(LED19-K_RED) -> Net-(LED107-R)
- LED76 pad 2: SW5 -> SW9
- LED76 pad 3: Net-(LED19-K_GREEN) -> Net-(LED107-B)
- LED76 pad 4: Net-(LED19-K_BLUE) -> Net-(LED107-G)
- LED77 pad 1: Net-(LED20-K_RED) -> Net-(LED59-R)
- LED77 pad 2: SW5 -> SW9
- LED77 pad 3: Net-(LED20-K_GREEN) -> Net-(LED59-B)
- LED77 pad 4: Net-(LED20-K_BLUE) -> Net-(LED59-G)
- LED78 pad 1: Net-(LED21-K_RED) -> Net-(LED100-B)
- LED78 pad 2: SW5 -> SW9
- LED78 pad 3: Net-(LED21-K_GREEN) -> Net-(LED100-B)
- LED78 pad 4: Net-(LED21-K_BLUE) -> Net-(LED100-B)
- LED79 pad 1: Net-(LED22-K_RED) -> Net-(LED101-R)
- LED79 pad 2: SW5 -> SW9
- LED79 pad 3: Net-(LED22-K_GREEN) -> Net-(LED101-B)
- LED79 pad 4: Net-(LED22-K_BLUE) -> Net-(LED101-G)
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Routing:
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Other:
- board text added: "LED10"

Commit message: Started Routing LED Drivers
Parts:
- moved R_B11 81.1 mm to (300.5, 212.0), turned to 90 degrees
- moved R_G11 67.6 mm to (304.8, 212.0), turned to 90 degrees
- moved R_R11 59.8 mm to (302.6, 212.0), turned to 90 degrees
- moved C19 9.24 mm to (423.2, 159.0)
- moved C16 9.12 mm to (425.4, 159.0)
- moved R13 9.09 mm to (412.6, 160.7)
- moved C21 8.09 mm to (424.2, 164.5), turned to 0 degrees
- moved C23 7.45 mm to (424.2, 162.2), turned to 0 degrees
- moved R9 5.76 mm to (411.8, 156.8)
- moved C29 5.42 mm to (413.9, 156.8)
- moved R11 5.12 mm to (410.6, 163.2), turned to 90 degrees
- moved C15 4.49 mm to (430.3, 171.6), turned to -90 degrees
- moved R10 4.36 mm to (412.6, 164.4), turned to 90 degrees
- moved R12 3.70 mm to (420.2, 160.0), turned to 180 degrees
- moved R4 2.99 mm to (377.2, 160.3), turned to 0 degrees
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Routing:
- net ROW4: track 138.9 -> 565.3 mm, vias 0 -> 1
- net SW11: track 0.00 -> 258.1 mm, vias 0 -> 7
- net SDA: track 50.9 -> 175.2 mm, vias 2 -> 4
- net INTB: track 91.1 -> 204.5 mm, vias 2 -> 4
- net SCL: track 60.6 -> 158.1 mm, vias 2 -> 4
- net SDB: track 96.5 -> 191.7 mm, vias 2 -> 4
- net Net-(LED103-G): track 0.00 -> 80.0 mm
- net COL16: track 195.4 -> 275.0 mm
- net Net-(LED101-B): track 0.00 -> 76.4 mm
- net +5V: track 134.6 -> 204.7 mm, vias 2 -> 7
- net Net-(LED103-B): track 0.00 -> 70.0 mm
- net Net-(LED102-G): track 0.00 -> 68.0 mm
- net Net-(LED101-G): track 0.00 -> 65.8 mm
- net Net-(LED102-B): track 0.00 -> 65.0 mm
- net SW12: track 0.00 -> 51.7 mm, vias 0 -> 1
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
Commit message: Began Routing Columns and Rows
Parts:
- removed LED107: MENU, XZMDKCBDDG45S-9:PLCC4_SMD-LED_3p2X2p8_SLD
- added LED99: MENU, XZMDKCBDDG45S-9:PLCC4_SMD-LED_3p2X2p8_SLD, B.Cu at (323.9, 207.4)
- F1: value 500m -> 2.5
- LED49: value L_CTRL -> SPACE
- LED50: value OS -> L_CTRL
- LED51: value L_ALT -> OS
- LED52: value L_SPACE -> L_ALT
- LED53: value SPACE -> L_SPACE
- LED56: value FN -> F9
- LED57: value F9 -> F10
- LED58: value F10 -> F11
- LED59: value F11 -> F12
- LED60: value F12 -> PRT_SC
- LED61: value PRT_SC -> SCR_LK
- LED62: value SCR_LK -> PAUSE
- LED63: value PAUSE -> O
- LED64: value O -> -
- LED65: value - -> =
- LED66: value = -> BACKSPACE
- LED67: value BACKSPACE -> INSERT
- LED68: value INSERT -> HOME
- LED69: value HOME -> PG_UP
- LED70: value PG_UP -> NUM_LOCK
- LED71: value NUM_LOCK -> PAD_/
- LED72: value PAD_/ -> *
- LED73: value * -> PAD_-
- LED74: value PAD_- -> P
- LED75: value P -> [
- LED76: value [ -> ]
- LED77: value ] -> \
- LED78: value \ -> DEL
- LED79: value DEL -> END
- LED80: value END -> PG_DN
- LED81: value PG_DN -> PAD_7
- LED82: value PAD_7 -> PAD_8
- LED83: value PAD_8 -> PAD_9
- LED84: value PAD_9 -> +
- LED85: value + -> ;
- LED86: value ; -> '
- LED87: value ' -> ENTER
- LED88: value ENTER -> PAD_4
- LED89: value PAD_4 -> PAD_5
- LED90: value PAD_5 -> PAD_6
- LED91: value PAD_6 -> .
- LED92: value . -> /
- LED93: value / -> R_SHIFT
- LED94: value R_SHIFT -> U_ARROW
- LED95: value U_ARROW -> PAD_1
- LED96: value PAD_1 -> PAD_2
- LED97: value PAD_2 -> PAD_3
- LED98: value PAD_3 -> FN
- moved R_B1 275.1 mm to (91.7, 209.9), turned to 90 degrees
- moved R_B2 268.6 mm to (101.9, 210.6), turned to 0 degrees
- moved R_G1 268.4 mm to (96.3, 209.9), turned to 90 degrees
- moved R_R1 268.1 mm to (94.1, 209.9), turned to 90 degrees
- moved R_G2 256.9 mm to (117.7, 206.2), turned to 180 degrees
- moved R_R2 254.7 mm to (117.7, 208.4), turned to 180 degrees
- moved R_B3 247.3 mm to (125.7, 210.4), turned to 0 degrees
- moved R_B4 221.5 mm to (152.1, 206.9), turned to 0 degrees
- moved R_G3 221.0 mm to (142.6, 206.8)
- moved R_R3 219.4 mm to (142.6, 209.0)
- moved LED74 217.5 mm to (283.5, 150.4)
- moved LED85 217.1 mm to (288.0, 169.2), turned to 180 degrees
- moved R_B5 213.8 mm to (161.8, 195.2), turned to -90 degrees
- moved LED91 203.1 mm to (278.6, 188.3)
- moved R_G5 197.1 mm to (168.8, 195.3), turned to -90 degrees
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Connections:
- LED100 pad 1: Net-(LED100-B) -> Net-(LED100-R)
- LED100 pad 4: Net-(LED100-B) -> Net-(LED100-G)
- LED49 pad 1: Net-(LED1-R) -> Net-(LED16-R)
- LED49 pad 3: Net-(LED1-B) -> Net-(LED16-B)
- LED49 pad 4: Net-(LED1-G) -> Net-(LED16-G)
- LED50 pad 1: Net-(LED11-R) -> Net-(LED1-R)
- LED50 pad 3: Net-(LED11-B) -> Net-(LED1-B)
- LED50 pad 4: Net-(LED11-G) -> Net-(LED1-G)
- LED51 pad 1: Net-(LED12-R) -> Net-(LED11-R)
- LED51 pad 3: Net-(LED12-B) -> Net-(LED11-B)
- LED51 pad 4: Net-(LED12-G) -> Net-(LED11-G)
- LED52 pad 1: Net-(LED13-R) -> Net-(LED12-R)
- LED52 pad 3: Net-(LED13-B) -> Net-(LED12-B)
- LED52 pad 4: Net-(LED13-G) -> Net-(LED12-G)
- LED53 pad 1: Net-(LED15-R) -> Net-(LED13-R)
- LED53 pad 3: Net-(LED15-B) -> Net-(LED13-B)
- LED53 pad 4: Net-(LED15-G) -> Net-(LED13-G)
- LED54 pad 1: Net-(LED17-R) -> Net-(LED18-R)
- LED54 pad 3: Net-(LED17-B) -> Net-(LED18-B)
- LED54 pad 4: Net-(LED17-G) -> Net-(LED18-G)
- LED55 pad 1: Net-(LED18-R) -> Net-(LED55-R)
- LED55 pad 2: SW6 -> SW12
- LED55 pad 3: Net-(LED18-B) -> Net-(LED55-B)
- LED55 pad 4: Net-(LED18-G) -> Net-(LED55-G)
- LED56 pad 1: Net-(LED56-R) -> Net-(LED55-R)
- LED56 pad 2: SW12 -> SW7
- LED56 pad 3: Net-(LED56-B) -> Net-(LED55-B)
- LED56 pad 4: Net-(LED56-G) -> Net-(LED55-G)
- LED57 pad 1: Net-(LED56-R) -> Net-(LED57-R)
- LED57 pad 3: Net-(LED56-B) -> Net-(LED57-B)
- LED57 pad 4: Net-(LED56-G) -> Net-(LED57-G)
- LED58 pad 1: Net-(LED107-R) -> Net-(LED58-R)
- LED58 pad 3: Net-(LED107-B) -> Net-(LED58-B)
- LED58 pad 4: Net-(LED107-G) -> Net-(LED58-G)
- LED59 pad 1: Net-(LED59-R) -> Net-(LED100-R)
- LED59 pad 3: Net-(LED59-B) -> Net-(LED100-B)
- LED59 pad 4: Net-(LED59-G) -> Net-(LED100-G)
- LED60 pad 1: Net-(LED100-B) -> Net-(LED101-R)
- LED60 pad 3: Net-(LED100-B) -> Net-(LED101-B)
- LED60 pad 4: Net-(LED100-B) -> Net-(LED101-G)
- LED61 pad 1: Net-(LED101-R) -> Net-(LED102-R)
- LED61 pad 3: Net-(LED101-B) -> Net-(LED102-B)
- LED61 pad 4: Net-(LED101-G) -> Net-(LED102-G)
- LED62 pad 1: Net-(LED102-R) -> Net-(LED103-R)
- LED62 pad 3: Net-(LED102-B) -> Net-(LED103-B)
- LED62 pad 4: Net-(LED102-G) -> Net-(LED103-G)
- LED63 pad 1: Net-(LED103-R) -> Net-(LED55-R)
- LED63 pad 2: SW7 -> SW8
- LED63 pad 3: Net-(LED103-B) -> Net-(LED55-B)
- LED63 pad 4: Net-(LED103-G) -> Net-(LED55-G)
- LED64 pad 1: Net-(LED56-R) -> Net-(LED57-R)
- LED64 pad 3: Net-(LED56-B) -> Net-(LED57-B)
- LED64 pad 4: Net-(LED56-G) -> Net-(LED57-G)
- LED65 pad 1: Net-(LED107-R) -> Net-(LED58-R)
- LED65 pad 3: Net-(LED107-B) -> Net-(LED58-B)
- LED65 pad 4: Net-(LED107-G) -> Net-(LED58-G)
- LED66 pad 1: Net-(LED59-R) -> Net-(LED100-R)
- LED66 pad 3: Net-(LED59-B) -> Net-(LED100-B)
- LED66 pad 4: Net-(LED59-G) -> Net-(LED100-G)
- LED67 pad 1: Net-(LED100-B) -> Net-(LED101-R)
- LED67 pad 3: Net-(LED100-B) -> Net-(LED101-B)
- LED67 pad 4: Net-(LED100-B) -> Net-(LED101-G)
- LED68 pad 1: Net-(LED101-R) -> Net-(LED102-R)
- LED68 pad 3: Net-(LED101-B) -> Net-(LED102-B)
- LED68 pad 4: Net-(LED101-G) -> Net-(LED102-G)
- LED69 pad 1: Net-(LED102-R) -> Net-(LED103-R)
- LED69 pad 3: Net-(LED102-B) -> Net-(LED103-B)
- LED69 pad 4: Net-(LED102-G) -> Net-(LED103-G)
- LED70 pad 1: Net-(LED103-R) -> Net-(LED104-R)
- LED70 pad 3: Net-(LED103-B) -> Net-(LED104-B)
- LED70 pad 4: Net-(LED103-G) -> Net-(LED104-G)
- LED71 pad 1: Net-(LED104-R) -> Net-(LED105-R)
- LED71 pad 3: Net-(LED104-B) -> Net-(LED105-B)
- LED71 pad 4: Net-(LED104-G) -> Net-(LED105-G)
- LED72 pad 2: SW8 -> SW7
- LED73 pad 1: Net-(LED105-R) -> Net-(LED106-R)
- LED73 pad 3: Net-(LED105-B) -> Net-(LED106-B)
- LED73 pad 4: Net-(LED105-G) -> Net-(LED106-G)
- LED74 pad 1: Net-(LED106-R) -> Net-(LED55-R)
- LED74 pad 2: SW7 -> SW9
- LED74 pad 3: Net-(LED106-B) -> Net-(LED55-B)
- LED74 pad 4: Net-(LED106-G) -> Net-(LED55-G)
- LED75 pad 1: Net-(LED56-R) -> Net-(LED57-R)
- LED75 pad 3: Net-(LED56-B) -> Net-(LED57-B)
- LED75 pad 4: Net-(LED56-G) -> Net-(LED57-G)
- LED76 pad 1: Net-(LED107-R) -> Net-(LED58-R)
- LED76 pad 3: Net-(LED107-B) -> Net-(LED58-B)
- LED76 pad 4: Net-(LED107-G) -> Net-(LED58-G)
- LED77 pad 1: Net-(LED59-R) -> Net-(LED100-R)
- LED77 pad 3: Net-(LED59-B) -> Net-(LED100-B)
- LED77 pad 4: Net-(LED59-G) -> Net-(LED100-G)
- LED78 pad 1: Net-(LED100-B) -> Net-(LED101-R)
- LED78 pad 3: Net-(LED100-B) -> Net-(LED101-B)
- LED78 pad 4: Net-(LED100-B) -> Net-(LED101-G)
- LED79 pad 1: Net-(LED101-R) -> Net-(LED102-R)
- LED79 pad 3: Net-(LED101-B) -> Net-(LED102-B)
- LED79 pad 4: Net-(LED101-G) -> Net-(LED102-G)
- LED80 pad 1: Net-(LED102-R) -> Net-(LED103-R)
- LED80 pad 3: Net-(LED102-B) -> Net-(LED103-B)
- LED80 pad 4: Net-(LED102-G) -> Net-(LED103-G)
- LED81 pad 1: Net-(LED103-R) -> Net-(LED104-R)
- LED81 pad 3: Net-(LED103-B) -> Net-(LED104-B)
- LED81 pad 4: Net-(LED103-G) -> Net-(LED104-G)
- LED82 pad 1: Net-(LED104-R) -> Net-(LED105-R)
- LED82 pad 3: Net-(LED104-B) -> Net-(LED105-B)
- LED82 pad 4: Net-(LED104-G) -> Net-(LED105-G)
- LED83 pad 1: Net-(LED105-R) -> Net-(LED106-R)
- LED83 pad 3: Net-(LED105-B) -> Net-(LED106-B)
- LED83 pad 4: Net-(LED105-G) -> Net-(LED106-G)
- LED84 pad 2: SW9 -> SW8
- LED85 pad 1: Net-(LED106-R) -> Net-(LED55-R)
- LED85 pad 2: SW8 -> SW10
- LED85 pad 3: Net-(LED106-B) -> Net-(LED55-B)
- LED85 pad 4: Net-(LED106-G) -> Net-(LED55-G)
- LED86 pad 1: Net-(LED56-R) -> Net-(LED57-R)
- LED86 pad 3: Net-(LED56-B) -> Net-(LED57-B)
- LED86 pad 4: Net-(LED56-G) -> Net-(LED57-G)
- LED87 pad 1: Net-(LED107-R) -> Net-(LED100-R)
- LED87 pad 3: Net-(LED107-B) -> Net-(LED100-B)
- LED87 pad 4: Net-(LED107-G) -> Net-(LED100-G)
- LED88 pad 1: Net-(LED100-B) -> Net-(LED104-R)
- LED88 pad 3: Net-(LED100-B) -> Net-(LED104-B)
- LED88 pad 4: Net-(LED100-B) -> Net-(LED104-G)
- LED89 pad 1: Net-(LED104-R) -> Net-(LED105-R)
- LED89 pad 3: Net-(LED104-B) -> Net-(LED105-B)
- LED89 pad 4: Net-(LED104-G) -> Net-(LED105-G)
- LED90 pad 1: Net-(LED105-R) -> Net-(LED106-R)
- LED90 pad 3: Net-(LED105-B) -> Net-(LED106-B)
- LED90 pad 4: Net-(LED105-G) -> Net-(LED106-G)
- LED91 pad 1: Net-(LED106-R) -> Net-(LED55-R)
- LED91 pad 2: SW10 -> SW11
- LED91 pad 3: Net-(LED106-B) -> Net-(LED55-B)
- LED91 pad 4: Net-(LED106-G) -> Net-(LED55-G)
- LED92 pad 1: Net-(LED56-R) -> Net-(LED57-R)
- LED92 pad 3: Net-(LED56-B) -> Net-(LED57-B)
- LED92 pad 4: Net-(LED56-G) -> Net-(LED57-G)
- LED93 pad 1: Net-(LED107-R) -> Net-(LED100-R)
- LED93 pad 3: Net-(LED107-B) -> Net-(LED100-B)
- LED93 pad 4: Net-(LED107-G) -> Net-(LED100-G)
- LED94 pad 1: Net-(LED100-B) -> Net-(LED102-R)
- LED94 pad 3: Net-(LED100-B) -> Net-(LED102-B)
- LED94 pad 4: Net-(LED100-B) -> Net-(LED102-G)
- LED95 pad 1: Net-(LED102-R) -> Net-(LED104-R)
- LED95 pad 3: Net-(LED102-B) -> Net-(LED104-B)
- LED95 pad 4: Net-(LED102-G) -> Net-(LED104-G)
- LED96 pad 1: Net-(LED104-R) -> Net-(LED105-R)
- LED96 pad 3: Net-(LED104-B) -> Net-(LED105-B)
- LED96 pad 4: Net-(LED104-G) -> Net-(LED105-G)
- LED97 pad 1: Net-(LED105-R) -> Net-(LED106-R)
- LED97 pad 3: Net-(LED105-B) -> Net-(LED106-B)
- LED97 pad 4: Net-(LED105-G) -> Net-(LED106-G)
- LED98 pad 1: Net-(LED106-R) -> Net-(LED57-R)
- LED98 pad 2: SW11 -> SW12
- LED98 pad 3: Net-(LED106-B) -> Net-(LED57-B)
- LED98 pad 4: Net-(LED106-G) -> Net-(LED57-G)
- R12 pad 1: Net-(U4-ISET) -> GND
- R12 pad 2: GND -> Net-(U4-ISET)
- R_B11 pad 1: CS33 -> CS60
- R_B11 pad 2: Net-(LED56-B) -> Net-(LED55-B)
- R_B12 pad 1: CS36 -> CS57
- R_B12 pad 2: Net-(LED107-B) -> Net-(LED57-B)
- R_B13 pad 1: CS39 -> CS54
- R_B13 pad 2: Net-(LED59-B) -> Net-(LED58-B)
- R_B14 pad 1: CS42 -> CS51
- R_B15 pad 1: CS45 -> CS48
- R_B16 pad 1: CS48 -> CS45
- R_B17 pad 1: CS51 -> CS42
- R_B18 pad 1: CS54 -> CS31
- R_B19 pad 1: CS57 -> CS34
- R_B20 pad 1: CS60 -> CS39
- R_G11 pad 1: CS31 -> CS58
- R_G11 pad 2: Net-(LED56-G) -> Net-(LED55-G)
- R_G12 pad 1: CS34 -> CS55
- R_G12 pad 2: Net-(LED107-G) -> Net-(LED57-G)
- R_G13 pad 1: CS37 -> CS52
- R_G13 pad 2: Net-(LED59-G) -> Net-(LED58-G)
- R_G14 pad 1: CS40 -> CS49
- R_G14 pad 2: Net-(LED100-B) -> Net-(LED100-G)
- R_G15 pad 1: CS43 -> CS46
- R_G16 pad 1: CS46 -> CS43
- R_G17 pad 1: CS49 -> CS40
- R_G18 pad 1: CS52 -> CS33
- R_G19 pad 1: CS55 -> CS36
- R_G20 pad 1: CS58 -> CS38
- R_R11 pad 1: CS32 -> CS59
- R_R11 pad 2: Net-(LED56-R) -> Net-(LED55-R)
- R_R12 pad 1: CS35 -> CS56
- R_R12 pad 2: Net-(LED107-R) -> Net-(LED57-R)
- R_R13 pad 1: CS38 -> CS53
- R_R13 pad 2: Net-(LED59-R) -> Net-(LED58-R)
- R_R14 pad 1: CS41 -> CS50
- R_R14 pad 2: Net-(LED100-B) -> Net-(LED100-R)
- R_R15 pad 1: CS44 -> CS47
- R_R16 pad 1: CS47 -> CS44
- R_R17 pad 1: CS50 -> CS41
- R_R18 pad 1: CS53 -> CS32
- R_R19 pad 1: CS56 -> CS35
- R_R20 pad 1: CS59 -> CS37
Routing:
- net ROW5: track 163.5 -> 663.5 mm, vias 1 -> 11
- net ROW0: track 2.46 -> 459.1 mm, vias 1 -> 4
- net ROW1: track 74.0 -> 512.6 mm, vias 0 -> 2
- net ROW3: track 119.1 -> 550.5 mm, vias 0 -> 2
- net ROW2: track 95.5 -> 523.2 mm, vias 1 -> 3
- net SW8: track 40.1 -> 321.4 mm, vias 0 -> 2
- net SW7: track 47.3 -> 324.2 mm, vias 0 -> 3
- net SW1: track 0.00 -> 268.5 mm, vias 0 -> 2
- net SW12: track 51.7 -> 317.7 mm, vias 1 -> 10
- net SW5: track 0.00 -> 199.5 mm, vias 0 -> 4
- net SW3: track 0.00 -> 186.0 mm, vias 0 -> 3
- net SW6: track 0.00 -> 181.5 mm, vias 0 -> 6
- net SW2: track 0.00 -> 179.6 mm, vias 0 -> 2
- net Net-(LED106-R): track 0.00 -> 177.3 mm, vias 0 -> 11
- net Net-(LED1-R): track 0.00 -> 169.8 mm, vias 1 -> 10
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
Commit message: Right LED Driver almost connected
Parts:
- moved R_G17 2.25 mm to (422.5, 204.0), turned to -90 degrees
- moved D89 0.85 mm to (436.5, 187.2)
- moved R_R17 0.51 mm to (421.4, 208.3)
- moved R_G16 0.11 mm to (403.0, 206.1)
Connections:
- R_B1 pad 1: CS3 -> CS1
- R_B10 pad 1: CS30 -> CS28
- R_B11 pad 1: CS60 -> CS40
- R_B12 pad 1: CS57 -> CS43
- R_B13 pad 1: CS54 -> CS46
- R_B14 pad 1: CS51 -> CS49
- R_B15 pad 1: CS48 -> CS52
- R_B16 pad 1: CS45 -> CS55
- R_B17 pad 1: CS42 -> CS58
- R_B2 pad 1: CS6 -> CS4
- R_B3 pad 1: CS9 -> CS7
- R_B4 pad 1: CS12 -> CS10
- R_B5 pad 1: CS15 -> CS13
- R_B6 pad 1: CS18 -> CS16
- R_B7 pad 1: CS21 -> CS19
- R_B8 pad 1: CS24 -> CS22
- R_B9 pad 1: CS27 -> CS25
- R_G1 pad 1: CS1 -> CS3
- R_G10 pad 1: CS28 -> CS30
- R_G11 pad 1: CS58 -> CS42
- R_G12 pad 1: CS55 -> CS45
- R_G13 pad 1: CS52 -> CS48
- R_G14 pad 1: CS49 -> CS51
- R_G15 pad 1: CS46 -> CS54
- R_G16 pad 1: CS43 -> CS57
- R_G17 pad 1: CS40 -> CS60
- R_G2 pad 1: CS4 -> CS6
- R_G3 pad 1: CS7 -> CS9
- R_G4 pad 1: CS10 -> CS12
- R_G5 pad 1: CS13 -> CS15
- R_G6 pad 1: CS16 -> CS18
- R_G7 pad 1: CS19 -> CS21
- R_G8 pad 1: CS22 -> CS24
- R_G9 pad 1: CS25 -> CS27
- R_R11 pad 1: CS59 -> CS41
- R_R12 pad 1: CS56 -> CS44
- R_R13 pad 1: CS53 -> CS47
- R_R15 pad 1: CS47 -> CS53
- R_R16 pad 1: CS44 -> CS56
- R_R17 pad 1: CS41 -> CS59
Routing:
- net CS45: track 0.00 -> 174.1 mm
- net CS44: track 0.00 -> 172.6 mm
- net CS46: track 0.00 -> 160.0 mm
- net CS48: track 3.78 -> 150.1 mm
- net CS47: track 3.09 -> 146.8 mm
- net Net-(LED100-B): track 0.00 -> 139.8 mm
- net CS49: track 4.56 -> 138.9 mm
- net CS50: track 5.25 -> 122.7 mm
- net Net-(LED100-G): track 0.00 -> 115.6 mm
- net Net-(LED103-R): track 0.00 -> 85.0 mm, vias 0 -> 4
- net CS51: track 50.7 -> 123.6 mm
- net CS52: track 51.4 -> 108.3 mm
- net CS54: track 52.6 -> 97.9 mm
- net CS53: track 52.1 -> 96.4 mm
- net CS55: track 53.1 -> 88.8 mm
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