File: KB-pcb-practice.kicad_pcb (KiCad board)
At the start: 2 copper layers, 430 parts, among them J1 Conn_01x03, SW1 Reset, SW10 F7, SW100 R_CTRL, SW101 L_ARROW, SW102 DN_ARROW, SW103 R_ARROW, SW104 PAD_0, SW105 PAD_., SW106 PAD_ENTER, SW11 F8, SW12 F9, SW13 F10, SW14 F11, SW15 F12, SW16 PRT_SC, SW17 SCR_LK, SW18 PAUSE, SW19 TILDE, SW2 Boot, SW20 1, SW21 2, SW22 3, SW23 4, SW24 5, SW25 6, SW26 7, SW27 8, SW28 9, SW29 0, SW3 ESC, SW30 -, SW31 =, SW32 BACKSPACE, SW33 INSERT, SW34 HOME, SW35 PG_UP, SW36 NUM_LK, SW37 PAD_/, SW38 *, SW39 PAD_-, SW4 F1, SW40 TAB, SW41 Q, SW42 W, SW43 E, SW44 R, SW45 T, SW46 Y, SW47 U, SW48 I, SW49 O, SW5 F2, SW50 P, SW51 [, SW52 ], SW53 \, SW54 DEL, SW55 END, SW56 PG_DN, SW57 PAD_7, SW58 PAD_8, SW59 PAD_9, SW6 F3, SW60 +, SW61 CAPS, SW62 A, SW63 S, SW64 D, SW65 F, SW66 G, SW67 H, SW68 J, SW69 K, SW7 F4, SW70 L, SW71 ;, SW72 ', SW73 ENTER, SW74 PAD_4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

Commit message: Added RGB Underglow
Parts:
- removed R17: 27, Resistor_SMD:R_0805_2012Metric_Pad1.20x1.40mm_HandSolder
- added C18: 104, Capacitor_SMD:C_0805_2012Metric_Pad1.18x1.45mm_HandSolder, B.Cu at (76.8, 146.3)
- added C32: 104, Capacitor_SMD:C_0805_2012Metric_Pad1.18x1.45mm_HandSolder, B.Cu at (76.6, 169.0)
- added C34: 104, Capacitor_SMD:C_0805_2012Metric_Pad1.18x1.45mm_HandSolder, B.Cu at (102.9, 90.8)
- added C35: 104, Capacitor_SMD:C_0805_2012Metric_Pad1.18x1.45mm_HandSolder, B.Cu at (192.7, 92.6)
- added C36: 104, Capacitor_SMD:C_0805_2012Metric_Pad1.18x1.45mm_HandSolder, B.Cu at (278.3, 92.3)
- added C37: 104, Capacitor_SMD:C_0805_2012Metric_Pad1.18x1.45mm_HandSolder, B.Cu at (492.4, 138.7)
- added C38: 104, Capacitor_SMD:C_0805_2012Metric_Pad1.18x1.45mm_HandSolder, B.Cu at (498.6, 180.7)
- added C39: 104, Capacitor_SMD:C_0805_2012Metric_Pad1.18x1.45mm_HandSolder, B.Cu at (97.7, 205.4)
- added C40: 104, Capacitor_SMD:C_0805_2012Metric_Pad1.18x1.45mm_HandSolder, B.Cu at (148.5, 194.9)
- added C41: 104, Capacitor_SMD:C_0805_2012Metric_Pad1.18x1.45mm_HandSolder, B.Cu at (230.0, 204.6)
- added C42: 104, Capacitor_SMD:C_0805_2012Metric_Pad1.18x1.45mm_HandSolder, B.Cu at (362.2, 92.5)
- added C43: 104, Capacitor_SMD:C_0805_2012Metric_Pad1.18x1.45mm_HandSolder, B.Cu at (445.4, 96.8)
- added C44: 104, Capacitor_SMD:C_0805_2012Metric_Pad1.18x1.45mm_HandSolder, B.Cu at (311.8, 200.5)
- added C45: 104, Capacitor_SMD:C_0805_2012Metric_Pad1.18x1.45mm_HandSolder, B.Cu at (430.7, 207.0)
- added LED107: IN-PI55TATPRPGPB, ul_IN-PI55TATPRPGPB:IN-PI55TATPRPGPB, B.Cu at (103.5, 95.4)
- added LED108: IN-PI55TATPRPGPB, ul_IN-PI55TATPRPGPB:IN-PI55TATPRPGPB, B.Cu at (193.2, 97.2)
- added LED109: IN-PI55TATPRPGPB, ul_IN-PI55TATPRPGPB:IN-PI55TATPRPGPB, B.Cu at (278.8, 97.0)
- added LED110: IN-PI55TATPRPGPB, ul_IN-PI55TATPRPGPB:IN-PI55TATPRPGPB, B.Cu at (76.2, 141.2)
- added LED111: IN-PI55TATPRPGPB, ul_IN-PI55TATPRPGPB:IN-PI55TATPRPGPB, B.Cu at (77.9, 174.6)
- added LED112: IN-PI55TATPRPGPB, ul_IN-PI55TATPRPGPB:IN-PI55TATPRPGPB, B.Cu at (491.7, 134.2)
- added LED113: IN-PI55TATPRPGPB, ul_IN-PI55TATPRPGPB:IN-PI55TATPRPGPB, B.Cu at (498.0, 176.3)
- added LED114: IN-PI55TATPRPGPB, ul_IN-PI55TATPRPGPB:IN-PI55TATPRPGPB, B.Cu at (97.0, 200.7)
- added LED115: IN-PI55TATPRPGPB, ul_IN-PI55TATPRPGPB:IN-PI55TATPRPGPB, B.Cu at (148.8, 199.5)
- added LED116: IN-PI55TATPRPGPB, ul_IN-PI55TATPRPGPB:IN-PI55TATPRPGPB, B.Cu at (229.4, 199.9)
- added LED117: IN-PI55TATPRPGPB, ul_IN-PI55TATPRPGPB:IN-PI55TATPRPGPB, B.Cu at (362.7, 97.0)
- added LED118: IN-PI55TATPRPGPB, ul_IN-PI55TATPRPGPB:IN-PI55TATPRPGPB, B.Cu at (440.7, 94.4)
- added LED119: IN-PI55TATPRPGPB, ul_IN-PI55TATPRPGPB:IN-PI55TATPRPGPB, B.Cu at (311.3, 196.0)
- added LED120: IN-PI55TATPRPGPB, ul_IN-PI55TATPRPGPB:IN-PI55TATPRPGPB, B.Cu at (430.1, 202.5)
- added R3: 500, Resistor_SMD:R_0805_2012Metric_Pad1.20x1.40mm_HandSolder, B.Cu at (443.4, 89.5)
- added R4: 500, Resistor_SMD:R_0805_2012Metric_Pad1.20x1.40mm_HandSolder, B.Cu at (496.1, 137.8)
- added R5: 27, Resistor_SMD:R_0805_2012Metric_Pad1.20x1.40mm_HandSolder, B.Cu at (468.4, 105.8)
- Y1: value XTAL_ABLS_ABR -> ABLS-12.000MHZ-B4-T
- moved R8 2.03 mm to (475.0, 89.0)
- moved D38 1.55 mm to (492.1, 127.8)
- moved SW2 1.40 mm to (482.0, 90.2)
- moved R_B5 0.76 mm to (159.6, 192.9)
- moved C28 0.76 mm to (468.2, 89.3)
- moved R_B4 0.68 mm to (157.7, 202.8), turned to 90 degrees
- moved C30 0.64 mm to (453.4, 99.8), turned to 0 degrees
- moved C31 0.63 mm to (456.6, 104.4)
- moved U3 0.58 mm to (472.2, 93.2)
- moved C12 0.36 mm to (481.7, 97.3)
- moved R14 0.25 mm to (464.2, 94.7)
- moved C13 0.13 mm to (467.4, 101.3)
- moved C14 0.13 mm to (467.9, 109.9)
- moved C6 0.13 mm to (467.4, 103.6)
Connections:
- U1 pad 11: ROW3 -> ROW4
- U1 pad 12: ROW2 -> ROW3
- U1 pad 13: ROW1 -> ROW2
- U1 pad 14: ROW0 -> ROW1
- U1 pad 15: RGB_DI -> ROW0
- U1 pad 4: COL3 -> RGB_DI
- U1 pad 5: COL2 -> COL3
- U1 pad 6: COL1 -> COL2
- U1 pad 7: COL0 -> COL1
- U1 pad 8: ROW5 -> COL0
- U1 pad 9: ROW4 -> ROW5
- U2 pad 49: unconnected-(U2-GND-Pad49) -> GND
- U4 pad 49: unconnected-(U4-GND-Pad49) -> GND
Routing:
- net +5V: track 506.0 -> 1431.2 mm, vias 6 -> 17
- net GND: track 171.5 -> 330.5 mm, vias 16 -> 17
- net Net-(LED119-DOUT): track 0.00 -> 125.1 mm, vias 0 -> 2
- net Net-(LED117-DIN): track 0.00 -> 94.8 mm, vias 0 -> 2
- net Net-(LED107-DIN): track 0.00 -> 90.5 mm, vias 0 -> 2
- net Net-(LED108-DIN): track 0.00 -> 85.7 mm, vias 0 -> 2
- net Net-(LED109-DIN): track 0.00 -> 84.3 mm, vias 0 -> 2
- net Net-(LED116-DOUT): track 0.00 -> 83.7 mm, vias 0 -> 2
- net Net-(LED115-DOUT): track 0.00 -> 83.0 mm, vias 0 -> 2
- net Net-(LED113-DIN): track 0.00 -> 79.4 mm, vias 0 -> 2
- net Net-(LED107-DOUT): track 0.00 -> 78.7 mm
- net RGB_DI: track 0.00 -> 66.3 mm
- net Net-(LED112-DIN): track 0.00 -> 55.1 mm, vias 0 -> 2
- net Net-(LED114-DOUT): track 0.00 -> 53.2 mm, vias 0 -> 2
- net Net-(LED111-DOUT): track 0.00 -> 41.6 mm, vias 0 -> 2
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Other:
- board outline added: 438.7 x 131.6 mm

Commit message: Fixed Errors Relating to edge cuts
Parts:
- removed R4: 500, Resistor_SMD:R_0805_2012Metric_Pad1.20x1.40mm_HandSolder
- LED107, LED108, LED109, LED110, LED111, LED112, LED113, LED114, LED115, LED116, LED117, LED118, LED119, LED120: value IN-PI55TATPRPGPB -> LED_IN-PI55TAT_INL
Connections:
- LED112 pad 2: Net-(LED112-DOUT) -> unconnected-(LED112-DOUT-Pad2)
Routing:
- net Net-(LED112-DOUT): track 6.04 -> 0.00 mm
- net GND: track 330.5 -> 336.2 mm
- net COL0: track 560.3 -> 558.6 mm
- net COL5: track 408.6 -> 408.0 mm
Other:
- outline, holes or cut-outs redrawn
